File: pcb/soc.sch (KiCad schematic (older format))
At the start: 22 parts, among them IC7 CC2541F128RHAT, J1 CC Debugger, SW1 SW_Push, Y1 32 Mhz

Commit message: Migrated project/libraries to KiCad nightly build
Revision: 821668d96

Reason being the simulator feature and the better library management.
Parts:
- AE1: symbol Antenna -> device:Antenna
- C20, C21, C22, C23, C24, C25, C26, C27, C28, C29: symbol C_Small -> device:C_Small
- IC7: symbol CC2541F128RHAT -> CC2541F128RHAT:CC2541F128RHAT
- J1: symbol Conn_02x05_Odd_Even -> conn:Conn_02x05_Odd_Even
- L1, L2, L3, L4: symbol L_Small -> device:L_Small
- R2, R3, R4: symbol R -> device:R
- SW1: symbol SW_Push -> switches:SW_Push
- Y1: symbol Crystal -> device:Crystal
Changed lines of the file:
@@
-EESchema Schematic File Version 2
-LIBS:power
-LIBS:device
-LIBS:switches
-LIBS:relays
-LIBS:motors
-LIBS:transistors
-LIBS:conn
-LIBS:linear
-LIBS:regul
-LIBS:74xx
-LIBS:cmos4000
-LIBS:adc-dac
-LIBS:memory
-LIBS:xilinx
-LIBS:microcontrollers
-LIBS:dsp
-LIBS:microchip
-LIBS:analog_switches
-LIBS:motorola
-LIBS:texas
-LIBS:intel
-LIBS:audio
-LIBS:interface
-LIBS:digital-audio
-LIBS:philips
-LIBS:display
-LIBS:cypress
-LIBS:siliconi
-LIBS:opto
-LIBS:atmel
-LIBS:contrib
-LIBS:valves
-LIBS:LPV802DGKT
-LIBS:SI2323DS-T1-E3
-LIBS:1N4148X-TP
-LIBS:TLV3691IDCKR
-LIBS:IRA-S210ST01
-LIBS:CC2540F256RHAT
-LIBS:CC2541F256RHAR
-LIBS:CC2541F128RHAT
-LIBS:MAX44009EDT+T
+EESchema Schematic File Version 4
 LIBS:pir-cache
-EELAYER 25 0
+EELAYER 26 0
 EELAYER END
 $Descr A4 11693 8268
@@
 PIR_LOW
 $Comp
-L CC2541F128RHAT IC7
+L CC2541F128RHAT:CC2541F128RHAT IC7
 U 1 1 5A76B408
 P 4250 3100
@@
 SHUTTER
 $Comp
-L Earth #PWR24
+L power:Earth #PWR24
 U 1 1 5A76DE63
 P 3850 2750
@@
 $EndComp
 $Comp
-L VCC #PWR33
+L power:VCC #PWR33
 U 1 1 5A76DE98
 P 6550 3350
@@
 $EndComp
 $Comp
-L VCC #PWR25
+L power:VCC #PWR25
 U 1 1 5A76E05D
 P 3850 4250
@@
 $EndComp
 $Comp
-L VCC #PWR30
+L power:VCC #PWR30
 U 1 1 5A76E1D1
 P 5550 1750
@@
 $EndComp
 $Comp
-L VCC #PWR28
+L power:VCC #PWR28
 U 1 1 5A76E1F7
 P 4750 1750
@@
 NoConn ~ 5350 1900
 $Comp
-L R R4
+L device:R R4
 U 1 1 5A76E4F0
 P 6150 3100
@@
 $EndComp
 $Comp
-L C_Small C25
+L device:C_Small C25
 U 1 1 5A76E83A
 P 7000 3350
@@
 $EndComp
 $Comp
-L C_Small C26
+L device:C_Small C26
 U 1 1 5A76EB9B
 P 7000 3750
@@
 $EndComp
 $Comp
-L C_Small C28
+L device:C_Small C28
 U 1 1 5A76EBCB
 P 7500 3350
@@
 $EndComp
 $Comp
-L C_Small C27
+L device:C_Small C27
 U 1 1 5A76EC10
 P 7300 4100
@@
 $EndComp
 $Comp
-L L_Small L2
+L device:L_Small L2
 U 1 1 5A76EC99
 P 7500 3750
@@
 $EndComp
 $Comp
-L Earth #PWR35
+L power:Earth #PWR35
 U 1 1 5A76EF79
 P 7300 4350
@@
 $EndComp
 $Comp
-L Earth #PWR32
+L power:Earth #PWR32
 U 1 1 5A76F127
 P 6300 3200
@@
 $EndComp
 $Comp
-L Earth #PWR36
+L power:Earth #PWR36
 U 1 1 5A76F249
 P 7400 2900
@@
 $EndComp
 $Comp
-L L_Small L1
+L device:L_Small L1
 U 1 1 5A76F269
 P 7200 3100
@@
 $EndComp
 $Comp
-L L_Small L3
+L device:L_Small L3
 U 1 1 5A76F317
 P 8000 3550
@@
 $EndComp
 $Comp
-L L_Small L4
+L device:L_Small L4
 U 1 1 5A76F356
 P 8400 3550
@@
 $EndComp
 $Comp
-L C_Small C29
+L device:C_Small C29
 U 1 1 5A76F398
 P 8200 4100
@@
 $EndComp
 $Comp
-L Earth #PWR37
+L power:Earth #PWR37
 U 1 1 5A76F405
 P 8200 4350
@@
 $EndComp
 $Comp
-L Antenna AE1
+L device:Antenna AE1
 U 1 1 5A76F5F0
 P 8800 3250
@@
 $EndComp
 $Comp
-L C_Small C23
+L device:C_Small C23
 U 1 1 5A76F951
 P 6150 4800
@@
 $EndComp
 $Comp
-L C_Small C24
+L device:C_Small C24
 U 1 1 5A76F9C8
 P 6550 4800
@@
 $EndComp
 $Comp
-L Crystal Y1
+L device:Crystal Y1
 U 1 1 5A76FA28
 P 6350 4400
@@
 Connection ~ 6550 4400
 $Comp
-L Earth #PWR31
+L power:Earth #PWR31
 U 1 1 5A76FDE5
 P 6150 5000
@@
 $EndComp
 $Comp
-L Earth #PWR34
+L power:Earth #PWR34
 U 1 1 5A76FE1D
 P 6550 5000
@@
 	5150 1900 5150 1600
 $Comp
-L Conn_02x05_Odd_Even J1
+L conn:Conn_02x05_Odd_Even J1
 U 1 1 5A762773
 P 2250 7000
@@
 	1900 6900 2050 6900
 $Comp
-L Earth #PWR22
+L power:Earth #PWR22
 U 1 1 5A762D06
 P 1800 6650
@@
 	1800 6550 1800 6650
 $Comp
-L VCC #PWR23
+L power:VCC #PWR23
 U 1 1 5A762F97
 P 2650 6650
@@
 	4950 1800 4950 1900
 $Comp
-L R R3
+L device:R R3
 U 1 1 5A7649A0
 P 5700 5500
@@
 	6000 5500 5850 5500
 $Comp
-L C_Small C22
+L device:C_Small C22
 U 1 1 5A764EFF
 P 5450 5750
@@
 $EndComp
 $Comp
-L Earth #PWR29
+L power:Earth #PWR29
 U 1 1 5A764F83
 P 5450 6000
@@
 CC3V3
 $Comp
-L VCC #PWR19
+L power:VCC #PWR19
 U 1 1 5A76CA51
 P 1050 1400
@@
 $EndComp
 $Comp
-L R R2
+L device:R R2
 U 1 1 5A76CB17
 P 1050 1700
@@
 $EndComp
 $Comp
-L SW_Push SW1
+L switches:SW_Push SW1
 U 1 1 5A76CDA3
 P 1050 2200
@@
 $EndComp
 $Comp
-L C_Small C20
+L device:C_Small C20
 U 1 1 5A76CF70
 P 1500 2200
@@
 $EndComp
 $Comp
-L Earth #PWR20
+L power:Earth #PWR20
 U 1 1 5A76D398
 P 1050 2550
@@
 Connection ~ 1050 1950
 $Comp
-L Earth #PWR21
+L power:Earth #PWR21
 U 1 1 5A76D8AA
 P 1500 2400
@@
 NoConn ~ 4650 4800
 $Comp
-L Earth #PWR27
+L power:Earth #PWR27
 U 1 1 5A76FB36
 P 4250 1900
@@
 	4250 1800 4250 1900
 $Comp
-L C_Small C21
+L device:C_Small C21
 U 1 1 5A770125
 P 4000 1650
@@
 $EndComp
 $Comp
-L Earth #PWR26
+L power:Earth #PWR26
 U 1 1 5A7703A1
 P 4000 1900

Commit message: Added E-Ink display
Parts:
- removed AE1: 50 Ohm, symbol device:Antenna
- removed C20: 2200pF, symbol device:C_Small
- removed C25, C26, C29: 18pF, symbol device:C_Small
- removed C27, C28: 1pF, symbol device:C_Small
- removed IC7: CC2541F128RHAT, QFN50P600X600X100-41N, symbol CC2541F128RHAT:CC2541F128RHAT
- removed L1, L2: 2nH, symbol device:L_Small
- removed L3: 1nH, symbol device:L_Small
- removed L4: 3nH, symbol device:L_Small
- removed R2: 47K, symbol device:R
- removed SW1: SW_Push, symbol switches:SW_Push
- added U?: STM32L051C6Tx, Housings_QFP:LQFP-48_7x7mm_Pitch0.5mm, symbol stm32:STM32L051C6Tx
Connections:
- wire segments 95 -> 78
Other:
- note removed: "User button"
- moved on the sheet: C21, C22, C23, C24, R3, R4, Y1
