File: pcb/soc.sch (KiCad schematic (older format))
At the start: 31 parts, among them J3 SWD, J4 UART, U1 STM32L476RETx, Y1 32 Mhz, Y2 32 Mhz

Commit message: Added testpoints
Parts:
- added TP29: TEST, symbol TEST
- renumbered R24 to R27, TP1 to TP23, TP2 to TP24, TP3 to TP25, TP4 to TP26, TP5 to TP27, TP6 to TP28, TP7 to TP30, TP8 to TP31, TP9 to TP32, TP10 to TP33, TP11 to TP34, TP12 to TP35, TP13 to TP36, TP14 to TP37, TP15 to TP38, TP16 to TP39, TP17 to TP40, TP18 to TP41
Changed lines of the file:
@@
 EINK_PWR
 $Comp
-L power:Earth #PWR040
+L power:Earth #PWR53
 U 1 1 5A7F7482
 P 8800 3400
-F 0 "#PWR040" H 8800 3150 50  0001 C CNN
+F 0 "#PWR53" H 8800 3150 50  0001 C CNN
 F 1 "Earth" H 8800 3250 50  0001 C CNN
 F 2 "" H 8800 3400 50  0001 C CNN
@@
 $EndComp
 $Comp
-L power:VCC #PWR041
+L power:VCC #PWR50
 U 1 1 5A7F7645
 P 7850 3250
-F 0 "#PWR041" H 7850 3100 50  0001 C CNN
+F 0 "#PWR50" H 7850 3100 50  0001 C CNN
 F 1 "VCC" H 7850 3400 50  0000 C CNN
 F 2 "" H 7850 3250 50  0001 C CNN
@@
 $EndComp
 $Comp
-L power:Earth #PWR042
+L power:Earth #PWR52
 U 1 1 5A7F7940
 P 8400 7950
-F 0 "#PWR042" H 8400 7700 50  0001 C CNN
+F 0 "#PWR52" H 8400 7700 50  0001 C CNN
 F 1 "Earth" H 8400 7800 50  0001 C CNN
 F 2 "" H 8400 7950 50  0001 C CNN
@@
 $EndComp
 $Comp
-L power:Earth #PWR043
+L power:Earth #PWR41
 U 1 1 5A7F8695
 P 800 6400
-F 0 "#PWR043" H 800 6150 50  0001 C CNN
+F 0 "#PWR41" H 800 6150 50  0001 C CNN
 F 1 "Earth" H 800 6250 50  0001 C CNN
 F 2 "" H 800 6400 50  0001 C CNN
@@
 $EndComp
 $Comp
-L power:Earth #PWR044
+L power:Earth #PWR42
 U 1 1 5A7F869B
 P 1200 6400
-F 0 "#PWR044" H 1200 6150 50  0001 C CNN
+F 0 "#PWR42" H 1200 6150 50  0001 C CNN
 F 1 "Earth" H 1200 6250 50  0001 C CNN
 F 2 "" H 1200 6400 50  0001 C CNN
@@
 $EndComp
 $Comp
-L power:Earth #PWR045
+L power:Earth #PWR44
 U 1 1 5A7F8A34
 P 1500 8300
-F 0 "#PWR045" H 1500 8050 50  0001 C CNN
+F 0 "#PWR44" H 1500 8050 50  0001 C CNN
 F 1 "Earth" H 1500 8150 50  0001 C CNN
 F 2 "" H 1500 8300 50  0001 C CNN
@@
 $EndComp
 $Comp
-L power:Earth #PWR046
+L power:Earth #PWR47
 U 1 1 5A7F8A3A
 P 1900 8300
-F 0 "#PWR046" H 1900 8050 50  0001 C CNN
+F 0 "#PWR47" H 1900 8050 50  0001 C CNN
 F 1 "Earth" H 1900 8150 50  0001 C CNN
 F 2 "" H 1900 8300 50  0001 C CNN
@@
 $EndComp
 $Comp
-L device:R R24
+L device:R R27
 U 1 1 5A7F96A5
 P 1500 3650
-F 0 "R24" V 1580 3650 50  0000 C CNN
+F 0 "R27" V 1580 3650 50  0000 C CNN
 F 1 "1K" V 1500 3650 50  0000 C CNN
 F 2 "" V 1430 3650 50  0001 C CNN
@@
 $EndComp
 $Comp
-L power:Earth #PWR047
+L power:Earth #PWR46
 U 1 1 5A7F96B5
 P 1900 4050
-F 0 "#PWR047" H 1900 3800 50  0001 C CNN
+F 0 "#PWR46" H 1900 3800 50  0001 C CNN
 F 1 "Earth" H 1900 3900 50  0001 C CNN
 F 2 "" H 1900 4050 50  0001 C CNN
@@
 $EndComp
 $Comp
-L Earth #PWR048
+L Earth #PWR43
 U 1 1 5A7FA9BE
 P 1400 4200
-F 0 "#PWR048" H 1400 3950 50  0001 C CNN
+F 0 "#PWR43" H 1400 3950 50  0001 C CNN
 F 1 "Earth" H 1400 4050 50  0001 C CNN
 F 2 "" H 1400 4200 50  0001 C CNN
@@
 $EndComp
 $Comp
-L power:VCC #PWR049
+L power:VCC #PWR40
 U 1 1 5A7FAB49
 P 600 4150
-F 0 "#PWR049" H 600 4000 50  0001 C CNN
+F 0 "#PWR40" H 600 4000 50  0001 C CNN
 F 1 "VCC" H 600 4300 50  0000 C CNN
 F 2 "" H 600 4150 50  0001 C CNN
@@
 SWDIO
 $Comp
-L power:Earth #PWR050
+L power:Earth #PWR45
 U 1 1 5A7FC200
 P 1650 10100
-F 0 "#PWR050" H 1650 9850 50  0001 C CNN
+F 0 "#PWR45" H 1650 9850 50  0001 C CNN
 F 1 "Earth" H 1650 9950 50  0001 C CNN
 F 2 "" H 1650 10100 50  0001 C CNN
@@
 	3600 9950 3750 9950
 $Comp
-L power:Earth #PWR051
+L power:Earth #PWR49
 U 1 1 5A7FF0DB
 P 3900 10100
-F 0 "#PWR051" H 3900 9850 50  0001 C CNN
+F 0 "#PWR49" H 3900 9850 50  0001 C CNN
 F 1 "Earth" H 3900 9950 50  0001 C CNN
 F 2 "" H 3900 10100 50  0001 C CNN
@@
 	14750 6050 14550 6050
 $Comp
-L power:VCC #PWR052
+L power:VCC #PWR48
 U 1 1 5A8061D8
 P 2150 4550
-F 0 "#PWR052" H 2150 4400 50  0001 C CNN
+F 0 "#PWR48" H 2150 4400 50  0001 C CNN
 F 1 "VCC" H 2150 4700 50  0000 C CNN
 F 2 "" H 2150 4550 50  0001 C CNN
@@
 $EndComp
 $Comp
-L power:Earth #PWR053
+L power:Earth #PWR51
 U 1 1 5A806A82
 P 7850 3550
-F 0 "#PWR053" H 7850 3300 50  0001 C CNN
+F 0 "#PWR51" H 7850 3300 50  0001 C CNN
 F 1 "Earth" H 7850 3400 50  0001 C CNN
 F 2 "" H 7850 3550 50  0001 C CNN
@@
 	2150 5950 2350 5950
 $Comp
-L TEST TP13
+L TEST TP36
 U 1 1 5A841551
 P 2350 5650
-F 0 "TP13" H 2350 5950 50  0000 C BNN
+F 0 "TP36" H 2350 5950 50  0000 C BNN
 F 1 "TEST" H 2350 5900 50  0000 C CNN
 F 2 "" H 2350 5650 50  0001 C CNN
@@
 $EndComp
 $Comp
-L TEST TP7
+L TEST TP30
 U 1 1 5A8419B6
 P 2250 6050
-F 0 "TP7" H 2250 6350 50  0000 C BNN
+F 0 "TP30" H 2250 6350 50  0000 C BNN
 F 1 "TEST" H 2250 6300 50  0000 C CNN
 F 2 "" H 2250 6050 50  0001 C CNN
@@
 $EndComp
 $Comp
-L TEST TP1
+L TEST TP23
 U 1 1 5A841A23
 P 1950 6150
-F 0 "TP1" H 1950 6450 50  0000 C BNN
+F 0 "TP23" H 1950 6450 50  0000 C BNN
 F 1 "TEST" H 1950 6400 50  0000 C CNN
 F 2 "" H 1950 6150 50  0001 C CNN
@@
 $EndComp
 $Comp
-L TEST TP8
+L TEST TP31
 U 1 1 5A841A77
 P 2250 6250
-F 0 "TP8" H 2250 6550 50  0000 C BNN
+F 0 "TP31" H 2250 6550 50  0000 C BNN
 F 1 "TEST" H 2250 6500 50  0000 C CNN
 F 2 "" H 2250 6250 50  0001 C CNN
@@
 $EndComp
 $Comp
-L TEST TP2
+L TEST TP24
 U 1 1 5A841ACA
 P 1950 6350
-F 0 "TP2" H 1950 6650 50  0000 C BNN
+F 0 "TP24" H 1950 6650 50  0000 C BNN
 F 1 "TEST" H 1950 6600 50  0000 C CNN
 F 2 "" H 1950 6350 50  0001 C CNN
@@
 $EndComp
 $Comp
-L TEST TP9
+L TEST TP32
 U 1 1 5A841B2C
 P 2250 6450
-F 0 "TP9" H 2250 6750 50  0000 C BNN
+F 0 "TP32" H 2250 6750 50  0000 C BNN
 F 1 "TEST" H 2250 6700 50  0000 C CNN
 F 2 "" H 2250 6450 50  0001 C CNN
@@
 $EndComp
 $Comp
-L TEST TP3
+L TEST TP25
 U 1 1 5A841B81
 P 1950 6550
-F 0 "TP3" H 1950 6850 50  0000 C BNN
+F 0 "TP25" H 1950 6850 50  0000 C BNN
 F 1 "TEST" H 1950 6800 50  0000 C CNN
 F 2 "" H 1950 6550 50  0001 C CNN
@@
 $EndComp
 $Comp
-L TEST TP10
+L TEST TP33
 U 1 1 5A841BED
 P 2250 6650
-F 0 "TP10" H 2250 6950 50  0000 C BNN
+F 0 "TP33" H 2250 6950 50  0000 C BNN
 F 1 "TEST" H 2250 6900 50  0000 C CNN
 F 2 "" H 2250 6650 50  0001 C CNN
@@
 $EndComp
 $Comp
-L TEST TP4
+L TEST TP26
 U 1 1 5A841C4E
 P 1950 6750
-F 0 "TP4" H 1950 7050 50  0000 C BNN
+F 0 "TP26" H 1950 7050 50  0000 C BNN
 F 1 "TEST" H 1950 7000 50  0000 C CNN
 F 2 "" H 1950 6750 50  0001 C CNN
@@
 $EndComp
 $Comp
-L TEST TP11
+L TEST TP34
 U 1 1 5A841CC0
 P 2250 6850
-F 0 "TP11" H 2250 7150 50  0000 C BNN
+F 0 "TP34" H 2250 7150 50  0000 C BNN
 F 1 "TEST" H 2250 7100 50  0000 C CNN
 F 2 "" H 2250 6850 50  0001 C CNN
@@
 $EndComp
 $Comp
-L TEST TP5
+L TEST TP27
 U 1 1 5A841D23
 P 1950 6950
-F 0 "TP5" H 1950 7250 50  0000 C BNN
+F 0 "TP27" H 1950 7250 50  0000 C BNN
 F 1 "TEST" H 1950 7200 50  0000 C CNN
 F 2 "" H 1950 6950 50  0001 C CNN
@@
 $EndComp
 $Comp
-L TEST TP12
+L TEST TP35
 U 1 1 5A841D8F
 P 2250 7050
-F 0 "TP12" H 2250 7350 50  0000 C BNN
+F 0 "TP35" H 2250 7350 50  0000 C BNN
 F 1 "TEST" H 2250 7300 50  0000 C CNN
 F 2 "" H 2250 7050 50  0001 C CNN
@@
 $EndComp
 $Comp
-L TEST TP6
+L TEST TP28
 U 1 1 5A841DFE
 P 1950 7150
-F 0 "TP6" H 1950 7450 50  0000 C BNN
+F 0 "TP28" H 1950 7450 50  0000 C BNN
 F 1 "TEST" H 1950 7400 50  0000 C CNN
 F 2 "" H 1950 7150 50  0001 C CNN
@@
 	1950 7150 2350 7150
 $Comp
-L TEST TP14
+L TEST TP37
 U 1 1 5A842F88
 P 15550 4350
-F 0 "TP14" H 15550 4650 50  0000 C BNN
+F 0 "TP37" H 15550 4650 50  0000 C BNN
 F 1 "TEST" H 15550 4600 50  0000 C CNN
 F 2 "" H 15550 4350 50  0001 C CNN
@@
 $EndComp
 $Comp
-L TEST TP15
+L TEST TP38
 U 1 1 5A8431E8
 P 15550 4550
-F 0 "TP15" H 15550 4850 50  0000 C BNN
+F 0 "TP38" H 15550 4850 50  0000 C BNN
 F 1 "TEST" H 15550 4800 50  0000 C CNN
 F 2 "" H 15550 4550 50  0001 C CNN
@@
 $EndComp
 $Comp
-L TEST TP16
+L TEST TP39
 U 1 1 5A843254
 P 15550 4950
-F 0 "TP16" H 15550 5250 50  0000 C BNN
+F 0 "TP39" H 15550 5250 50  0000 C BNN
 F 1 "TEST" H 15550 5200 50  0000 C CNN
 F 2 "" H 15550 4950 50  0001 C CNN
@@
 $EndComp
 $Comp
-L TEST TP17
+L TEST TP40
 U 1 1 5A84333F
 P 15550 5250
-F 0 "TP17" H 15550 5550 50  0000 C BNN
+F 0 "TP40" H 15550 5550 50  0000 C BNN
 F 1 "TEST" H 15550 5500 50  0000 C CNN
 F 2 "" H 15550 5250 50  0001 C CNN
@@
 Ambient
 $Comp
-L TEST TP18
+L TEST TP41
 U 1 1 5A80E6EA
 P 15550 6250
-F 0 "TP18" H 15550 6550 50  0000 C BNN
+F 0 "TP41" H 15550 6550 50  0000 C BNN
 F 1 "TEST" H 15550 6500 50  0000 C CNN
 F 2 "" H 15550 6250 50  0001 C CNN
@@
 	0    1    1    0
 $EndComp
+$Comp
+L TEST TP29
+U 1 1 5A83B349
+P 2200 3650
+F 0 "TP29" H 2200 3950 50  0000 C BNN
+F 1 "TEST" H 2200 3900 50  0000 C CNN
+F 2 "" H 2200 3650 50  0001 C CNN
+F 3 "" H 2200 3650 50  0001 C CNN
+	1    2200 3650
+	1    0    0    -1
+$EndComp
 $EndSCHEMATC

Commit message: Assigned footprints to all components
Parts:
- C35, C36, C37, C38, C39, C40: footprint (none) -> Capacitors_SMD:C_1210
- J3: footprint (none) -> Pin_Headers:Pin_Header_Angled_1x06_Pitch2.54mm
- J4, JP3: footprint (none) -> Pin_Headers:Pin_Header_Angled_1x03_Pitch2.54mm
- R27: footprint (none) -> Resistors_SMD:R_1210
- TP23, TP24, TP25, TP26, TP27, TP28, TP29, TP30, TP31, TP32, TP33, TP34, TP35, TP36, TP37, TP38, TP39, TP40, TP41: footprint (none) -> Measurement_Points:Measurement_Point_Round-TH_Small
- U1: footprint LQFP64 -> Housings_QFP:LQFP-64_10x10mm_Pitch0.5mm
- Y1, Y2: footprint (none) -> Crystals:Crystal_SMD_2012-2pin_2.0x1.2mm_HandSoldering
Changed lines of the file:
@@
 F 0 "C35" H 810 6270 50  0000 L CNN
 F 1 "12pF" H 810 6120 50  0000 L CNN
-F 2 "" H 800 6200 50  0001 C CNN
+F 2 "Capacitors_SMD:C_1210" H 800 6200 50  0001 C CNN
 F 3 "" H 800 6200 50  0001 C CNN
 	1    800  6200
@@
 F 0 "C36" H 1210 6270 50  0000 L CNN
 F 1 "12pF" H 1210 6120 50  0000 L CNN
-F 2 "" H 1200 6200 50  0001 C CNN
+F 2 "Capacitors_SMD:C_1210" H 1200 6200 50  0001 C CNN
 F 3 "" H 1200 6200 50  0001 C CNN
 	1    1200 6200
@@
 F 0 "Y1" H 1000 5950 50  0000 C CNN
 F 1 "32 Mhz" H 1000 5650 50  0000 C CNN
-F 2 "" H 1000 5800 50  0001 C CNN
+F 2 "Crystals:Crystal_SMD_2012-2pin_2.0x1.2mm_HandSoldering" H 1000 5800 50  0001 C CNN
 F 3 "" H 1000 5800 50  0001 C CNN
 	1    1000 5800
@@
 F 0 "C37" H 1510 8170 50  0000 L CNN
 F 1 "12pF" H 1510 8020 50  0000 L CNN
-F 2 "" H 1500 8100 50  0001 C CNN
+F 2 "Capacitors_SMD:C_1210" H 1500 8100 50  0001 C CNN
 F 3 "" H 1500 8100 50  0001 C CNN
 	1    1500 8100
@@
 F 0 "C39" H 1910 8170 50  0000 L CNN
 F 1 "12pF" H 1910 8020 50  0000 L CNN
-F 2 "" H 1900 8100 50  0001 C CNN
+F 2 "Capacitors_SMD:C_1210" H 1900 8100 50  0001 C CNN
 F 3 "" H 1900 8100 50  0001 C CNN
 	1    1900 8100
@@
 F 0 "Y2" H 1700 7850 50  0000 C CNN
 F 1 "32 Mhz" H 1700 7550 50  0000 C CNN
-F 2 "" H 1700 7700 50  0001 C CNN
+F 2 "Crystals:Crystal_SMD_2012-2pin_2.0x1.2mm_HandSoldering" H 1700 7700 50  0001 C CNN
 F 3 "" H 1700 7700 50  0001 C CNN
 	1    1700 7700
@@
 F 0 "R27" V 1580 3650 50  0000 C CNN
 F 1 "1K" V 1500 3650 50  0000 C CNN
-F 2 "" V 1430 3650 50  0001 C CNN
+F 2 "Resistors_SMD:R_1210" V 1430 3650 50  0001 C CNN
 F 3 "" H 1500 3650 50  0001 C CNN
 	1    1500 3650
@@
 F 0 "C38" H 1910 3870 50  0000 L CNN
 F 1 "100nF" H 1910 3720 50  0000 L CNN
-F 2 "" H 1900 3800 50  0001 C CNN
+F 2 "Capacitors_SMD:C_1210" H 1900 3800 50  0001 C CNN
 F 3 "" H 1900 3800 50  0001 C CNN
 	1    1900 3800
@@
 F 0 "JP3" H 1100 4050 50  0000 L CNN
 F 1 "Jumper_NC_Dual" H 1050 4250 50  0000 C BNN
-F 2 "" H 1050 4150 50  0001 C CNN
+F 2 "Pin_Headers:Pin_Header_Angled_1x03_Pitch2.54mm" H 1050 4150 50  0001 C CNN
 F 3 "" H 1050 4150 50  0001 C CNN
 	1    1050 4150
@@
 F 0 "J3" H 1450 10400 50  0000 C CNN
 F 1 "SWD" H 1450 9700 50  0000 C CNN
-F 2 "" H 1450 10100 50  0001 C CNN
+F 2 "Pin_Headers:Pin_Header_Angled_1x06_Pitch2.54mm" H 1450 10100 50  0001 C CNN
 F 3 "" H 1450 10100 50  0001 C CNN
 	1    1450 10100
@@
 F 0 "J4" H 3400 10150 50  0000 C CNN
 F 1 "UART" H 3400 9750 50  0000 C CNN
-F 2 "" H 3400 9950 50  0001 C CNN
+F 2 "Pin_Headers:Pin_Header_Angled_1x03_Pitch2.54mm" H 3400 9950 50  0001 C CNN
 F 3 "" H 3400 9950 50  0001 C CNN
 	1    3400 9950
@@
 F 0 "C40" H 7860 3520 50  0000 L CNN
 F 1 "100nF" H 7860 3370 50  0000 L CNN
-F 2 "" H 7850 3450 50  0001 C CNN
+F 2 "Capacitors_SMD:C_1210" H 7850 3450 50  0001 C CNN
 F 3 "" H 7850 3450 50  0001 C CNN
 	1    7850 3450
@@
 F 0 "U1" H 2450 7775 50  0000 L BNN
 F 1 "STM32L476RETx" H 14450 7775 50  0000 R BNN
-F 2 "LQFP64" H 14450 7725 50  0001 R TNN
+F 2 "Housings_QFP:LQFP-64_10x10mm_Pitch0.5mm" H 14450 7725 50  0001 R TNN
 F 3 "" H 8450 5750 50  0001 C CNN
 	1    8450 5750
@@
 F 0 "TP36" H 2350 5950 50  0000 C BNN
 F 1 "TEST" H 2350 5900 50  0000 C CNN
-F 2 "" H 2350 5650 50  0001 C CNN
+F 2 "Measurement_Points:Measurement_Point_Round-TH_Small" H 2350 5650 50  0001 C CNN
 F 3 "" H 2350 5650 50  0001 C CNN
 	1    2350 5650
@@
 F 0 "TP30" H 2250 6350 50  0000 C BNN
 F 1 "TEST" H 2250 6300 50  0000 C CNN
-F 2 "" H 2250 6050 50  0001 C CNN
+F 2 "Measurement_Points:Measurement_Point_Round-TH_Small" H 2250 6050 50  0001 C CNN
 F 3 "" H 2250 6050 50  0001 C CNN
 	1    2250 6050
@@
 F 0 "TP23" H 1950 6450 50  0000 C BNN
 F 1 "TEST" H 1950 6400 50  0000 C CNN
-F 2 "" H 1950 6150 50  0001 C CNN
+F 2 "Measurement_Points:Measurement_Point_Round-TH_Small" H 1950 6150 50  0001 C CNN
 F 3 "" H 1950 6150 50  0001 C CNN
 	1    1950 6150
@@
 F 0 "TP31" H 2250 6550 50  0000 C BNN
 F 1 "TEST" H 2250 6500 50  0000 C CNN
-F 2 "" H 2250 6250 50  0001 C CNN
+F 2 "Measurement_Points:Measurement_Point_Round-TH_Small" H 2250 6250 50  0001 C CNN
 F 3 "" H 2250 6250 50  0001 C CNN
 	1    2250 6250
@@
 F 0 "TP24" H 1950 6650 50  0000 C BNN
 F 1 "TEST" H 1950 6600 50  0000 C CNN
-F 2 "" H 1950 6350 50  0001 C CNN
+F 2 "Measurement_Points:Measurement_Point_Round-TH_Small" H 1950 6350 50  0001 C CNN
 F 3 "" H 1950 6350 50  0001 C CNN
 	1    1950 6350
@@
 F 0 "TP32" H 2250 6750 50  0000 C BNN
 F 1 "TEST" H 2250 6700 50  0000 C CNN
-F 2 "" H 2250 6450 50  0001 C CNN
+F 2 "Measurement_Points:Measurement_Point_Round-TH_Small" H 2250 6450 50  0001 C CNN
 F 3 "" H 2250 6450 50  0001 C CNN
 	1    2250 6450
@@
 F 0 "TP25" H 1950 6850 50  0000 C BNN
 F 1 "TEST" H 1950 6800 50  0000 C CNN
-F 2 "" H 1950 6550 50  0001 C CNN
+F 2 "Measurement_Points:Measurement_Point_Round-TH_Small" H 1950 6550 50  0001 C CNN
 F 3 "" H 1950 6550 50  0001 C CNN
 	1    1950 6550
@@
 F 0 "TP33" H 2250 6950 50  0000 C BNN
 F 1 "TEST" H 2250 6900 50  0000 C CNN
-F 2 "" H 2250 6650 50  0001 C CNN
+F 2 "Measurement_Points:Measurement_Point_Round-TH_Small" H 2250 6650 50  0001 C CNN
 F 3 "" H 2250 6650 50  0001 C CNN
 	1    2250 6650
@@
 F 0 "TP26" H 1950 7050 50  0000 C BNN
 F 1 "TEST" H 1950 7000 50  0000 C CNN
-F 2 "" H 1950 6750 50  0001 C CNN
+F 2 "Measurement_Points:Measurement_Point_Round-TH_Small" H 1950 6750 50  0001 C CNN
 F 3 "" H 1950 6750 50  0001 C CNN
 	1    1950 6750
@@
 F 0 "TP34" H 2250 7150 50  0000 C BNN
 F 1 "TEST" H 2250 7100 50  0000 C CNN
-F 2 "" H 2250 6850 50  0001 C CNN
+F 2 "Measurement_Points:Measurement_Point_Round-TH_Small" H 2250 6850 50  0001 C CNN
 F 3 "" H 2250 6850 50  0001 C CNN
 	1    2250 6850
@@
 F 0 "TP27" H 1950 7250 50  0000 C BNN
 F 1 "TEST" H 1950 7200 50  0000 C CNN
-F 2 "" H 1950 6950 50  0001 C CNN
+F 2 "Measurement_Points:Measurement_Point_Round-TH_Small" H 1950 6950 50  0001 C CNN
 F 3 "" H 1950 6950 50  0001 C CNN
 	1    1950 6950
@@
 F 0 "TP35" H 2250 7350 50  0000 C BNN
 F 1 "TEST" H 2250 7300 50  0000 C CNN
-F 2 "" H 2250 7050 50  0001 C CNN
+F 2 "Measurement_Points:Measurement_Point_Round-TH_Small" H 2250 7050 50  0001 C CNN
 F 3 "" H 2250 7050 50  0001 C CNN
 	1    2250 7050
@@
 F 0 "TP28" H 1950 7450 50  0000 C BNN
 F 1 "TEST" H 1950 7400 50  0000 C CNN
-F 2 "" H 1950 7150 50  0001 C CNN
+F 2 "Measurement_Points:Measurement_Point_Round-TH_Small" H 1950 7150 50  0001 C CNN
 F 3 "" H 1950 7150 50  0001 C CNN
 	1    1950 7150
@@
 F 0 "TP37" H 15550 4650 50  0000 C BNN
 F 1 "TEST" H 15550 4600 50  0000 C CNN
-F 2 "" H 15550 4350 50  0001 C CNN
+F 2 "Measurement_Points:Measurement_Point_Round-TH_Small" H 15550 4350 50  0001 C CNN
 F 3 "" H 15550 4350 50  0001 C CNN
 	1    15550 4350
@@
 F 0 "TP38" H 15550 4850 50  0000 C BNN
 F 1 "TEST" H 15550 4800 50  0000 C CNN
-F 2 "" H 15550 4550 50  0001 C CNN
+F 2 "Measurement_Points:Measurement_Point_Round-TH_Small" H 15550 4550 50  0001 C CNN
 F 3 "" H 15550 4550 50  0001 C CNN
 	1    15550 4550
@@
 F 0 "TP39" H 15550 5250 50  0000 C BNN
 F 1 "TEST" H 15550 5200 50  0000 C CNN
-F 2 "" H 15550 4950 50  0001 C CNN
+F 2 "Measurement_Points:Measurement_Point_Round-TH_Small" H 15550 4950 50  0001 C CNN
 F 3 "" H 15550 4950 50  0001 C CNN
 	1    15550 4950
@@
 F 0 "TP40" H 15550 5550 50  0000 C BNN
 F 1 "TEST" H 15550 5500 50  0000 C CNN
-F 2 "" H 15550 5250 50  0001 C CNN
+F 2 "Measurement_Points:Measurement_Point_Round-TH_Small" H 15550 5250 50  0001 C CNN
 F 3 "" H 15550 5250 50  0001 C CNN
 	1    15550 5250
@@
 F 0 "TP41" H 15550 6550 50  0000 C BNN
 F 1 "TEST" H 15550 6500 50  0000 C CNN
-F 2 "" H 15550 6250 50  0001 C CNN
+F 2 "Measurement_Points:Measurement_Point_Round-TH_Small" H 15550 6250 50  0001 C CNN
 F 3 "" H 15550 6250 50  0001 C CNN
 	1    15550 6250
@@
 F 0 "TP29" H 2200 3950 50  0000 C BNN
 F 1 "TEST" H 2200 3900 50  0000 C CNN
-F 2 "" H 2200 3650 50  0001 C CNN
+F 2 "Measurement_Points:Measurement_Point_Round-TH_Small" H 2200 3650 50  0001 C CNN
 F 3 "" H 2200 3650 50  0001 C CNN
 	1    2200 3650

Commit message: I think I found a way to have Panasonic interface
Uses 2 more optocouplers, 3 more diodes and some current limiting
resistors.
Parts:
- removed TP40, TP41: TEST, Measurement_Points:Measurement_Point_Round-TH_Small, symbol TEST
Connections:
- net labels added: PANAFOCUS, PANASHUTTER
Changed lines of the file:
@@
 EINK_PWR
 $Comp
-L power:Earth #PWR040
+L power:Earth #PWR042
 U 1 1 5A7F7482
 P 8800 3400
-F 0 "#PWR040" H 8800 3150 50  0001 C CNN
+F 0 "#PWR042" H 8800 3150 50  0001 C CNN
 F 1 "Earth" H 8800 3250 50  0001 C CNN
 F 2 "" H 8800 3400 50  0001 C CNN
@@
 $EndComp
 $Comp
-L power:VCC #PWR041
+L power:VCC #PWR043
 U 1 1 5A7F7645
 P 7850 3250
-F 0 "#PWR041" H 7850 3100 50  0001 C CNN
+F 0 "#PWR043" H 7850 3100 50  0001 C CNN
 F 1 "VCC" H 7850 3400 50  0000 C CNN
 F 2 "" H 7850 3250 50  0001 C CNN
@@
 $EndComp
 $Comp
-L power:Earth #PWR042
+L power:Earth #PWR044
 U 1 1 5A7F7940
 P 8400 7950
-F 0 "#PWR042" H 8400 7700 50  0001 C CNN
+F 0 "#PWR044" H 8400 7700 50  0001 C CNN
 F 1 "Earth" H 8400 7800 50  0001 C CNN
 F 2 "" H 8400 7950 50  0001 C CNN
@@
 $EndComp
 $Comp
-L power:Earth #PWR043
+L power:Earth #PWR045
 U 1 1 5A7F8695
 P 800 6400
-F 0 "#PWR043" H 800 6150 50  0001 C CNN
+F 0 "#PWR045" H 800 6150 50  0001 C CNN
 F 1 "Earth" H 800 6250 50  0001 C CNN
 F 2 "" H 800 6400 50  0001 C CNN
@@
 $EndComp
 $Comp
-L power:Earth #PWR044
+L power:Earth #PWR046
 U 1 1 5A7F869B
 P 1200 6400
-F 0 "#PWR044" H 1200 6150 50  0001 C CNN
+F 0 "#PWR046" H 1200 6150 50  0001 C CNN
 F 1 "Earth" H 1200 6250 50  0001 C CNN
 F 2 "" H 1200 6400 50  0001 C CNN
@@
 $EndComp
 $Comp
-L power:Earth #PWR045
+L power:Earth #PWR047
 U 1 1 5A7F8A34
 P 1500 8300
-F 0 "#PWR045" H 1500 8050 50  0001 C CNN
+F 0 "#PWR047" H 1500 8050 50  0001 C CNN
 F 1 "Earth" H 1500 8150 50  0001 C CNN
 F 2 "" H 1500 8300 50  0001 C CNN
@@
 $EndComp
 $Comp
-L power:Earth #PWR046
+L power:Earth #PWR048
 U 1 1 5A7F8A3A
 P 1900 8300
-F 0 "#PWR046" H 1900 8050 50  0001 C CNN
+F 0 "#PWR048" H 1900 8050 50  0001 C CNN
 F 1 "Earth" H 1900 8150 50  0001 C CNN
 F 2 "" H 1900 8300 50  0001 C CNN
@@
 $EndComp
 $Comp
-L power:Earth #PWR047
+L power:Earth #PWR049
 U 1 1 5A7F96B5
 P 1900 4050
-F 0 "#PWR047" H 1900 3800 50  0001 C CNN
+F 0 "#PWR049" H 1900 3800 50  0001 C CNN
 F 1 "Earth" H 1900 3900 50  0001 C CNN
 F 2 "" H 1900 4050 50  0001 C CNN
@@
 $EndComp
 $Comp
-L Earth #PWR048
+L Earth #PWR050
 U 1 1 5A7FA9BE
 P 1400 4200
-F 0 "#PWR048" H 1400 3950 50  0001 C CNN
+F 0 "#PWR050" H 1400 3950 50  0001 C CNN
 F 1 "Earth" H 1400 4050 50  0001 C CNN
 F 2 "" H 1400 4200 50  0001 C CNN
@@
 $EndComp
 $Comp
-L power:VCC #PWR049
+L power:VCC #PWR051
 U 1 1 5A7FAB49
 P 600 4150
-F 0 "#PWR049" H 600 4000 50  0001 C CNN
+F 0 "#PWR051" H 600 4000 50  0001 C CNN
 F 1 "VCC" H 600 4300 50  0000 C CNN
 F 2 "" H 600 4150 50  0001 C CNN
@@
 SWDIO
 $Comp
-L power:Earth #PWR050
+L power:Earth #PWR052
 U 1 1 5A7FC200
 P 1650 10100
-F 0 "#PWR050" H 1650 9850 50  0001 C CNN
+F 0 "#PWR052" H 1650 9850 50  0001 C CNN
 F 1 "Earth" H 1650 9950 50  0001 C CNN
 F 2 "" H 1650 10100 50  0001 C CNN
@@
 	3600 9950 3750 9950
 $Comp
-L power:Earth #PWR051
+L power:Earth #PWR053
 U 1 1 5A7FF0DB
 P 3900 10100
-F 0 "#PWR051" H 3900 9850 50  0001 C CNN
+F 0 "#PWR053" H 3900 9850 50  0001 C CNN
 F 1 "Earth" H 3900 9950 50  0001 C CNN
 F 2 "" H 3900 10100 50  0001 C CNN
@@
 	14750 6050 14550 6050
 $Comp
-L power:VCC #PWR052
+L power:VCC #PWR054
 U 1 1 5A8061D8
 P 2150 4550
-F 0 "#PWR052" H 2150 4400 50  0001 C CNN
+F 0 "#PWR054" H 2150 4400 50  0001 C CNN
 F 1 "VCC" H 2150 4700 50  0000 C CNN
 F 2 "" H 2150 4550 50  0001 C CNN
@@
 $EndComp
 $Comp
-L power:Earth #PWR053
+L power:Earth #PWR055
 U 1 1 5A806A82
 P 7850 3550
-F 0 "#PWR053" H 7850 3300 50  0001 C CNN
+F 0 "#PWR055" H 7850 3300 50  0001 C CNN
 F 1 "Earth" H 7850 3400 50  0001 C CNN
 F 2 "" H 7850 3550 50  0001 C CNN
@@
 Wire Wire Line
 	14550 7150 14750 7150
-Wire Wire Line
-	14550 6250 15550 6250
 Text HLabel 2350 8150 0    60   BiDi ~ 0
 SCL
@@
 	0    1    1    0
 $EndComp
-$Comp
-L TEST TP40
-U 1 1 5A84333F
-P 15550 5250
-F 0 "TP40" H 15550 5550 50  0000 C BNN
-F 1 "TEST" H 15550 5500 50  0000 C CNN
-F 2 "Measurement_Points:Measurement_Point_Round-TH_Small" H 15550 5250 50  0001 C CNN
-F 3 "" H 15550 5250 50  0001 C CNN
-	1    15550 5250
-	0    1    1    0
-$EndComp
-Wire Wire Line
-	14550 5350 14750 5350
-Wire Wire Line
-	14550 5250 15550 5250
 Wire Wire Line
 	14550 4950 15550 4950
@@
 Wire Wire Line
 	14550 4350 15550 4350
-Text HLabel 14750 5350 2    60   Input ~ 0
+Text HLabel 14750 6250 2    60   Input ~ 0
 Ambient
-$Comp
-L TEST TP41
-U 1 1 5A80E6EA
-P 15550 6250
-F 0 "TP41" H 15550 6550 50  0000 C BNN
-F 1 "TEST" H 15550 6500 50  0000 C CNN
-F 2 "Measurement_Points:Measurement_Point_Round-TH_Small" H 15550 6250 50  0001 C CNN
-F 3 "" H 15550 6250 50  0001 C CNN
-	1    15550 6250
-	0    1    1    0
-$EndComp
 $Comp
 L TEST TP29
@@
 	1    0    0    -1
 $EndComp
+Wire Wire Line
+	14550 6250 14750 6250
+Text HLabel 14750 5250 2    60   Output ~ 0
+PANASHUTTER
+Text HLabel 14750 5350 2    60   Output ~ 0
+PANAFOCUS
+Wire Wire Line
+	14550 5250 14750 5250
+Wire Wire Line
+	14550 5350 14750 5350
 $EndSCHEMATC
