File: pcb/soc.sch (KiCad schematic (older format))
At the start: 30 parts, among them J3 SWD, J4 UART, U1 STM32L476RETx, Y1 32 Mhz, Y2 32 Mhz

Commit message: Reassigned some footprints, added some libraries
Normally I can start working on PCB.
Parts:
- C35, C36, C37, C38, C39, C40: footprint Capacitors_SMD:C_1210 -> Capacitors_SMD:C_1206
- J3: footprint Pin_Headers:Pin_Header_Angled_1x06_Pitch2.54mm -> Pin_Headers:Pin_Header_Straight_1x06_Pitch2.54mm
- J4, JP3: footprint Pin_Headers:Pin_Header_Angled_1x03_Pitch2.54mm -> Pin_Headers:Pin_Header_Straight_1x03_Pitch2.54mm
- R27: footprint Resistors_SMD:R_1210 -> Resistors_SMD:R_1206
Changed lines of the file:
@@
 LIBS:EL817S
 LIBS:IRA-S210ST01
+LIBS:RE1C002UNTCL
+LIBS:SJ-2523-SMT-TR
 LIBS:pir-cache
 EELAYER 25 0
@@
 EINK_PWR
 $Comp
-L power:Earth #PWR042
+L power:Earth #PWR043
 U 1 1 5A7F7482
 P 8800 3400
-F 0 "#PWR042" H 8800 3150 50  0001 C CNN
+F 0 "#PWR043" H 8800 3150 50  0001 C CNN
 F 1 "Earth" H 8800 3250 50  0001 C CNN
 F 2 "" H 8800 3400 50  0001 C CNN
@@
 $EndComp
 $Comp
-L power:VCC #PWR043
+L power:VCC #PWR044
 U 1 1 5A7F7645
 P 7850 3250
-F 0 "#PWR043" H 7850 3100 50  0001 C CNN
+F 0 "#PWR044" H 7850 3100 50  0001 C CNN
 F 1 "VCC" H 7850 3400 50  0000 C CNN
 F 2 "" H 7850 3250 50  0001 C CNN
@@
 $EndComp
 $Comp
-L power:Earth #PWR044
+L power:Earth #PWR045
 U 1 1 5A7F7940
 P 8400 7950
-F 0 "#PWR044" H 8400 7700 50  0001 C CNN
+F 0 "#PWR045" H 8400 7700 50  0001 C CNN
 F 1 "Earth" H 8400 7800 50  0001 C CNN
 F 2 "" H 8400 7950 50  0001 C CNN
@@
 F 0 "C35" H 810 6270 50  0000 L CNN
 F 1 "12pF" H 810 6120 50  0000 L CNN
-F 2 "Capacitors_SMD:C_1210" H 800 6200 50  0001 C CNN
+F 2 "Capacitors_SMD:C_1206" H 800 6200 50  0001 C CNN
 F 3 "" H 800 6200 50  0001 C CNN
 	1    800  6200
@@
 F 0 "C36" H 1210 6270 50  0000 L CNN
 F 1 "12pF" H 1210 6120 50  0000 L CNN
-F 2 "Capacitors_SMD:C_1210" H 1200 6200 50  0001 C CNN
+F 2 "Capacitors_SMD:C_1206" H 1200 6200 50  0001 C CNN
 F 3 "" H 1200 6200 50  0001 C CNN
 	1    1200 6200
@@
 $EndComp
 $Comp
-L power:Earth #PWR045
+L power:Earth #PWR046
 U 1 1 5A7F8695
 P 800 6400
-F 0 "#PWR045" H 800 6150 50  0001 C CNN
+F 0 "#PWR046" H 800 6150 50  0001 C CNN
 F 1 "Earth" H 800 6250 50  0001 C CNN
 F 2 "" H 800 6400 50  0001 C CNN
@@
 $EndComp
 $Comp
-L power:Earth #PWR046
+L power:Earth #PWR047
 U 1 1 5A7F869B
 P 1200 6400
-F 0 "#PWR046" H 1200 6150 50  0001 C CNN
+F 0 "#PWR047" H 1200 6150 50  0001 C CNN
 F 1 "Earth" H 1200 6250 50  0001 C CNN
 F 2 "" H 1200 6400 50  0001 C CNN
@@
 F 0 "C37" H 1510 8170 50  0000 L CNN
 F 1 "12pF" H 1510 8020 50  0000 L CNN
-F 2 "Capacitors_SMD:C_1210" H 1500 8100 50  0001 C CNN
+F 2 "Capacitors_SMD:C_1206" H 1500 8100 50  0001 C CNN
 F 3 "" H 1500 8100 50  0001 C CNN
 	1    1500 8100
@@
 F 0 "C39" H 1910 8170 50  0000 L CNN
 F 1 "12pF" H 1910 8020 50  0000 L CNN
-F 2 "Capacitors_SMD:C_1210" H 1900 8100 50  0001 C CNN
+F 2 "Capacitors_SMD:C_1206" H 1900 8100 50  0001 C CNN
 F 3 "" H 1900 8100 50  0001 C CNN
 	1    1900 8100
@@
 $EndComp
 $Comp
-L power:Earth #PWR047
+L power:Earth #PWR048
 U 1 1 5A7F8A34
 P 1500 8300
-F 0 "#PWR047" H 1500 8050 50  0001 C CNN
+F 0 "#PWR048" H 1500 8050 50  0001 C CNN
 F 1 "Earth" H 1500 8150 50  0001 C CNN
 F 2 "" H 1500 8300 50  0001 C CNN
@@
 $EndComp
 $Comp
-L power:Earth #PWR048
+L power:Earth #PWR049
 U 1 1 5A7F8A3A
 P 1900 8300
-F 0 "#PWR048" H 1900 8050 50  0001 C CNN
+F 0 "#PWR049" H 1900 8050 50  0001 C CNN
 F 1 "Earth" H 1900 8150 50  0001 C CNN
 F 2 "" H 1900 8300 50  0001 C CNN
@@
 F 0 "R27" V 1580 3650 50  0000 C CNN
 F 1 "1K" V 1500 3650 50  0000 C CNN
-F 2 "Resistors_SMD:R_1210" V 1430 3650 50  0001 C CNN
+F 2 "Resistors_SMD:R_1206" V 1430 3650 50  0001 C CNN
 F 3 "" H 1500 3650 50  0001 C CNN
 	1    1500 3650
@@
 F 0 "C38" H 1910 3870 50  0000 L CNN
 F 1 "100nF" H 1910 3720 50  0000 L CNN
-F 2 "Capacitors_SMD:C_1210" H 1900 3800 50  0001 C CNN
+F 2 "Capacitors_SMD:C_1206" H 1900 3800 50  0001 C CNN
 F 3 "" H 1900 3800 50  0001 C CNN
 	1    1900 3800
@@
 $EndComp
 $Comp
-L power:Earth #PWR049
+L power:Earth #PWR050
 U 1 1 5A7F96B5
 P 1900 4050
-F 0 "#PWR049" H 1900 3800 50  0001 C CNN
+F 0 "#PWR050" H 1900 3800 50  0001 C CNN
 F 1 "Earth" H 1900 3900 50  0001 C CNN
 F 2 "" H 1900 4050 50  0001 C CNN
@@
 F 0 "JP3" H 1100 4050 50  0000 L CNN
 F 1 "Jumper_NC_Dual" H 1050 4250 50  0000 C BNN
-F 2 "Pin_Headers:Pin_Header_Angled_1x03_Pitch2.54mm" H 1050 4150 50  0001 C CNN
+F 2 "Pin_Headers:Pin_Header_Straight_1x03_Pitch2.54mm" H 1050 4150 50  0001 C CNN
 F 3 "" H 1050 4150 50  0001 C CNN
 	1    1050 4150
@@
 $EndComp
 $Comp
-L Earth #PWR050
+L Earth #PWR051
 U 1 1 5A7FA9BE
 P 1400 4200
-F 0 "#PWR050" H 1400 3950 50  0001 C CNN
+F 0 "#PWR051" H 1400 3950 50  0001 C CNN
 F 1 "Earth" H 1400 4050 50  0001 C CNN
 F 2 "" H 1400 4200 50  0001 C CNN
@@
 $EndComp
 $Comp
-L power:VCC #PWR051
+L power:VCC #PWR052
 U 1 1 5A7FAB49
 P 600 4150
-F 0 "#PWR051" H 600 4000 50  0001 C CNN
+F 0 "#PWR052" H 600 4000 50  0001 C CNN
 F 1 "VCC" H 600 4300 50  0000 C CNN
 F 2 "" H 600 4150 50  0001 C CNN
@@
 SWDIO
 $Comp
-L power:Earth #PWR052
+L power:Earth #PWR053
 U 1 1 5A7FC200
 P 1650 10100
-F 0 "#PWR052" H 1650 9850 50  0001 C CNN
+F 0 "#PWR053" H 1650 9850 50  0001 C CNN
 F 1 "Earth" H 1650 9950 50  0001 C CNN
 F 2 "" H 1650 10100 50  0001 C CNN
@@
 F 0 "J3" H 1450 10400 50  0000 C CNN
 F 1 "SWD" H 1450 9700 50  0000 C CNN
-F 2 "Pin_Headers:Pin_Header_Angled_1x06_Pitch2.54mm" H 1450 10100 50  0001 C CNN
+F 2 "Pin_Headers:Pin_Header_Straight_1x06_Pitch2.54mm" H 1450 10100 50  0001 C CNN
 F 3 "" H 1450 10100 50  0001 C CNN
 	1    1450 10100
@@
 F 0 "J4" H 3400 10150 50  0000 C CNN
 F 1 "UART" H 3400 9750 50  0000 C CNN
-F 2 "Pin_Headers:Pin_Header_Angled_1x03_Pitch2.54mm" H 3400 9950 50  0001 C CNN
+F 2 "Pin_Headers:Pin_Header_Straight_1x03_Pitch2.54mm" H 3400 9950 50  0001 C CNN
 F 3 "" H 3400 9950 50  0001 C CNN
 	1    3400 9950
@@
 	3600 9950 3750 9950
 $Comp
-L power:Earth #PWR053
+L power:Earth #PWR054
 U 1 1 5A7FF0DB
 P 3900 10100
-F 0 "#PWR053" H 3900 9850 50  0001 C CNN
+F 0 "#PWR054" H 3900 9850 50  0001 C CNN
 F 1 "Earth" H 3900 9950 50  0001 C CNN
 F 2 "" H 3900 10100 50  0001 C CNN
@@
 	14750 6050 14550 6050
 $Comp
-L power:VCC #PWR054
+L power:VCC #PWR055
 U 1 1 5A8061D8
 P 2150 4550
-F 0 "#PWR054" H 2150 4400 50  0001 C CNN
+F 0 "#PWR055" H 2150 4400 50  0001 C CNN
 F 1 "VCC" H 2150 4700 50  0000 C CNN
 F 2 "" H 2150 4550 50  0001 C CNN
@@
 F 0 "C40" H 7860 3520 50  0000 L CNN
 F 1 "100nF" H 7860 3370 50  0000 L CNN
-F 2 "Capacitors_SMD:C_1210" H 7850 3450 50  0001 C CNN
+F 2 "Capacitors_SMD:C_1206" H 7850 3450 50  0001 C CNN
 F 3 "" H 7850 3450 50  0001 C CNN
 	1    7850 3450
@@
 $EndComp
 $Comp
-L power:Earth #PWR055
+L power:Earth #PWR056
 U 1 1 5A806A82
 P 7850 3550
-F 0 "#PWR055" H 7850 3300 50  0001 C CNN
+F 0 "#PWR056" H 7850 3300 50  0001 C CNN
 F 1 "Earth" H 7850 3400 50  0001 C CNN
 F 2 "" H 7850 3550 50  0001 C CNN

Commit message: Started placing some components, finally
Parts:
- removed TP28, TP35: TEST, Measurement_Points:Measurement_Point_Round-TH_Small, symbol TEST
Changed lines of the file:
@@
 Text HLabel 14750 4650 2    50   Output ~ 0
 EINK_SCK
-Text HLabel 14750 6350 2    50   Output ~ 0
+Text HLabel 14750 6250 2    50   Output ~ 0
 EINK_MOSI
 Text HLabel 14750 5650 2    50   Output ~ 0
@@
 Text HLabel 14750 7350 2    50   Output ~ 0
 EINK_RST
-Text HLabel 14750 7050 2    50   Input ~ 0
+Text HLabel 1400 7050 0    50   Input ~ 0
 EINK_D/C
 Text HLabel 14750 7150 2    50   Input ~ 0
 EINK_BS
-Text HLabel 14750 6450 2    50   Output ~ 0
+Text HLabel 1700 7150 0    50   Output ~ 0
 EINK_PWR
 $Comp
@@
 Wire Wire Line
 	14550 5450 15100 5450
-Text HLabel 14750 6550 2    60   Input ~ 0
+Text HLabel 14750 6650 2    60   Input ~ 0
 Left
-Text HLabel 14750 6650 2    60   Input ~ 0
+Text HLabel 14750 6750 2    60   Input ~ 0
 Right
-Text HLabel 14750 6750 2    60   Input ~ 0
+Text HLabel 14750 6850 2    60   Input ~ 0
 Up
-Text HLabel 14750 6850 2    60   Input ~ 0
+Text HLabel 14750 6950 2    60   Input ~ 0
 Down
-Text HLabel 14750 6950 2    60   Input ~ 0
+Text HLabel 14750 7050 2    60   Input ~ 0
 OK
 Wire Wire Line
@@
 	0    -1   -1   0
 $EndComp
-$Comp
-L TEST TP35
-U 1 1 5A841D8F
-P 2250 7050
-F 0 "TP35" H 2250 7350 50  0000 C BNN
-F 1 "TEST" H 2250 7300 50  0000 C CNN
-F 2 "Measurement_Points:Measurement_Point_Round-TH_Small" H 2250 7050 50  0001 C CNN
-F 3 "" H 2250 7050 50  0001 C CNN
-	1    2250 7050
-	0    -1   -1   0
-$EndComp
-$Comp
-L TEST TP28
-U 1 1 5A841DFE
-P 1950 7150
-F 0 "TP28" H 1950 7450 50  0000 C BNN
-F 1 "TEST" H 1950 7400 50  0000 C CNN
-F 2 "Measurement_Points:Measurement_Point_Round-TH_Small" H 1950 7150 50  0001 C CNN
-F 3 "" H 1950 7150 50  0001 C CNN
-	1    1950 7150
-	0    -1   -1   0
-$EndComp
 Wire Wire Line
 	2250 6050 2350 6050
@@
 	1950 6950 2350 6950
 Wire Wire Line
-	2250 7050 2350 7050
-Wire Wire Line
-	1950 7150 2350 7150
+	1400 7050 2350 7050
+Wire Wire Line
+	1700 7150 2350 7150
 $Comp
 L TEST TP37
@@
 Wire Wire Line
 	14550 4350 15550 4350
-Text HLabel 14750 6250 2    60   Input ~ 0
+Text HLabel 14750 6350 2    60   Input ~ 0
 Ambient
 $Comp
@@
 Wire Wire Line
 	14550 5350 14750 5350
+Text HLabel 14750 6550 2    60   Input ~ 0
+SDA
+Text HLabel 14750 6450 2    60   Input ~ 0
+SCL
 $EndSCHEMATC

Commit message: More work on the PCB
The opamp circuit is done.
Currently working on camera interface.
TODO: screen, buttons.
Changed lines of the file:
@@
 LIBS:xilinx
 LIBS:zetex
-LIBS:SparkFun
-LIBS:ab2_7segment
-LIBS:ab2_audio
-LIBS:ab2_buffer
-LIBS:ab2_capacitor
-LIBS:ab2_connectivity
-LIBS:ab2_dac
-LIBS:ab2_diode
-LIBS:ab2_fuse
-LIBS:ab2_gpio_expansion
-LIBS:ab2_header
-LIBS:ab2_idc
-LIBS:ab2_inductor
-LIBS:ab2_input_devices
-LIBS:ab2_jumper
-LIBS:ab2_lcd
-LIBS:ab2_led
-LIBS:ab2_memory
-LIBS:ab2_opamp
-LIBS:ab2_pinouts
-LIBS:ab2_pot
-LIBS:ab2_power
-LIBS:ab2_regulator
-LIBS:ab2_relay
-LIBS:ab2_resistor
-LIBS:ab2_sensor
-LIBS:ab2_stepper
-LIBS:ab2_supply
-LIBS:ab2_terminal_block
-LIBS:ab2_test
-LIBS:ab2_transistor
-LIBS:ab2_uC
-LIBS:ab2_usb
-LIBS:ab2_xtal
 LIBS:EL817S
 LIBS:IRA-S210ST01
@@
 Text HLabel 14750 4650 2    50   Output ~ 0
 EINK_SCK
-Text HLabel 14750 6250 2    50   Output ~ 0
+Text HLabel 14750 6350 2    50   Output ~ 0
 EINK_MOSI
 Text HLabel 14750 5650 2    50   Output ~ 0
@@
 Wire Wire Line
 	14550 4350 15550 4350
-Text HLabel 14750 6350 2    60   Input ~ 0
+Text HLabel 14750 6250 2    60   Input ~ 0
 Ambient
 $Comp

Commit message: Finished the display components placement.
Connections:
- wire segments 98 -> 97
Other:
- moved on the sheet: TP25, TP26, TP32, TP33, TP34, TP39
Changed lines of the file:
@@
 LIBS:xilinx
 LIBS:zetex
+LIBS:SparkFun
+LIBS:ab2_7segment
+LIBS:ab2_audio
+LIBS:ab2_buffer
+LIBS:ab2_capacitor
+LIBS:ab2_connectivity
+LIBS:ab2_dac
+LIBS:ab2_diode
+LIBS:ab2_fuse
+LIBS:ab2_gpio_expansion
+LIBS:ab2_header
+LIBS:ab2_idc
+LIBS:ab2_inductor
+LIBS:ab2_input_devices
+LIBS:ab2_jumper
+LIBS:ab2_lcd
+LIBS:ab2_led
+LIBS:ab2_memory
+LIBS:ab2_opamp
+LIBS:ab2_pinouts
+LIBS:ab2_pot
+LIBS:ab2_power
+LIBS:ab2_regulator
+LIBS:ab2_relay
+LIBS:ab2_resistor
+LIBS:ab2_sensor
+LIBS:ab2_stepper
+LIBS:ab2_supply
+LIBS:ab2_terminal_block
+LIBS:ab2_test
+LIBS:ab2_transistor
+LIBS:ab2_uC
+LIBS:ab2_usb
+LIBS:ab2_xtal
 LIBS:EL817S
 LIBS:IRA-S210ST01
@@
 	2350 4150 2200 4150
 Wire Wire Line
-	2200 4150 2200 3650
-Wire Wire Line
-	2200 3650 1650 3650
+	2200 3650 2200 4150
+Wire Wire Line
+	1650 3650 2200 3650
 Wire Wire Line
 	1900 3650 1900 3700
@@
 	1    0    0    -1
 $EndComp
-Text GLabel 3950 9850 2    60   Input ~ 0
+Text GLabel 3900 10050 2    60   Input ~ 0
 TX
 Text GLabel 3750 9950 2    60   Input ~ 0
@@
 L power:Earth #PWR054
 U 1 1 5A7FF0DB
-P 3900 10100
-F 0 "#PWR054" H 3900 9850 50  0001 C CNN
-F 1 "Earth" H 3900 9950 50  0001 C CNN
-F 2 "" H 3900 10100 50  0001 C CNN
-F 3 "" H 3900 10100 50  0001 C CNN
-	1    3900 10100
-	1    0    0    -1
-$EndComp
-Wire Wire Line
-	3900 10100 3900 10050
+P 3950 9850
+F 0 "#PWR054" H 3950 9600 50  0001 C CNN
+F 1 "Earth" H 3950 9700 50  0001 C CNN
+F 2 "" H 3950 9850 50  0001 C CNN
+F 3 "" H 3950 9850 50  0001 C CNN
+	1    3950 9850
+	0    -1   -1   0
+$EndComp
 Wire Wire Line
 	3900 10050 3600 10050
@@
 	14750 7250 14550 7250
 Wire Wire Line
-	14550 7050 14750 7050
+	14550 7050 15000 7050
 Wire Wire Line
 	14550 7150 14750 7150
@@
 Wire Wire Line
 	14550 5450 15100 5450
-Text HLabel 14750 6650 2    60   Input ~ 0
+Text HLabel 2150 6750 0    60   Input ~ 0
 Left
-Text HLabel 14750 6750 2    60   Input ~ 0
+Text HLabel 2150 6550 0    60   Input ~ 0
 Right
-Text HLabel 14750 6850 2    60   Input ~ 0
+Text HLabel 15550 4950 2    60   Input ~ 0
 Up
-Text HLabel 14750 6950 2    60   Input ~ 0
+Text HLabel 2150 6450 0    60   Input ~ 0
 Down
-Text HLabel 14750 7050 2    60   Input ~ 0
+Text HLabel 2150 6650 0    60   Input ~ 0
 OK
 Wire Wire Line
 	14550 6550 14750 6550
 Wire Wire Line
-	14550 6650 14750 6650
-Wire Wire Line
-	14550 6750 14750 6750
-Wire Wire Line
-	14550 6850 14750 6850
-Wire Wire Line
-	14550 6950 14750 6950
+	14550 6650 15000 6650
+Wire Wire Line
+	14550 6750 15400 6750
+Wire Wire Line
+	14550 6850 15000 6850
+Wire Wire Line
+	14550 6950 15400 6950
 Text HLabel 14750 4150 2    60   Input ~ 0
 OPAMP1+
@@
 L TEST TP32
 U 1 1 5A841B2C
-P 2250 6450
-F 0 "TP32" H 2250 6750 50  0000 C BNN
-F 1 "TEST" H 2250 6700 50  0000 C CNN
-F 2 "Measurement_Points:Measurement_Point_Round-TH_Small" H 2250 6450 50  0001 C CNN
-F 3 "" H 2250 6450 50  0001 C CNN
-	1    2250 6450
-	0    -1   -1   0
+P 15400 6750
+F 0 "TP32" H 15400 7050 50  0000 C BNN
+F 1 "TEST" H 15400 7000 50  0000 C CNN
+F 2 "Measurement_Points:Measurement_Point_Round-TH_Small" H 15400 6750 50  0001 C CNN
+F 3 "" H 15400 6750 50  0001 C CNN
+	1    15400 6750
+	0    1    1    0
 $EndComp
 $Comp
 L TEST TP25
 U 1 1 5A841B81
-P 1950 6550
-F 0 "TP25" H 1950 6850 50  0000 C BNN
-F 1 "TEST" H 1950 6800 50  0000 C CNN
-F 2 "Measurement_Points:Measurement_Point_Round-TH_Small" H 1950 6550 50  0001 C CNN
-F 3 "" H 1950 6550 50  0001 C CNN
-	1    1950 6550
-	0    -1   -1   0
+P 15000 6650
+F 0 "TP25" H 15000 6950 50  0000 C BNN
+F 1 "TEST" H 15000 6900 50  0000 C CNN
+F 2 "Measurement_Points:Measurement_Point_Round-TH_Small" H 15000 6650 50  0001 C CNN
+F 3 "" H 15000 6650 50  0001 C CNN
+	1    15000 6650
+	0    1    1    0
 $EndComp
 $Comp
 L TEST TP33
 U 1 1 5A841BED
-P 2250 6650
-F 0 "TP33" H 2250 6950 50  0000 C BNN
-F 1 "TEST" H 2250 6900 50  0000 C CNN
-F 2 "Measurement_Points:Measurement_Point_Round-TH_Small" H 2250 6650 50  0001 C CNN
-F 3 "" H 2250 6650 50  0001 C CNN
-	1    2250 6650
-	0    -1   -1   0
+P 15400 6950
+F 0 "TP33" H 15400 7250 50  0000 C BNN
+F 1 "TEST" H 15400 7200 50  0000 C CNN
+F 2 "Measurement_Points:Measurement_Point_Round-TH_Small" H 15400 6950 50  0001 C CNN
+F 3 "" H 15400 6950 50  0001 C CNN
+	1    15400 6950
+	0    1    1    0
 $EndComp
 $Comp
 L TEST TP26
 U 1 1 5A841C4E
-P 1950 6750
-F 0 "TP26" H 1950 7050 50  0000 C BNN
-F 1 "TEST" H 1950 7000 50  0000 C CNN
-F 2 "Measurement_Points:Measurement_Point_Round-TH_Small" H 1950 6750 50  0001 C CNN
-F 3 "" H 1950 6750 50  0001 C CNN
-	1    1950 6750
-	0    -1   -1   0
+P 15000 7050
+F 0 "TP26" H 15000 7350 50  0000 C BNN
+F 1 "TEST" H 15000 7300 50  0000 C CNN
+F 2 "Measurement_Points:Measurement_Point_Round-TH_Small" H 15000 7050 50  0001 C CNN
+F 3 "" H 15000 7050 50  0001 C CNN
+	1    15000 7050
+	0    1    1    0
 $EndComp
 $Comp
 L TEST TP34
 U 1 1 5A841CC0
-P 2250 6850
-F 0 "TP34" H 2250 7150 50  0000 C BNN
-F 1 "TEST" H 2250 7100 50  0000 C CNN
-F 2 "Measurement_Points:Measurement_Point_Round-TH_Small" H 2250 6850 50  0001 C CNN
-F 3 "" H 2250 6850 50  0001 C CNN
-	1    2250 6850
+P 1600 6850
+F 0 "TP34" H 1600 7150 50  0000 C BNN
+F 1 "TEST" H 1600 7100 50  0000 C CNN
+F 2 "Measurement_Points:Measurement_Point_Round-TH_Small" H 1600 6850 50  0001 C CNN
+F 3 "" H 1600 6850 50  0001 C CNN
+	1    1600 6850
 	0    -1   -1   0
 $EndComp
@@
 	1950 6350 2350 6350
 Wire Wire Line
-	2350 6450 2250 6450
-Wire Wire Line
-	1950 6550 2350 6550
-Wire Wire Line
-	2250 6650 2350 6650
-Wire Wire Line
-	1950 6750 2350 6750
-Wire Wire Line
-	2250 6850 2350 6850
+	2350 6450 2150 6450
+Wire Wire Line
+	2150 6550 2350 6550
+Wire Wire Line
+	2150 6650 2350 6650
+Wire Wire Line
+	2150 6750 2350 6750
+Wire Wire Line
+	1600 6850 2350 6850
 Wire Wire Line
 	1950 6950 2350 6950
@@
 L TEST TP39
 U 1 1 5A843254
-P 15550 4950
-F 0 "TP39" H 15550 5250 50  0000 C BNN
-F 1 "TEST" H 15550 5200 50  0000 C CNN
-F 2 "Measurement_Points:Measurement_Point_Round-TH_Small" H 15550 4950 50  0001 C CNN
-F 3 "" H 15550 4950 50  0001 C CNN
-	1    15550 4950
+P 15000 6850
+F 0 "TP39" H 15000 7150 50  0000 C BNN
+F 1 "TEST" H 15000 7100 50  0000 C CNN
+F 2 "Measurement_Points:Measurement_Point_Round-TH_Small" H 15000 6850 50  0001 C CNN
+F 3 "" H 15000 6850 50  0001 C CNN
+	1    15000 6850
 	0    1    1    0
 $EndComp
