File: pcb/battery.sch (KiCad schematic (older format))
At the start: 8 parts, among them Q1 SI2323DS

Commit message: User pushbutton
Parts:
- removed Q1: SI2323DS, symbol Q_PMOS_GSD
- added D3: D_Schottky, symbol D_Schottky
- added IC6: SI2323DS-T1-E3, SOT95P237X112-3N, symbol SI2323DS-T1-E3
- added JP2: Jumper, symbol Jumper
- added R3: 100K, symbol R
Connections:
- net labels added: CC3V3
- wire segments 17 -> 24
Other:
- note added: "Battery & Debugger power switch & Reservoir Capacitors"
- note removed: "Battery connector & Reservoir Capacitors"

Commit message: Added light sensor with IIC interface
Parts:
- renumbered C1 to C15, C2 to C16, C3 to C17, C4 to C18, C5 to C19, JP2 to JP1, JP1 to JP2, R3 to R1
Changed lines of the file:
@@
 LIBS:CC2541F256RHAR
 LIBS:CC2541F128RHAT
+LIBS:MAX44009EDT+T
 LIBS:pir-cache
 EELAYER 25 0
@@
 $EndComp
 $Comp
-L Earth #PWR15
+L Earth #PWR18
 U 1 1 5A76A190
 P 7450 4350
-F 0 "#PWR15" H 7450 4100 50  0001 C CNN
+F 0 "#PWR18" H 7450 4100 50  0001 C CNN
 F 1 "Earth" H 7450 4200 50  0001 C CNN
 F 2 "" H 7450 4350 50  0001 C CNN
@@
 $EndComp
 $Comp
-L Jumper JP1
+L Jumper JP2
 U 1 1 5A76A19D
 P 4200 3450
-F 0 "JP1" H 4200 3600 50  0000 C CNN
+F 0 "JP2" H 4200 3600 50  0000 C CNN
 F 1 "Jumper" H 4200 3370 50  0000 C CNN
 F 2 "" H 4200 3450 50  0001 C CNN
@@
 $EndComp
 $Comp
-L C C1
+L C C15
 U 1 1 5A76A1A4
 P 6750 3600
-F 0 "C1" H 6775 3700 50  0000 L CNN
+F 0 "C15" H 6775 3700 50  0000 L CNN
 F 1 "100μF" H 6775 3500 50  0000 L CNN
 F 2 "" H 6788 3450 50  0001 C CNN
@@
 $EndComp
 $Comp
-L C C2
+L C C16
 U 1 1 5A76A1AB
 P 7100 3600
-F 0 "C2" H 7125 3700 50  0000 L CNN
+F 0 "C16" H 7125 3700 50  0000 L CNN
 F 1 "10μF" H 7125 3500 50  0000 L CNN
 F 2 "" H 7138 3450 50  0001 C CNN
@@
 $EndComp
 $Comp
-L C C3
+L C C17
 U 1 1 5A76A1B2
 P 7450 3600
-F 0 "C3" H 7475 3700 50  0000 L CNN
+F 0 "C17" H 7475 3700 50  0000 L CNN
 F 1 "1μF" H 7475 3500 50  0000 L CNN
 F 2 "" H 7488 3450 50  0001 C CNN
@@
 $EndComp
 $Comp
-L C C4
+L C C18
 U 1 1 5A76A1B9
 P 7750 3600
-F 0 "C4" H 7775 3700 50  0000 L CNN
+F 0 "C18" H 7775 3700 50  0000 L CNN
 F 1 "0.1μF" H 7775 3500 50  0000 L CNN
 F 2 "" H 7788 3450 50  0001 C CNN
@@
 $EndComp
 $Comp
-L C C5
+L C C19
 U 1 1 5A76A1C0
 P 8050 3600
-F 0 "C5" H 8075 3700 50  0000 L CNN
+F 0 "C19" H 8075 3700 50  0000 L CNN
 F 1 "0.01μF" H 8075 3500 50  0000 L CNN
 F 2 "" H 8088 3450 50  0001 C CNN
@@
 	4750 3450 4500 3450
 $Comp
-L R R3
+L R R1
 U 1 1 5A768BF5
 P 3100 3850
-F 0 "R3" V 3180 3850 50  0000 C CNN
+F 0 "R1" V 3180 3850 50  0000 C CNN
 F 1 "100K" V 3100 3850 50  0000 C CNN
 F 2 "" V 3030 3850 50  0001 C CNN
@@
 $EndComp
 $Comp
-L Earth #PWR13
+L Earth #PWR16
 U 1 1 5A768D52
 P 3800 4250
-F 0 "#PWR13" H 3800 4000 50  0001 C CNN
+F 0 "#PWR16" H 3800 4000 50  0001 C CNN
 F 1 "Earth" H 3800 4100 50  0001 C CNN
 F 2 "" H 3800 4250 50  0001 C CNN
@@
 $EndComp
 $Comp
-L Earth #PWR12
+L Earth #PWR15
 U 1 1 5A768DD5
 P 3100 4250
-F 0 "#PWR12" H 3100 4000 50  0001 C CNN
+F 0 "#PWR15" H 3100 4000 50  0001 C CNN
 F 1 "Earth" H 3100 4100 50  0001 C CNN
 F 2 "" H 3100 4250 50  0001 C CNN
@@
 	5700 2900 5700 3350
 $Comp
-L Jumper JP2
+L Jumper JP1
 U 1 1 5A769069
 P 3800 2900
-F 0 "JP2" H 3800 3050 50  0000 C CNN
+F 0 "JP1" H 3800 3050 50  0000 C CNN
 F 1 "Jumper" H 3800 2820 50  0000 C CNN
 F 2 "" H 3800 2900 50  0001 C CNN
@@
 Connection ~ 7100 4150
 $Comp
-L VCC #PWR14
+L VCC #PWR17
 U 1 1 5A769C0A
 P 7450 2950
-F 0 "#PWR14" H 7450 2800 50  0001 C CNN
+F 0 "#PWR17" H 7450 2800 50  0001 C CNN
 F 1 "VCC" H 7450 3100 50  0000 C CNN
 F 2 "" H 7450 2950 50  0001 C CNN

Commit message: Migrated project/libraries to KiCad nightly build
Revision: 821668d96

Reason being the simulator feature and the better library management.
Parts:
- added V?: VSOURCE, symbol pspice:VSOURCE
- BT1: symbol Battery_Cell -> device:Battery_Cell
- C15, C16, C17, C18, C19: symbol C -> device:C
- D3: symbol D_Schottky -> device:D_Schottky
- IC6: symbol SI2323DS-T1-E3 -> SI2323DS-T1-E3:SI2323DS-T1-E3
- JP1, JP2: symbol Jumper -> device:Jumper
- R1: symbol R -> device:R
Connections:
- wire segments 24 -> 36
Changed lines of the file:
@@
-EESchema Schematic File Version 2
-LIBS:power
-LIBS:device
-LIBS:switches
-LIBS:relays
-LIBS:motors
-LIBS:transistors
-LIBS:conn
-LIBS:linear
-LIBS:regul
-LIBS:74xx
-LIBS:cmos4000
-LIBS:adc-dac
-LIBS:memory
-LIBS:xilinx
-LIBS:microcontrollers
-LIBS:dsp
-LIBS:microchip
-LIBS:analog_switches
-LIBS:motorola
-LIBS:texas
-LIBS:intel
-LIBS:audio
-LIBS:interface
-LIBS:digital-audio
-LIBS:philips
-LIBS:display
-LIBS:cypress
-LIBS:siliconi
-LIBS:opto
-LIBS:atmel
-LIBS:contrib
-LIBS:valves
-LIBS:LPV802DGKT
-LIBS:SI2323DS-T1-E3
-LIBS:1N4148X-TP
-LIBS:TLV3691IDCKR
-LIBS:IRA-S210ST01
-LIBS:CC2540F256RHAT
-LIBS:CC2541F256RHAR
-LIBS:CC2541F128RHAT
-LIBS:MAX44009EDT+T
+EESchema Schematic File Version 4
 LIBS:pir-cache
-EELAYER 25 0
+EELAYER 26 0
 EELAYER END
 $Descr A4 11693 8268
@@
 $EndDescr
 $Comp
-L Battery_Cell BT1
+L device:Battery_Cell BT1
 U 1 1 5A76A189
 P 3800 4000
@@
 $EndComp
 $Comp
-L Earth #PWR18
+L power:Earth #PWR18
 U 1 1 5A76A190
 P 7450 4350
@@
 $EndComp
 $Comp
-L Jumper JP2
+L device:Jumper JP2
 U 1 1 5A76A19D
 P 4200 3450
@@
 $EndComp
 $Comp
-L C C15
+L device:C C15
 U 1 1 5A76A1A4
 P 6750 3600
@@
 $EndComp
 $Comp
-L C C16
+L device:C C16
 U 1 1 5A76A1AB
 P 7100 3600
@@
 $EndComp
 $Comp
-L C C17
+L device:C C17
 U 1 1 5A76A1B2
 P 7450 3600
@@
 $EndComp
 $Comp
-L C C18
+L device:C C18
 U 1 1 5A76A1B9
 P 7750 3600
@@
 $EndComp
 $Comp
-L C C19
+L device:C C19
 U 1 1 5A76A1C0
 P 8050 3600
@@
 $EndComp
 Wire Wire Line
-	6750 4150 8050 4150
+	6750 4150 7100 4150
 Wire Wire Line
 	6750 4150 6750 3750
 Wire Wire Line
-	7450 3750 7450 4350
+	7450 3750 7450 4150
 Wire Wire Line
 	7100 4150 7100 3750
@@
 Connection ~ 7750 4150
 Wire Wire Line
-	5450 3350 8050 3350
+	5450 3350 5700 3350
 Wire Wire Line
 	6750 3350 6750 3450
@@
 	7100 3350 7100 3450
 Wire Wire Line
-	7450 2950 7450 3450
+	7450 2950 7450 3350
 Connection ~ 7100 3350
 Wire Wire Line
@@
 CC3V3
 $Comp
-L D_Schottky D3
+L device:D_Schottky D3
 U 1 1 5A76813E
 P 5100 2900
@@
 	3800 4100 3800 4250
 $Comp
-L SI2323DS-T1-E3 IC6
+L SI2323DS-T1-E3:SI2323DS-T1-E3 IC6
 U 1 1 5A7685A7
 P 4750 3350
@@
 	4750 3450 4500 3450
 $Comp
-L R R1
+L device:R R1
 U 1 1 5A768BF5
 P 3100 3850
@@
 $EndComp
 $Comp
-L Earth #PWR16
+L power:Earth #PWR16
 U 1 1 5A768D52
 P 3800 4250
@@
 $EndComp
 $Comp
-L Earth #PWR15
+L power:Earth #PWR15
 U 1 1 5A768DD5
 P 3100 4250
@@
 $EndComp
 Wire Wire Line
-	2750 2900 3500 2900
-Wire Wire Line
-	4100 2900 4950 2900
+	2750 2900 3100 2900
+Wire Wire Line
+	4100 2900 4550 2900
 Wire Wire Line
 	3100 2900 3100 3700
@@
 	5700 2900 5700 3350
 $Comp
-L Jumper JP1
+L device:Jumper JP1
 U 1 1 5A769069
 P 3800 2900
@@
 Connection ~ 7100 4150
 $Comp
-L VCC #PWR17
+L power:VCC #PWR17
 U 1 1 5A769C0A
 P 7450 2950
@@
 	1    0    0    -1
 $EndComp
+Wire Wire Line
+	7750 4150 8050 4150
+Wire Wire Line
+	7100 3350 7450 3350
+Wire Wire Line
+	7450 3350 7450 3450
+Wire Wire Line
+	7450 3350 7750 3350
+Wire Wire Line
+	7750 3350 8050 3350
+Wire Wire Line
+	6750 3350 7100 3350
+Wire Wire Line
+	3100 2900 3500 2900
+Wire Wire Line
+	4550 2900 4950 2900
+Wire Wire Line
+	5700 3350 6750 3350
+Wire Wire Line
+	7450 4150 7750 4150
+Wire Wire Line
+	7450 4150 7450 4350
+Wire Wire Line
+	7100 4150 7450 4150
+$Comp
+L pspice:VSOURCE V?
+U 1 1 5A775452
+P 1900 5700
+F 0 "V?" H 2328 5746 50  0000 L CNN
+F 1 "VSOURCE" H 2328 5655 50  0000 L CNN
+F 2 "" H 1900 5700 50  0001 C CNN
+F 3 "" H 1900 5700 50  0001 C CNN
+F 4 "V" H 1900 5700 50  0001 C CNN "Spice_Primitive"
+F 5 "dc 3.3 pulse(0 3.3 1 0 0 1 1)" H 1900 5700 50  0001 C CNN "Spice_Model"
+F 6 "Y" H 1900 5700 50  0001 C CNN "Spice_Netlist_Enabled"
+	1    1900 5700
+	1    0    0    -1
+$EndComp
+$Comp
+L power:Earth #PWR?
+U 1 1 5A775D13
+P 1900 6400
+F 0 "#PWR?" H 1900 6150 50  0001 C CNN
+F 1 "Earth" H 1900 6250 50  0001 C CNN
+F 2 "" H 1900 6400 50  0001 C CNN
+F 3 "" H 1900 6400 50  0001 C CNN
+	1    1900 6400
+	1    0    0    -1
+$EndComp
+Text HLabel 1900 5000 0    60   Input ~ 0
+CC3V3
 $EndSCHEMATC

Commit message: Battery/debugger switch implemented
Parts:
- removed IC6: SI2323DS-T1-E3, SOT95P237X112-3N, symbol SI2323DS-T1-E3:SI2323DS-T1-E3
- removed V?: VSOURCE, symbol pspice:VSOURCE
- added Q1: SI2323DS, symbol device:Q_PMOS_GSD
- BT1: value Battery_Cell -> CR2477 3V Battery
- D3: value D_Schottky -> ZHCS350TA
- R1: value 100K -> 3.3K
Connections:
- wire segments 36 -> 35
Changed lines of the file:
@@
 L device:Battery_Cell BT1
 U 1 1 5A76A189
-P 3800 4000
-F 0 "BT1" H 3900 4100 50  0000 L CNN
-F 1 "Battery_Cell" H 3900 4000 50  0000 L CNN
-F 2 "" V 3800 4060 50  0001 C CNN
-F 3 "" V 3800 4060 50  0001 C CNN
-	1    3800 4000
-	1    0    0    -1
-$EndComp
-$Comp
-L power:Earth #PWR18
+P 3600 3650
+F 0 "BT1" H 3700 3750 50  0000 L CNN
+F 1 "CR2477 3V Battery" H 3700 3650 50  0000 L CNN
+F 2 "" V 3600 3710 50  0001 C CNN
+F 3 "" V 3600 3710 50  0001 C CNN
+	1    3600 3650
+	1    0    0    -1
+$EndComp
+$Comp
+L power:Earth #PWR018
 U 1 1 5A76A190
 P 7450 4350
-F 0 "#PWR18" H 7450 4100 50  0001 C CNN
+F 0 "#PWR018" H 7450 4100 50  0001 C CNN
 F 1 "Earth" H 7450 4200 50  0001 C CNN
 F 2 "" H 7450 4350 50  0001 C CNN
@@
 L device:Jumper JP2
 U 1 1 5A76A19D
-P 4200 3450
-F 0 "JP2" H 4200 3600 50  0000 C CNN
-F 1 "Jumper" H 4200 3370 50  0000 C CNN
-F 2 "" H 4200 3450 50  0001 C CNN
-F 3 "" H 4200 3450 50  0001 C CNN
-	1    4200 3450
+P 4100 3350
+F 0 "JP2" H 4100 3500 50  0000 C CNN
+F 1 "Jumper" H 4100 3270 50  0000 C CNN
+F 2 "" H 4100 3350 50  0001 C CNN
+F 3 "" H 4100 3350 50  0001 C CNN
+	1    4100 3350
 	1    0    0    -1
 $EndComp
@@
 	6750 4150 6750 3750
 Wire Wire Line
-	7450 3750 7450 4150
-Wire Wire Line
 	7100 4150 7100 3750
 Wire Wire Line
@@
 	8050 4150 8050 3750
 Connection ~ 7750 4150
-Wire Wire Line
-	5450 3350 5700 3350
 Wire Wire Line
 	6750 3350 6750 3450
@@
 Text Notes 7050 2300 2    60   ~ 0
 Battery & Debugger power switch & Reservoir Capacitors
-Connection ~ 6750 3350
-Text HLabel 2750 2900 0    60   Input ~ 0
+Text HLabel 3600 4650 3    60   Input ~ 0
 CC3V3
 $Comp
 L device:D_Schottky D3
 U 1 1 5A76813E
-P 5100 2900
-F 0 "D3" H 5100 3000 50  0000 C CNN
-F 1 "D_Schottky" H 5100 2800 50  0000 C CNN
-F 2 "" H 5100 2900 50  0001 C CNN
-F 3 "" H 5100 2900 50  0001 C CNN
-	1    5100 2900
+P 5700 3750
+F 0 "D3" H 5700 3850 50  0000 C CNN
+F 1 "ZHCS350TA" H 5700 3650 50  0000 C CNN
+F 2 "" H 5700 3750 50  0001 C CNN
+F 3 "" H 5700 3750 50  0001 C CNN
+	1    5700 3750
 	-1   0    0    1
 $EndComp
 Wire Wire Line
-	3800 3800 3800 3450
-Wire Wire Line
-	3800 3450 3900 3450
-Wire Wire Line
-	3800 4100 3800 4250
-$Comp
-L SI2323DS-T1-E3:SI2323DS-T1-E3 IC6
-U 1 1 5A7685A7
-P 4750 3350
-F 0 "IC6" H 5100 3500 50  0000 C CNN
-F 1 "SI2323DS-T1-E3" H 5100 3100 50  0000 C CNN
-F 2 "SOT95P237X112-3N" H 5100 3000 50  0001 C CNN
-F 3 "http://docs-europe.electrocomponents.com/webdocs/0ed1/0900766b80ed1e9a.pdf" H 5100 2900 50  0001 C CNN
-F 4 "SI2323DS-T1-E3, P-channel MOSFET Transistor 3.7 A 20 V, 3-Pin SOT-23, TO-236" H 5100 2800 50  0001 C CNN "Description"
-F 5 "RS" H 5100 2700 50  0001 C CNN "Supplier_Name"
-F 6 "7104698P" H 5100 2600 50  0001 C CNN "RS Part Number"
-F 7 "Vishay" H 5100 2500 50  0001 C CNN "Manufacturer_Name"
-F 8 "SI2323DS-T1-E3" H 5100 2400 50  0001 C CNN "Manufacturer_Part_Number"
-F 9 "70026097" H 5100 2300 50  0001 C CNN "Allied_Number"
-F 10 "" H 5100 2200 50  0001 C CNN "Other Part Number"
-F 11 "1.12" H 5300 2100 50  0001 C CNN "Height"
-	1    4750 3350
-	1    0    0    -1
-$EndComp
-Wire Wire Line
-	4750 3450 4500 3450
-$Comp
-L device:R R1
-U 1 1 5A768BF5
-P 3100 3850
-F 0 "R1" V 3180 3850 50  0000 C CNN
-F 1 "100K" V 3100 3850 50  0000 C CNN
-F 2 "" V 3030 3850 50  0001 C CNN
-F 3 "" H 3100 3850 50  0001 C CNN
-	1    3100 3850
-	1    0    0    -1
-$EndComp
-$Comp
-L power:Earth #PWR16
+	3600 3450 3600 3350
+Wire Wire Line
+	3600 3350 3800 3350
+Wire Wire Line
+	5100 3350 4400 3350
+$Comp
+L power:Earth #PWR016
 U 1 1 5A768D52
-P 3800 4250
-F 0 "#PWR16" H 3800 4000 50  0001 C CNN
-F 1 "Earth" H 3800 4100 50  0001 C CNN
-F 2 "" H 3800 4250 50  0001 C CNN
-F 3 "" H 3800 4250 50  0001 C CNN
-	1    3800 4250
-	1    0    0    -1
-$EndComp
-$Comp
-L power:Earth #PWR15
-U 1 1 5A768DD5
-P 3100 4250
-F 0 "#PWR15" H 3100 4000 50  0001 C CNN
-F 1 "Earth" H 3100 4100 50  0001 C CNN
-F 2 "" H 3100 4250 50  0001 C CNN
-F 3 "" H 3100 4250 50  0001 C CNN
-	1    3100 4250
-	1    0    0    -1
-$EndComp
-Wire Wire Line
-	2750 2900 3100 2900
-Wire Wire Line
-	4100 2900 4550 2900
-Wire Wire Line
-	3100 2900 3100 3700
-Wire Wire Line
-	3100 4250 3100 4000
-Wire Wire Line
-	4550 2900 4550 3350
-Wire Wire Line
-	4550 3350 4750 3350
-Wire Wire Line
-	5250 2900 5700 2900
-Wire Wire Line
-	5700 2900 5700 3350
+P 3600 3750
+F 0 "#PWR016" H 3600 3500 50  0001 C CNN
+F 1 "Earth" H 3600 3600 50  0001 C CNN
+F 2 "" H 3600 3750 50  0001 C CNN
+F 3 "" H 3600 3750 50  0001 C CNN
+	1    3600 3750
+	1    0    0    -1
+$EndComp
 $Comp
 L device:Jumper JP1
 U 1 1 5A769069
-P 3800 2900
-F 0 "JP1" H 3800 3050 50  0000 C CNN
-F 1 "Jumper" H 3800 2820 50  0000 C CNN
-F 2 "" H 3800 2900 50  0001 C CNN
-F 3 "" H 3800 2900 50  0001 C CNN
-	1    3800 2900
-	1    0    0    -1
-$EndComp
-Connection ~ 3100 2900
-Connection ~ 4550 2900
-Connection ~ 5700 3350
+P 4150 4650
+F 0 "JP1" H 4150 4800 50  0000 C CNN
+F 1 "Jumper" H 4150 4570 50  0000 C CNN
+F 2 "" H 4150 4650 50  0001 C CNN
+F 3 "" H 4150 4650 50  0001 C CNN
+	1    4150 4650
+	1    0    0    -1
+$EndComp
 Connection ~ 7450 4150
 Connection ~ 7100 4150
 $Comp
-L power:VCC #PWR17
+L power:VCC #PWR017
 U 1 1 5A769C0A
 P 7450 2950
-F 0 "#PWR17" H 7450 2800 50  0001 C CNN
+F 0 "#PWR017" H 7450 2800 50  0001 C CNN
 F 1 "VCC" H 7450 3100 50  0000 C CNN
 F 2 "" H 7450 2950 50  0001 C CNN
@@
 	6750 3350 7100 3350
 Wire Wire Line
-	3100 2900 3500 2900
-Wire Wire Line
-	4550 2900 4950 2900
-Wire Wire Line
-	5700 3350 6750 3350
-Wire Wire Line
 	7450 4150 7750 4150
 Wire Wire Line
@@
 Wire Wire Line
 	7100 4150 7450 4150
-$Comp
-L pspice:VSOURCE V?
-U 1 1 5A775452
-P 1900 5700
-F 0 "V?" H 2328 5746 50  0000 L CNN
-F 1 "VSOURCE" H 2328 5655 50  0000 L CNN
-F 2 "" H 1900 5700 50  0001 C CNN
-F 3 "" H 1900 5700 50  0001 C CNN
-F 4 "V" H 1900 5700 50  0001 C CNN "Spice_Primitive"
-F 5 "dc 3.3 pulse(0 3.3 1 0 0 1 1)" H 1900 5700 50  0001 C CNN "Spice_Model"
-F 6 "Y" H 1900 5700 50  0001 C CNN "Spice_Netlist_Enabled"
-	1    1900 5700
-	1    0    0    -1
-$EndComp
-$Comp
-L power:Earth #PWR?
-U 1 1 5A775D13
-P 1900 6400
-F 0 "#PWR?" H 1900 6150 50  0001 C CNN
-F 1 "Earth" H 1900 6250 50  0001 C CNN
-F 2 "" H 1900 6400 50  0001 C CNN
-F 3 "" H 1900 6400 50  0001 C CNN
-	1    1900 6400
-	1    0    0    -1
-$EndComp
-Text HLabel 1900 5000 0    60   Input ~ 0
-CC3V3
+Wire Wire Line
+	3600 4650 3850 4650
+Wire Wire Line
+	4450 4650 5300 4650
+Wire Wire Line
+	5300 4650 5300 4350
+$Comp
+L device:R R1
+U 1 1 5A77BAAF
+P 5650 4650
+F 0 "R1" H 5720 4696 50  0000 L CNN
+F 1 "3.3K" H 5720 4605 50  0000 L CNN
+F 2 "" V 5580 4650 50  0001 C CNN
+F 3 "" H 5650 4650 50  0001 C CNN
+	1    5650 4650
+	1    0    0    -1
+$EndComp
+$Comp
+L power:Earth #PWR015
+U 1 1 5A77BB41
+P 5650 4800
+F 0 "#PWR015" H 5650 4550 50  0001 C CNN
+F 1 "Earth" H 5650 4650 50  0001 C CNN
+F 2 "" H 5650 4800 50  0001 C CNN
+F 3 "" H 5650 4800 50  0001 C CNN
+	1    5650 4800
+	1    0    0    -1
+$EndComp
+Wire Wire Line
+	5650 4500 5650 4350
+Wire Wire Line
+	5650 4350 5300 4350
+Connection ~ 5300 4350
+Wire Wire Line
+	5300 4350 5300 3750
+Wire Wire Line
+	5300 3750 5550 3750
+Connection ~ 5300 3750
+Wire Wire Line
+	5300 3750 5300 3650
+Wire Wire Line
+	5850 3750 6100 3750
+Wire Wire Line
+	6100 3750 6100 3350
+Wire Wire Line
+	6100 3350 5500 3350
+Wire Wire Line
+	6100 3350 6750 3350
+Connection ~ 6100 3350
+Connection ~ 6750 3350
+$Comp
+L device:Q_PMOS_GSD Q1
+U 1 1 5A77DE74
+P 5300 3450
+F 0 "Q1" V 5643 3450 50  0000 C CNN
+F 1 "SI2323DS" V 5552 3450 50  0000 C CNN
+F 2 "" H 5500 3550 50  0001 C CNN
+F 3 "" H 5300 3450 50  0001 C CNN
+	1    5300 3450
+	0    -1   -1   0
+$EndComp
+Wire Wire Line
+	7450 3750 7450 4150
 $EndSCHEMATC

Commit message: Reverted to KiCad 4.0.7
+ Reworked debouncing for pushbuttons
Connections:
- wire segments 35 -> 23
Changed lines of the file:
@@
-EESchema Schematic File Version 4
+EESchema Schematic File Version 2
+LIBS:power
 LIBS:pir-cache
-EELAYER 26 0
+EELAYER 25 0
 EELAYER END
 $Descr A4 11693 8268
@@
 $EndComp
 Wire Wire Line
-	6750 4150 7100 4150
+	6750 4150 8050 4150
 Wire Wire Line
 	6750 4150 6750 3750
@@
 	7100 3350 7100 3450
 Wire Wire Line
-	7450 2950 7450 3350
+	7450 2950 7450 3450
 Connection ~ 7100 3350
 Wire Wire Line
@@
 $EndComp
 Wire Wire Line
-	7750 4150 8050 4150
-Wire Wire Line
-	7100 3350 7450 3350
-Wire Wire Line
-	7450 3350 7450 3450
-Wire Wire Line
-	7450 3350 7750 3350
-Wire Wire Line
-	7750 3350 8050 3350
-Wire Wire Line
-	6750 3350 7100 3350
-Wire Wire Line
-	7450 4150 7750 4150
-Wire Wire Line
-	7450 4150 7450 4350
-Wire Wire Line
-	7100 4150 7450 4150
+	5500 3350 8050 3350
+Wire Wire Line
+	7450 3750 7450 4350
 Wire Wire Line
 	3600 4650 3850 4650
 Wire Wire Line
-	4450 4650 5300 4650
-Wire Wire Line
-	5300 4650 5300 4350
+	5300 4650 4450 4650
+Wire Wire Line
+	5300 3650 5300 4650
 $Comp
 L device:R R1
@@
 Connection ~ 5300 4350
 Wire Wire Line
-	5300 4350 5300 3750
-Wire Wire Line
 	5300 3750 5550 3750
 Connection ~ 5300 3750
 Wire Wire Line
-	5300 3750 5300 3650
-Wire Wire Line
 	5850 3750 6100 3750
 Wire Wire Line
 	6100 3750 6100 3350
-Wire Wire Line
-	6100 3350 5500 3350
-Wire Wire Line
-	6100 3350 6750 3350
 Connection ~ 6100 3350
 Connection ~ 6750 3350
@@
 	0    -1   -1   0
 $EndComp
-Wire Wire Line
-	7450 3750 7450 4150
 $EndSCHEMATC

Commit message: MCU change, again
STM32L0 had quite a big problem, common reference for the comparators.
Another minus was the missing SWO for debugging.

STM32L4 has floating point, and most importantly, has embedded OPAMPS!
This means I can directly plug in the filter to the analog inputs and
everything is software. 2 opamps and 2 comparators (if needed).
External circuitry would be minimal for the PIR sensor.

It also means that I can read with the embedded 12-bit ADC the
amplified values. Precision is not crucial, we are interested in dips
and swells.
Connections:
- net labels added: Debugger3V3
- net labels removed: CC3V3
Changed lines of the file:
@@
 EESchema Schematic File Version 2
+LIBS:74xgxx
+LIBS:74xx
+LIBS:Altera
+LIBS:ESD_Protection
+LIBS:LEM
+LIBS:Lattice
+LIBS:Oscillators
+LIBS:Power_Management
+LIBS:RFSolutions
+LIBS:Worldsemi
+LIBS:Xicor
+LIBS:Zilog
+LIBS:ac-dc
+LIBS:actel
+LIBS:adc-dac
+LIBS:allegro
+LIBS:analog_devices
+LIBS:analog_switches
+LIBS:atmel
+LIBS:audio
+LIBS:battery_management
+LIBS:bbd
+LIBS:bosch
+LIBS:brooktre
+LIBS:cmos4000
+LIBS:cmos_ieee
+LIBS:conn
+LIBS:contrib
+LIBS:cypress
+LIBS:dc-dc
+LIBS:device
+LIBS:digital-audio
+LIBS:diode
+LIBS:display
+LIBS:dsp
+LIBS:elec-unifil
+LIBS:ftdi
+LIBS:gennum
+LIBS:graphic_symbols
+LIBS:hc11
+LIBS:infineon
+LIBS:intel
+LIBS:interface
+LIBS:intersil
+LIBS:ir
+LIBS:leds
+LIBS:linear
+LIBS:logic_programmable
+LIBS:maxim
+LIBS:mechanical
+LIBS:memory
+LIBS:microchip
+LIBS:microchip_dspic33dsc
+LIBS:microchip_pic10mcu
+LIBS:microchip_pic12mcu
+LIBS:microchip_pic16mcu
+LIBS:microchip_pic18mcu
+LIBS:microchip_pic24mcu
+LIBS:microchip_pic32mcu
+LIBS:microcontrollers
+LIBS:modules
+LIBS:motor_drivers
+LIBS:motorola
+LIBS:motors
+LIBS:msp430
+LIBS:nordicsemi
+LIBS:nxp
+LIBS:nxp_armmcu
+LIBS:onsemi
+LIBS:opto
+LIBS:philips
 LIBS:power
+LIBS:powerint
+LIBS:pspice
+LIBS:references
+LIBS:regul
+LIBS:relays
+LIBS:rfcom
+LIBS:sensors
+LIBS:silabs
+LIBS:siliconi
+LIBS:stm32
+LIBS:stm8
+LIBS:supertex
+LIBS:switches
+LIBS:texas
+LIBS:transf
+LIBS:transistors
+LIBS:triac_thyristor
+LIBS:ttl_ieee
+LIBS:valves
+LIBS:video
+LIBS:wiznet
+LIBS:xilinx
+LIBS:zetex
+LIBS:SparkFun
+LIBS:ab2_7segment
+LIBS:ab2_audio
+LIBS:ab2_buffer
+LIBS:ab2_capacitor
+LIBS:ab2_connectivity
+LIBS:ab2_dac
+LIBS:ab2_diode
+LIBS:ab2_fuse
+LIBS:ab2_gpio_expansion
+LIBS:ab2_header
+LIBS:ab2_idc
+LIBS:ab2_inductor
+LIBS:ab2_input_devices
+LIBS:ab2_jumper
+LIBS:ab2_lcd
+LIBS:ab2_led
+LIBS:ab2_memory
+LIBS:ab2_opamp
+LIBS:ab2_pinouts
+LIBS:ab2_pot
+LIBS:ab2_power
+LIBS:ab2_regulator
+LIBS:ab2_relay
+LIBS:ab2_resistor
+LIBS:ab2_sensor
+LIBS:ab2_stepper
+LIBS:ab2_supply
+LIBS:ab2_terminal_block
+LIBS:ab2_test
+LIBS:ab2_transistor
+LIBS:ab2_uC
+LIBS:ab2_usb
+LIBS:ab2_xtal
 LIBS:pir-cache
 EELAYER 25 0
@@
 Battery & Debugger power switch & Reservoir Capacitors
 Text HLabel 3600 4650 3    60   Input ~ 0
-CC3V3
+Debugger3V3
 $Comp
 L device:D_Schottky D3
