File: pcb/battery.sch (KiCad schematic (older format))
At the start: 11 parts, among them Q1 SI2323DS

Commit message: Renamed all components
Parts:
- renumbered C15 to C13, C16 to C14, C17 to C15, C18 to C16, C19 to C17, D3 to D2, JP2 to JP1, JP1 to JP2, R1 to R10
Changed lines of the file:
@@
 LIBS:ab2_usb
 LIBS:ab2_xtal
+LIBS:pir-cache
 EELAYER 25 0
 EELAYER END
@@
 $EndComp
 $Comp
-L power:Earth #PWR018
+L power:Earth #PWR12
 U 1 1 5A76A190
 P 7450 4350
-F 0 "#PWR018" H 7450 4100 50  0001 C CNN
+F 0 "#PWR12" H 7450 4100 50  0001 C CNN
 F 1 "Earth" H 7450 4200 50  0001 C CNN
 F 2 "" H 7450 4350 50  0001 C CNN
@@
 $EndComp
 $Comp
-L device:Jumper JP2
+L device:Jumper JP1
 U 1 1 5A76A19D
 P 4100 3350
-F 0 "JP2" H 4100 3500 50  0000 C CNN
+F 0 "JP1" H 4100 3500 50  0000 C CNN
 F 1 "Jumper" H 4100 3270 50  0000 C CNN
 F 2 "" H 4100 3350 50  0001 C CNN
@@
 $EndComp
 $Comp
-L device:C C15
+L device:C C13
 U 1 1 5A76A1A4
 P 6750 3600
-F 0 "C15" H 6775 3700 50  0000 L CNN
+F 0 "C13" H 6775 3700 50  0000 L CNN
 F 1 "100μF" H 6775 3500 50  0000 L CNN
 F 2 "" H 6788 3450 50  0001 C CNN
@@
 $EndComp
 $Comp
-L device:C C16
+L device:C C14
 U 1 1 5A76A1AB
 P 7100 3600
-F 0 "C16" H 7125 3700 50  0000 L CNN
+F 0 "C14" H 7125 3700 50  0000 L CNN
 F 1 "10μF" H 7125 3500 50  0000 L CNN
 F 2 "" H 7138 3450 50  0001 C CNN
@@
 $EndComp
 $Comp
-L device:C C17
+L device:C C15
 U 1 1 5A76A1B2
 P 7450 3600
-F 0 "C17" H 7475 3700 50  0000 L CNN
+F 0 "C15" H 7475 3700 50  0000 L CNN
 F 1 "1μF" H 7475 3500 50  0000 L CNN
 F 2 "" H 7488 3450 50  0001 C CNN
@@
 $EndComp
 $Comp
-L device:C C18
+L device:C C16
 U 1 1 5A76A1B9
 P 7750 3600
-F 0 "C18" H 7775 3700 50  0000 L CNN
+F 0 "C16" H 7775 3700 50  0000 L CNN
 F 1 "0.1μF" H 7775 3500 50  0000 L CNN
 F 2 "" H 7788 3450 50  0001 C CNN
@@
 $EndComp
 $Comp
-L device:C C19
+L device:C C17
 U 1 1 5A76A1C0
 P 8050 3600
-F 0 "C19" H 8075 3700 50  0000 L CNN
+F 0 "C17" H 8075 3700 50  0000 L CNN
 F 1 "0.01μF" H 8075 3500 50  0000 L CNN
 F 2 "" H 8088 3450 50  0001 C CNN
@@
 Debugger3V3
 $Comp
-L device:D_Schottky D3
+L device:D_Schottky D2
 U 1 1 5A76813E
 P 5700 3750
-F 0 "D3" H 5700 3850 50  0000 C CNN
+F 0 "D2" H 5700 3850 50  0000 C CNN
 F 1 "ZHCS350TA" H 5700 3650 50  0000 C CNN
 F 2 "" H 5700 3750 50  0001 C CNN
@@
 	5100 3350 4400 3350
 $Comp
-L power:Earth #PWR016
+L power:Earth #PWR9
 U 1 1 5A768D52
 P 3600 3750
-F 0 "#PWR016" H 3600 3500 50  0001 C CNN
+F 0 "#PWR9" H 3600 3500 50  0001 C CNN
 F 1 "Earth" H 3600 3600 50  0001 C CNN
 F 2 "" H 3600 3750 50  0001 C CNN
@@
 $EndComp
 $Comp
-L device:Jumper JP1
+L device:Jumper JP2
 U 1 1 5A769069
 P 4150 4650
-F 0 "JP1" H 4150 4800 50  0000 C CNN
+F 0 "JP2" H 4150 4800 50  0000 C CNN
 F 1 "Jumper" H 4150 4570 50  0000 C CNN
 F 2 "" H 4150 4650 50  0001 C CNN
@@
 Connection ~ 7100 4150
 $Comp
-L power:VCC #PWR017
+L power:VCC #PWR11
 U 1 1 5A769C0A
 P 7450 2950
-F 0 "#PWR017" H 7450 2800 50  0001 C CNN
+F 0 "#PWR11" H 7450 2800 50  0001 C CNN
 F 1 "VCC" H 7450 3100 50  0000 C CNN
 F 2 "" H 7450 2950 50  0001 C CNN
@@
 	5300 3650 5300 4650
 $Comp
-L device:R R1
+L device:R R10
 U 1 1 5A77BAAF
 P 5650 4650
-F 0 "R1" H 5720 4696 50  0000 L CNN
+F 0 "R10" H 5720 4696 50  0000 L CNN
 F 1 "3.3K" H 5720 4605 50  0000 L CNN
 F 2 "" V 5580 4650 50  0001 C CNN
@@
 $EndComp
 $Comp
-L power:Earth #PWR015
+L power:Earth #PWR10
 U 1 1 5A77BB41
 P 5650 4800
-F 0 "#PWR015" H 5650 4550 50  0001 C CNN
+F 0 "#PWR10" H 5650 4550 50  0001 C CNN
 F 1 "Earth" H 5650 4650 50  0001 C CNN
 F 2 "" H 5650 4800 50  0001 C CNN

Commit message: Added testpoints
Parts:
- removed D2: ZHCS350TA, symbol device:D_Schottky
- added D2: MBR0530, Diodes_SMD:SOD-123, symbol MBR0530
- added TP10: TEST, symbol TEST
- renumbered R10 to R11
Changed lines of the file:
@@
 $EndComp
 $Comp
-L power:Earth #PWR09
+L power:Earth #PWR12
 U 1 1 5A76A190
 P 7450 4350
-F 0 "#PWR09" H 7450 4100 50  0001 C CNN
+F 0 "#PWR12" H 7450 4100 50  0001 C CNN
 F 1 "Earth" H 7450 4200 50  0001 C CNN
 F 2 "" H 7450 4350 50  0001 C CNN
@@
 Text HLabel 3600 4650 3    60   Input ~ 0
 Debugger3V3
-$Comp
-L device:D_Schottky D2
-U 1 1 5A76813E
-P 5700 3750
-F 0 "D2" H 5700 3850 50  0000 C CNN
-F 1 "ZHCS350TA" H 5700 3650 50  0000 C CNN
-F 2 "" H 5700 3750 50  0001 C CNN
-F 3 "" H 5700 3750 50  0001 C CNN
-	1    5700 3750
-	-1   0    0    1
-$EndComp
 Wire Wire Line
 	3600 3450 3600 3350
@@
 	5100 3350 4400 3350
 $Comp
-L power:Earth #PWR010
+L power:Earth #PWR9
 U 1 1 5A768D52
 P 3600 3750
-F 0 "#PWR010" H 3600 3500 50  0001 C CNN
+F 0 "#PWR9" H 3600 3500 50  0001 C CNN
 F 1 "Earth" H 3600 3600 50  0001 C CNN
 F 2 "" H 3600 3750 50  0001 C CNN
@@
 Connection ~ 7100 4150
 $Comp
-L power:VCC #PWR011
+L power:VCC #PWR11
 U 1 1 5A769C0A
 P 7450 2950
-F 0 "#PWR011" H 7450 2800 50  0001 C CNN
+F 0 "#PWR11" H 7450 2800 50  0001 C CNN
 F 1 "VCC" H 7450 3100 50  0000 C CNN
 F 2 "" H 7450 2950 50  0001 C CNN
@@
 	5300 3650 5300 4650
 $Comp
-L device:R R10
+L device:R R11
 U 1 1 5A77BAAF
 P 5650 4650
-F 0 "R10" H 5720 4696 50  0000 L CNN
+F 0 "R11" H 5720 4696 50  0000 L CNN
 F 1 "3.3K" H 5720 4605 50  0000 L CNN
 F 2 "" V 5580 4650 50  0001 C CNN
@@
 $EndComp
 $Comp
-L power:Earth #PWR012
+L power:Earth #PWR10
 U 1 1 5A77BB41
 P 5650 4800
-F 0 "#PWR012" H 5650 4550 50  0001 C CNN
+F 0 "#PWR10" H 5650 4550 50  0001 C CNN
 F 1 "Earth" H 5650 4650 50  0001 C CNN
 F 2 "" H 5650 4800 50  0001 C CNN
@@
 	0    -1   -1   0
 $EndComp
+$Comp
+L TEST TP10
+U 1 1 5A8395CF
+P 8050 3350
+F 0 "TP10" H 8050 3650 50  0000 C BNN
+F 1 "TEST" H 8050 3600 50  0000 C CNN
+F 2 "" H 8050 3350 50  0001 C CNN
+F 3 "" H 8050 3350 50  0001 C CNN
+	1    8050 3350
+	1    0    0    -1
+$EndComp
+$Comp
+L MBR0530 D2
+U 1 1 5A83A7D7
+P 5700 3750
+F 0 "D2" H 5700 3850 50  0000 C CNN
+F 1 "MBR0530" H 5700 3650 50  0000 C CNN
+F 2 "Diodes_SMD:SOD-123" H 5700 3575 50  0001 C CNN
+F 3 "" H 5700 3750 50  0001 C CNN
+	1    5700 3750
+	-1   0    0    1
+$EndComp
 $EndSCHEMATC

Commit message: Assigned footprints to all components
Parts:
- removed C13: 100μF, symbol device:C
- added C13: 100u, Capacitors_SMD:CP_Elec_5x5.3, symbol CP
- BT1: footprint (none) -> Battery_Holders:Keystone_105_1x2430-CoinCell
- C14, C15, C16, C17: footprint (none) -> Capacitors_SMD:C_1210
- JP1, JP2: footprint (none) -> Pin_Headers:Pin_Header_Angled_1x02_Pitch2.54mm
- Q1: footprint (none) -> SI2323DS-T1-E3:SOT95P237X112-3N
- R11: footprint (none) -> Resistors_SMD:R_1210
- TP10: footprint (none) -> Measurement_Points:Measurement_Point_Round-TH_Small
Changed lines of the file:
@@
 F 0 "BT1" H 3700 3750 50  0000 L CNN
 F 1 "CR2477 3V Battery" H 3700 3650 50  0000 L CNN
-F 2 "" V 3600 3710 50  0001 C CNN
+F 2 "Battery_Holders:Keystone_105_1x2430-CoinCell" V 3600 3710 50  0001 C CNN
 F 3 "" V 3600 3710 50  0001 C CNN
 	1    3600 3650
@@
 F 0 "JP1" H 4100 3500 50  0000 C CNN
 F 1 "Jumper" H 4100 3270 50  0000 C CNN
-F 2 "" H 4100 3350 50  0001 C CNN
+F 2 "Pin_Headers:Pin_Header_Angled_1x02_Pitch2.54mm" H 4100 3350 50  0001 C CNN
 F 3 "" H 4100 3350 50  0001 C CNN
 	1    4100 3350
-	1    0    0    -1
-$EndComp
-$Comp
-L device:C C13
-U 1 1 5A76A1A4
-P 6750 3600
-F 0 "C13" H 6775 3700 50  0000 L CNN
-F 1 "100μF" H 6775 3500 50  0000 L CNN
-F 2 "" H 6788 3450 50  0001 C CNN
-F 3 "" H 6750 3600 50  0001 C CNN
-	1    6750 3600
 	1    0    0    -1
 $EndComp
@@
 F 0 "C14" H 7125 3700 50  0000 L CNN
 F 1 "10μF" H 7125 3500 50  0000 L CNN
-F 2 "" H 7138 3450 50  0001 C CNN
+F 2 "Capacitors_SMD:C_1210" H 7138 3450 50  0001 C CNN
 F 3 "" H 7100 3600 50  0001 C CNN
 	1    7100 3600
@@
 F 0 "C15" H 7475 3700 50  0000 L CNN
 F 1 "1μF" H 7475 3500 50  0000 L CNN
-F 2 "" H 7488 3450 50  0001 C CNN
+F 2 "Capacitors_SMD:C_1210" H 7488 3450 50  0001 C CNN
 F 3 "" H 7450 3600 50  0001 C CNN
 	1    7450 3600
@@
 F 0 "C16" H 7775 3700 50  0000 L CNN
 F 1 "0.1μF" H 7775 3500 50  0000 L CNN
-F 2 "" H 7788 3450 50  0001 C CNN
+F 2 "Capacitors_SMD:C_1210" H 7788 3450 50  0001 C CNN
 F 3 "" H 7750 3600 50  0001 C CNN
 	1    7750 3600
@@
 F 0 "C17" H 8075 3700 50  0000 L CNN
 F 1 "0.01μF" H 8075 3500 50  0000 L CNN
-F 2 "" H 8088 3450 50  0001 C CNN
+F 2 "Capacitors_SMD:C_1210" H 8088 3450 50  0001 C CNN
 F 3 "" H 8050 3600 50  0001 C CNN
 	1    8050 3600
@@
 Wire Wire Line
 	6750 4150 8050 4150
-Wire Wire Line
-	6750 4150 6750 3750
 Wire Wire Line
 	7100 4150 7100 3750
@@
 F 0 "JP2" H 4150 4800 50  0000 C CNN
 F 1 "Jumper" H 4150 4570 50  0000 C CNN
-F 2 "" H 4150 4650 50  0001 C CNN
+F 2 "Pin_Headers:Pin_Header_Angled_1x02_Pitch2.54mm" H 4150 4650 50  0001 C CNN
 F 3 "" H 4150 4650 50  0001 C CNN
 	1    4150 4650
@@
 F 0 "R11" H 5720 4696 50  0000 L CNN
 F 1 "3.3K" H 5720 4605 50  0000 L CNN
-F 2 "" V 5580 4650 50  0001 C CNN
+F 2 "Resistors_SMD:R_1210" V 5580 4650 50  0001 C CNN
 F 3 "" H 5650 4650 50  0001 C CNN
 	1    5650 4650
@@
 F 0 "Q1" V 5643 3450 50  0000 C CNN
 F 1 "SI2323DS" V 5552 3450 50  0000 C CNN
-F 2 "" H 5500 3550 50  0001 C CNN
+F 2 "SI2323DS-T1-E3:SOT95P237X112-3N" H 5500 3550 50  0001 C CNN
 F 3 "" H 5300 3450 50  0001 C CNN
 	1    5300 3450
@@
 F 0 "TP10" H 8050 3650 50  0000 C BNN
 F 1 "TEST" H 8050 3600 50  0000 C CNN
-F 2 "" H 8050 3350 50  0001 C CNN
+F 2 "Measurement_Points:Measurement_Point_Round-TH_Small" H 8050 3350 50  0001 C CNN
 F 3 "" H 8050 3350 50  0001 C CNN
 	1    8050 3350
@@
 	-1   0    0    1
 $EndComp
+$Comp
+L CP C13
+U 1 1 5A8357D1
+P 6750 3600
+F 0 "C13" H 6775 3700 50  0000 L CNN
+F 1 "100u" H 6775 3500 50  0000 L CNN
+F 2 "Capacitors_SMD:CP_Elec_5x5.3" H 6788 3450 50  0001 C CNN
+F 3 "" H 6750 3600 50  0001 C CNN
+	1    6750 3600
+	1    0    0    -1
+$EndComp
+Wire Wire Line
+	6750 4150 6750 3750
 $EndSCHEMATC

Commit message: Reassigned some footprints, added some libraries
Normally I can start working on PCB.
Parts:
- C14, C15, C16, C17: footprint Capacitors_SMD:C_1210 -> Capacitors_SMD:C_1206
- D2: footprint Diodes_SMD:SOD-123 -> MBR0530:SOD3716X135N
- JP1, JP2: footprint Pin_Headers:Pin_Header_Angled_1x02_Pitch2.54mm -> Pin_Headers:Pin_Header_Straight_1x02_Pitch2.54mm
- R11: footprint Resistors_SMD:R_1210 -> Resistors_SMD:R_1206
Changed lines of the file:
@@
 LIBS:EL817S
 LIBS:IRA-S210ST01
+LIBS:RE1C002UNTCL
+LIBS:SJ-2523-SMT-TR
 LIBS:pir-cache
 EELAYER 25 0
@@
 $EndComp
 $Comp
-L power:Earth #PWR09
+L power:Earth #PWR010
 U 1 1 5A76A190
 P 7450 4350
-F 0 "#PWR09" H 7450 4100 50  0001 C CNN
+F 0 "#PWR010" H 7450 4100 50  0001 C CNN
 F 1 "Earth" H 7450 4200 50  0001 C CNN
 F 2 "" H 7450 4350 50  0001 C CNN
@@
 F 0 "JP1" H 4100 3500 50  0000 C CNN
 F 1 "Jumper" H 4100 3270 50  0000 C CNN
-F 2 "Pin_Headers:Pin_Header_Angled_1x02_Pitch2.54mm" H 4100 3350 50  0001 C CNN
+F 2 "Pin_Headers:Pin_Header_Straight_1x02_Pitch2.54mm" H 4100 3350 50  0001 C CNN
 F 3 "" H 4100 3350 50  0001 C CNN
 	1    4100 3350
@@
 F 0 "C14" H 7125 3700 50  0000 L CNN
 F 1 "10μF" H 7125 3500 50  0000 L CNN
-F 2 "Capacitors_SMD:C_1210" H 7138 3450 50  0001 C CNN
+F 2 "Capacitors_SMD:C_1206" H 7138 3450 50  0001 C CNN
 F 3 "" H 7100 3600 50  0001 C CNN
 	1    7100 3600
@@
 F 0 "C15" H 7475 3700 50  0000 L CNN
 F 1 "1μF" H 7475 3500 50  0000 L CNN
-F 2 "Capacitors_SMD:C_1210" H 7488 3450 50  0001 C CNN
+F 2 "Capacitors_SMD:C_1206" H 7488 3450 50  0001 C CNN
 F 3 "" H 7450 3600 50  0001 C CNN
 	1    7450 3600
@@
 F 0 "C16" H 7775 3700 50  0000 L CNN
 F 1 "0.1μF" H 7775 3500 50  0000 L CNN
-F 2 "Capacitors_SMD:C_1210" H 7788 3450 50  0001 C CNN
+F 2 "Capacitors_SMD:C_1206" H 7788 3450 50  0001 C CNN
 F 3 "" H 7750 3600 50  0001 C CNN
 	1    7750 3600
@@
 F 0 "C17" H 8075 3700 50  0000 L CNN
 F 1 "0.01μF" H 8075 3500 50  0000 L CNN
-F 2 "Capacitors_SMD:C_1210" H 8088 3450 50  0001 C CNN
+F 2 "Capacitors_SMD:C_1206" H 8088 3450 50  0001 C CNN
 F 3 "" H 8050 3600 50  0001 C CNN
 	1    8050 3600
@@
 	5100 3350 4400 3350
 $Comp
-L power:Earth #PWR010
+L power:Earth #PWR011
 U 1 1 5A768D52
 P 3600 3750
-F 0 "#PWR010" H 3600 3500 50  0001 C CNN
+F 0 "#PWR011" H 3600 3500 50  0001 C CNN
 F 1 "Earth" H 3600 3600 50  0001 C CNN
 F 2 "" H 3600 3750 50  0001 C CNN
@@
 F 0 "JP2" H 4150 4800 50  0000 C CNN
 F 1 "Jumper" H 4150 4570 50  0000 C CNN
-F 2 "Pin_Headers:Pin_Header_Angled_1x02_Pitch2.54mm" H 4150 4650 50  0001 C CNN
+F 2 "Pin_Headers:Pin_Header_Straight_1x02_Pitch2.54mm" H 4150 4650 50  0001 C CNN
 F 3 "" H 4150 4650 50  0001 C CNN
 	1    4150 4650
@@
 Connection ~ 7100 4150
 $Comp
-L power:VCC #PWR011
+L power:VCC #PWR012
 U 1 1 5A769C0A
 P 7450 2950
-F 0 "#PWR011" H 7450 2800 50  0001 C CNN
+F 0 "#PWR012" H 7450 2800 50  0001 C CNN
 F 1 "VCC" H 7450 3100 50  0000 C CNN
 F 2 "" H 7450 2950 50  0001 C CNN
@@
 F 0 "R11" H 5720 4696 50  0000 L CNN
 F 1 "3.3K" H 5720 4605 50  0000 L CNN
-F 2 "Resistors_SMD:R_1210" V 5580 4650 50  0001 C CNN
+F 2 "Resistors_SMD:R_1206" V 5580 4650 50  0001 C CNN
 F 3 "" H 5650 4650 50  0001 C CNN
 	1    5650 4650
@@
 $EndComp
 $Comp
-L power:Earth #PWR012
+L power:Earth #PWR013
 U 1 1 5A77BB41
 P 5650 4800
-F 0 "#PWR012" H 5650 4550 50  0001 C CNN
+F 0 "#PWR013" H 5650 4550 50  0001 C CNN
 F 1 "Earth" H 5650 4650 50  0001 C CNN
 F 2 "" H 5650 4800 50  0001 C CNN
@@
 F 0 "D2" H 5700 3850 50  0000 C CNN
 F 1 "MBR0530" H 5700 3650 50  0000 C CNN
-F 2 "Diodes_SMD:SOD-123" H 5700 3575 50  0001 C CNN
+F 2 "MBR0530:SOD3716X135N" H 5700 3575 50  0001 C CNN
 F 3 "" H 5700 3750 50  0001 C CNN
 	1    5700 3750
