File: pcb/sensor.sch (KiCad schematic (older format))
At the start: 31 parts, among them IC1 IRA-S210ST01, IC2 LPV802DGKT, IC3 TLV3691IDCKR, IC4 TLV3691IDCKR

Commit message: User pushbutton
Parts:
- removed JP2: Jumper, symbol Jumper
Connections:
- wire segments 83 -> 119
Changed lines of the file:
@@
 L VCC #PWR1
 U 1 1 5A74E3A0
-P 850 4500
-F 0 "#PWR1" H 850 4350 50  0001 C CNN
-F 1 "VCC" H 850 4650 50  0000 C CNN
-F 2 "" H 850 4500 50  0001 C CNN
-F 3 "" H 850 4500 50  0001 C CNN
-	1    850  4500
-	1    0    0    -1
-$EndComp
-$Comp
-L Jumper JP2
-U 1 1 5A74E453
-P 1250 4850
-F 0 "JP2" H 1250 5000 50  0000 C CNN
-F 1 "Jumper" H 1250 4770 50  0000 C CNN
-F 2 "" H 1250 4850 50  0001 C CNN
-F 3 "" H 1250 4850 50  0001 C CNN
-	1    1250 4850
-	-1   0    0    1
+P 1400 4500
+F 0 "#PWR1" H 1400 4350 50  0001 C CNN
+F 1 "VCC" H 1400 4650 50  0000 C CNN
+F 2 "" H 1400 4500 50  0001 C CNN
+F 3 "" H 1400 4500 50  0001 C CNN
+	1    1400 4500
+	1    0    0    -1
 $EndComp
 $Comp
@@
 $EndComp
 Wire Wire Line
-	850  4850 950  4850
-Wire Wire Line
-	1550 4850 1750 4850
-Wire Wire Line
-	2050 4850 4200 4850
+	1400 4850 1750 4850
+Wire Wire Line
+	2050 4850 2300 4850
+Wire Wire Line
+	2300 4850 2650 4850
+Wire Wire Line
+	2650 4850 3000 4850
+Wire Wire Line
+	3000 4850 3300 4850
+Wire Wire Line
+	3300 4850 3600 4850
+Wire Wire Line
+	3600 4850 3900 4850
+Wire Wire Line
+	3900 4850 4200 4850
 Wire Wire Line
 	2300 4850 2300 5050
@@
 Connection ~ 3900 4850
 Wire Wire Line
-	2300 5350 2300 5600
+	2300 5350 2300 5500
+Wire Wire Line
+	2300 5500 2300 5600
 Wire Wire Line
 	2650 5500 2650 5350
@@
 	7850 4350 7850 4250
 Wire Wire Line
-	2300 5500 6600 5500
-Wire Wire Line
-	5850 4550 6650 4550
+	2300 5500 2650 5500
+Wire Wire Line
+	2650 5500 3000 5500
+Wire Wire Line
+	3000 5500 3300 5500
+Wire Wire Line
+	3300 5500 3600 5500
+Wire Wire Line
+	3600 5500 3900 5500
+Wire Wire Line
+	3900 5500 4200 5500
+Wire Wire Line
+	4200 5500 5050 5500
+Wire Wire Line
+	5050 5500 6300 5500
+Wire Wire Line
+	6300 5500 6600 5500
+Wire Wire Line
+	5850 4550 6300 4550
+Wire Wire Line
+	6300 4550 6650 4550
 Wire Wire Line
 	6650 4650 6600 4650
@@
 	5300 2500 5300 2450
 Wire Wire Line
-	5300 2450 5900 2450
+	5300 2450 5850 2450
+Wire Wire Line
+	5850 2450 5900 2450
 Wire Wire Line
 	6500 2450 6550 2450
 Wire Wire Line
-	6550 2450 6550 4350
+	6550 2450 6550 3000
+Wire Wire Line
+	6550 3000 6550 3500
+Wire Wire Line
+	6550 3500 6550 3900
+Wire Wire Line
+	6550 3900 6550 4350
 Wire Wire Line
 	6550 3000 6500 3000
@@
 	5900 3000 5850 3000
 Wire Wire Line
-	5850 2450 5850 4450
+	5850 2450 5850 3000
+Wire Wire Line
+	5850 3000 5850 3500
+Wire Wire Line
+	5850 3500 5850 3900
+Wire Wire Line
+	5850 3900 5850 4450
 Wire Wire Line
 	5850 3500 6050 3500
@@
 Connection ~ 5850 3500
 Wire Wire Line
-	6350 3900 6850 3900
+	6350 3900 6550 3900
+Wire Wire Line
+	6550 3900 6850 3900
 Connection ~ 6550 3500
 Wire Wire Line
@@
 	8000 3900 7700 3900
 Wire Wire Line
-	8000 3250 8000 4550
+	8000 3250 8000 3600
+Wire Wire Line
+	8000 3600 8000 3900
+Wire Wire Line
+	8000 3900 8000 4550
 Wire Wire Line
 	8000 4550 7750 4550
@@
 	8350 3250 8400 3250
 Wire Wire Line
-	8400 3250 8400 5250
+	8400 3250 8400 3600
+Wire Wire Line
+	8400 3600 8400 3900
+Wire Wire Line
+	8400 3900 8400 4450
+Wire Wire Line
+	8400 4450 8400 5250
 Wire Wire Line
 	8400 3600 8350 3600
@@
 	10450 5050 10600 5050
 Wire Wire Line
-	8950 3750 8950 4150
+	8950 3750 8950 4100
+Wire Wire Line
+	8950 4100 8950 4150
 Wire Wire Line
 	8950 5550 8950 5600
@@
 	8950 3450 8950 3200
 Wire Wire Line
-	8950 4100 9550 4100
+	8950 4100 9300 4100
+Wire Wire Line
+	9300 4100 9550 4100
 Connection ~ 8950 4100
 Wire Wire Line
-	8950 4450 8950 4700
+	8950 4450 8950 4650
+Wire Wire Line
+	8950 4650 8950 4700
 Wire Wire Line
 	9550 4000 9500 4000
@@
 	9550 5150 9500 5150
 Wire Wire Line
-	9500 5150 9500 5600
+	9500 5150 9500 5550
+Wire Wire Line
+	9500 5550 9500 5600
 Wire Wire Line
 	8400 5250 9550 5250
 Wire Wire Line
-	8950 5000 8950 5250
-Wire Wire Line
-	9500 4000 9500 4600
-Wire Wire Line
-	8950 5050 9550 5050
+	8950 5000 8950 5050
+Wire Wire Line
+	8950 5050 8950 5250
+Wire Wire Line
+	9500 4000 9500 4550
+Wire Wire Line
+	9500 4550 9500 4600
+Wire Wire Line
+	8950 5050 9300 5050
+Wire Wire Line
+	9300 5050 9550 5050
 Connection ~ 8950 5050
 Wire Wire Line
@@
 Connection ~ 9500 5550
 Wire Wire Line
-	7750 4650 8950 4650
+	7750 4650 7950 4650
+Wire Wire Line
+	7950 4650 8950 4650
 Connection ~ 8950 4650
 Wire Wire Line
@@
 Signal Conditioning
 Wire Wire Line
-	850  4850 850  4500
+	1400 4850 1400 4500
 Connection ~ 5850 2450
 Text HLabel 10600 3900 2    60   Output ~ 0

Commit message: Added light sensor with IIC interface
Parts:
- added 10K1, 10K2, 10K3: R, symbol R
- added IC1: MAX44009EDT+T, SON65P200X200X65-7N, symbol MAX44009EDT+T
- renumbered C6 to C1, C15 to C10, C16 to C11, C17 to C12, C18 to C13, C19 to C14, C7 to C2, C8 to C3, C9 to C4, C10 to C5, C11 to C6, C12 to C7, C13 to C8, C14 to C9, IC1 to IC2, IC2 to IC3, IC3 to IC4, IC4 to IC5
Connections:
- net labels added: INTn, SCL, SDA
- wire segments 119 -> 97
Other:
- note added: "Ambient Light Sensor"
- note added: "PIR Signal Amplification & Conditioning"
- note removed: "Signal Conditioning"

Commit message: Migrated project/libraries to KiCad nightly build
Revision: 821668d96

Reason being the simulator feature and the better library management.
Parts:
- 1.3M1, 1.5M1, 10K1, 10K2, 10K3, 15M1, 15M2, 15M3, 15M4, 6.81K1, 619K1, 68.1K1, 68.1K2: symbol R -> device:R
- C1, C10, C11, C12, C13, C14, C2, C3, C4, C5, C6, C7, C8, C9: symbol C -> device:C
- D1, D2: symbol 1N4148X-TP -> 1N4148X-TP:1N4148X-TP
- IC1: symbol MAX44009EDT+T -> MAX44009EDT+T:MAX44009EDT+T
- IC2: symbol IRA-S210ST01 -> IRA-S210ST01:IRA-S210ST01
- IC3: symbol LPV802DGKT -> LPV802DGKT:LPV802DGKT
- IC4, IC5: symbol TLV3691IDCKR -> TLV3691IDCKR:TLV3691IDCKR
Changed lines of the file:
@@
-EESchema Schematic File Version 2
-LIBS:power
-LIBS:device
-LIBS:switches
-LIBS:relays
-LIBS:motors
-LIBS:transistors
-LIBS:conn
-LIBS:linear
-LIBS:regul
-LIBS:74xx
-LIBS:cmos4000
-LIBS:adc-dac
-LIBS:memory
-LIBS:xilinx
-LIBS:microcontrollers
-LIBS:dsp
-LIBS:microchip
-LIBS:analog_switches
-LIBS:motorola
-LIBS:texas
-LIBS:intel
-LIBS:audio
-LIBS:interface
-LIBS:digital-audio
-LIBS:philips
-LIBS:display
-LIBS:cypress
-LIBS:siliconi
-LIBS:opto
-LIBS:atmel
-LIBS:contrib
-LIBS:valves
-LIBS:LPV802DGKT
-LIBS:SI2323DS-T1-E3
-LIBS:1N4148X-TP
-LIBS:TLV3691IDCKR
-LIBS:IRA-S210ST01
-LIBS:CC2540F256RHAT
-LIBS:CC2541F256RHAR
-LIBS:CC2541F128RHAT
-LIBS:MAX44009EDT+T
+EESchema Schematic File Version 4
 LIBS:pir-cache
-EELAYER 25 0
+EELAYER 26 0
 EELAYER END
 $Descr A4 11693 8268
@@
 $EndDescr
 $Comp
-L VCC #PWR3
+L power:VCC #PWR3
 U 1 1 5A74E3A0
 P 1200 4700
@@
 $EndComp
 $Comp
-L R 619K1
+L device:R 619K1
 U 1 1 5A74E6D1
 P 1700 5050
@@
 $EndComp
 $Comp
-L C C1
+L device:C C1
 U 1 1 5A74F7D6
 P 2100 5400
@@
 $EndComp
 $Comp
-L C C2
+L device:C C2
 U 1 1 5A74F7DC
 P 2450 5400
@@
 $EndComp
 $Comp
-L C C3
+L device:C C3
 U 1 1 5A74F7E2
 P 2800 5400
@@
 $EndComp
 $Comp
-L C C4
+L device:C C4
 U 1 1 5A74F7E8
 P 3100 5400
@@
 $EndComp
 $Comp
-L C C5
+L device:C C5
 U 1 1 5A74F7EE
 P 3400 5400
@@
 $EndComp
 $Comp
-L C C6
+L device:C C6
 U 1 1 5A74FABF
 P 3700 5400
@@
 $EndComp
 $Comp
-L C C7
+L device:C C7
 U 1 1 5A74FAC5
 P 4000 5400
@@
 $EndComp
 $Comp
-L Earth #PWR4
+L power:Earth #PWR4
 U 1 1 5A74FD7A
 P 2100 5800
@@
 $EndComp
 $Comp
-L IRA-S210ST01 IC2
+L IRA-S210ST01:IRA-S210ST01 IC2
 U 1 1 5A74E937
 P 4850 5100
@@
 $EndComp
 $Comp
-L LPV802DGKT IC3
+L LPV802DGKT:LPV802DGKT IC3
 U 1 1 5A74EE7D
 P 6450 4550
@@
 $EndComp
 $Comp
-L VCC #PWR7
+L power:VCC #PWR7
 U 1 1 5A74F424
 P 7650 4450
@@
 $EndComp
 $Comp
-L R 1.3M1
+L device:R 1.3M1
 U 1 1 5A74FD88
 P 6100 5200
@@
 $EndComp
 $Comp
-L R 1.5M1
+L device:R 1.5M1
 U 1 1 5A75816E
 P 6000 4100
@@
 $EndComp
 $Comp
-L C C9
+L device:C C9
 U 1 1 5A75830A
 P 6000 3700
@@
 $EndComp
 $Comp
-L 1N4148X-TP D1
+L 1N4148X-TP:1N4148X-TP D1
 U 1 1 5A758478
 P 5700 3200
@@
 $EndComp
 $Comp
-L 1N4148X-TP D2
+L 1N4148X-TP:1N4148X-TP D2
 U 1 1 5A7585B5
 P 6300 2650
@@
 $EndComp
 $Comp
-L Earth #PWR6
+L power:Earth #PWR6
 U 1 1 5A7586B3
 P 5100 3700
@@
 $EndComp
 $Comp
-L R 6.81K1
+L device:R 6.81K1
 U 1 1 5A758706
 P 5100 2850
@@
 $EndComp
 $Comp
-L C C8
+L device:C C8
 U 1 1 5A759015
 P 5100 3400
@@
 PIR Sensor
 $Comp
-L C C10
+L device:C C10
 U 1 1 5A75C2C5
 P 6800 4100
@@
 $EndComp
 $Comp
-L R 68.1K1
+L device:R 68.1K1
 U 1 1 5A75C4C6
 P 7350 4100
@@
 $EndComp
 $Comp
-L TLV3691IDCKR IC4
+L TLV3691IDCKR:TLV3691IDCKR IC4
 U 1 1 5A75C81D
 P 9350 4100
@@
 $EndComp
 $Comp
-L TLV3691IDCKR IC5
+L TLV3691IDCKR:TLV3691IDCKR IC5
 U 1 1 5A75C9FD
 P 9350 5250
@@
 $EndComp
 $Comp
-L C C12
+L device:C C12
 U 1 1 5A75CE5D
 P 8000 3800
@@
 $EndComp
 $Comp
-L R 68.1K2
+L device:R 68.1K2
 U 1 1 5A75CF06
 P 8000 3450
@@
 $EndComp
 $Comp
-L VCC #PWR13
+L power:VCC #PWR13
 U 1 1 5A75E6F0
 P 10300 4250
@@
 $EndComp
 $Comp
-L VCC #PWR14
+L power:VCC #PWR14
 U 1 1 5A75E75B
 P 10300 5400
@@
 $EndComp
 $Comp
-L R 15M1
+L device:R 15M1
 U 1 1 5A75F02F
 P 8750 3800
@@
 $EndComp
 $Comp
-L R 15M2
+L device:R 15M2
 U 1 1 5A75F0D4
 P 8750 4500
@@
 $EndComp
 $Comp
-L R 15M3
+L device:R 15M3
 U 1 1 5A75F386
 P 8750 5050
@@
 $EndComp
 $Comp
-L R 15M4
+L device:R 15M4
 U 1 1 5A75F4BA
 P 8750 5600
@@
 $EndComp
 $Comp
-L VCC #PWR9
+L power:VCC #PWR9
 U 1 1 5A75F9AF
 P 8750 3400
@@
 $EndComp
 $Comp
-L Earth #PWR11
+L power:Earth #PWR11
 U 1 1 5A75FB22
 P 9300 4800
@@
 $EndComp
 $Comp
-L Earth #PWR12
+L power:Earth #PWR12
 U 1 1 5A75FC29
 P 9300 5800
@@
 $EndComp
 $Comp
-L Earth #PWR10
+L power:Earth #PWR10
 U 1 1 5A75FF6B
 P 8750 5800
@@
 $EndComp
 $Comp
-L C C13
+L device:C C13
 U 1 1 5A7618C9
 P 9100 4500
@@
 $EndComp
 $Comp
-L C C14
+L device:C C14
 U 1 1 5A761E88
 P 9100 5550
@@
 $EndComp
 $Comp
-L C C11
+L device:C C11
 U 1 1 5A7623E0
 P 7750 5500
@@
 $EndComp
 $Comp
-L Earth #PWR8
+L power:Earth #PWR8
 U 1 1 5A7624AD
 P 7750 5800
@@
 PIR_LOW
 $Comp
-L Earth #PWR2
+L power:Earth #PWR2
 U 1 1 5A76FBFD
 P 1200 2150
@@
 $EndComp
 $Comp
-L VCC #PWR1
+L power:VCC #PWR1
 U 1 1 5A76FC4F
 P 1200 1800
@@
 Connection ~ 1200 2050
 $Comp
-L MAX44009EDT+T IC1
+L MAX44009EDT+T:MAX44009EDT+T IC1
 U 1 1 5A76F6EB
 P 2100 2000
@@
 $EndComp
 $Comp
-L R 10K1
+L device:R 10K1
 U 1 1 5A770F59
 P 2800 1600
@@
 $EndComp
 $Comp
-L R 10K2
+L device:R 10K2
 U 1 1 5A77107B
 P 3050 1600
@@
 $EndComp
 $Comp
-L R 10K3
+L device:R 10K3
 U 1 1 5A771104
 P 3300 1600
@@
 $EndComp
 $Comp
-L VCC #PWR5
+L power:VCC #PWR5
 U 1 1 5A7712E7
 P 3050 1300

Commit message: Added E-Ink display
Connections:
- wire segments 97 -> 140
Changed lines of the file:
@@
 $Descr A4 11693 8268
 encoding utf-8
-Sheet 2 5
+Sheet 2 6
 Title ""
 Date ""
@@
 	1200 5050 1550 5050
 Wire Wire Line
-	1850 5050 4000 5050
+	1850 5050 2100 5050
 Wire Wire Line
 	2100 5050 2100 5250
@@
 Connection ~ 3700 5050
 Wire Wire Line
-	2100 5550 2100 5800
+	2100 5550 2100 5700
 Wire Wire Line
 	2450 5700 2450 5550
@@
 	4000 5700 4000 5550
 Connection ~ 3700 5700
-Connection ~ 4000 5050
 Connection ~ 4000 5700
 Wire Wire Line
@@
 	7650 4550 7650 4450
 Wire Wire Line
-	2100 5700 6400 5700
-Wire Wire Line
-	5650 4750 6450 4750
+	2100 5700 2450 5700
+Wire Wire Line
+	5650 4750 6100 4750
 Wire Wire Line
 	6450 4850 6400 4850
@@
 	5100 2700 5100 2650
 Wire Wire Line
-	5100 2650 5700 2650
+	5100 2650 5650 2650
 Wire Wire Line
 	6300 2650 6350 2650
 Wire Wire Line
-	6350 2650 6350 4550
+	6350 2650 6350 3200
 Wire Wire Line
 	6350 3200 6300 3200
@@
 	5700 3200 5650 3200
 Wire Wire Line
-	5650 2650 5650 4650
+	5650 2650 5650 3200
 Wire Wire Line
 	5650 3700 5850 3700
@@
 Connection ~ 5650 3700
 Wire Wire Line
-	6150 4100 6650 4100
+	6150 4100 6350 4100
 Connection ~ 6350 3700
 Wire Wire Line
@@
 	7800 4100 7500 4100
 Wire Wire Line
-	7800 3450 7800 4750
+	7800 3450 7800 3800
 Wire Wire Line
 	7800 4750 7550 4750
@@
 	8150 3450 8200 3450
 Wire Wire Line
-	8200 3450 8200 5450
+	8200 3450 8200 3800
 Wire Wire Line
 	8200 3800 8150 3800
@@
 	10250 5250 10400 5250
 Wire Wire Line
-	8750 3950 8750 4350
+	8750 3950 8750 4300
 Wire Wire Line
 	8750 5750 8750 5800
@@
 	8750 3650 8750 3400
 Wire Wire Line
-	8750 4300 9350 4300
+	8750 4300 9100 4300
 Connection ~ 8750 4300
 Wire Wire Line
-	8750 4650 8750 4900
+	8750 4650 8750 4850
 Wire Wire Line
 	9350 4200 9300 4200
@@
 	9350 5350 9300 5350
 Wire Wire Line
-	9300 5350 9300 5800
+	9300 5350 9300 5750
 Wire Wire Line
 	8200 5450 9350 5450
 Wire Wire Line
-	8750 5200 8750 5450
-Wire Wire Line
-	9300 4200 9300 4800
-Wire Wire Line
-	8750 5250 9350 5250
+	8750 5200 8750 5250
+Wire Wire Line
+	9300 4200 9300 4750
+Wire Wire Line
+	8750 5250 9100 5250
 Connection ~ 8750 5250
 Wire Wire Line
@@
 Connection ~ 9300 5750
 Wire Wire Line
-	7550 4850 8750 4850
+	7550 4850 7750 4850
 Connection ~ 8750 4850
 Wire Wire Line
@@
 	1600 1950 1200 1950
 Wire Wire Line
-	1200 1950 1200 2150
+	1200 1950 1200 2050
 Wire Wire Line
 	1600 2050 1200 2050
@@
 $EndComp
 Wire Wire Line
-	2600 1850 3550 1850
+	2600 1850 2800 1850
 Wire Wire Line
 	2800 1850 2800 1750
 Wire Wire Line
-	2600 1950 3800 1950
+	2600 1950 3050 1950
 Wire Wire Line
 	3050 1950 3050 1750
 Wire Wire Line
-	2600 2050 4050 2050
+	2600 2050 3300 2050
 Wire Wire Line
 	3300 2050 3300 1750
@@
 	2800 1450 2800 1400
 Wire Wire Line
-	2800 1400 3300 1400
-Wire Wire Line
-	3050 1300 3050 1450
+	2800 1400 3050 1400
+Wire Wire Line
+	3050 1300 3050 1400
 Connection ~ 3050 1400
 Wire Wire Line
 	3300 1400 3300 1450
+Wire Wire Line
+	2100 5050 2450 5050
+Wire Wire Line
+	2450 5050 2800 5050
+Wire Wire Line
+	2800 5050 3100 5050
+Wire Wire Line
+	3100 5050 3400 5050
+Wire Wire Line
+	3400 5050 3700 5050
+Wire Wire Line
+	3700 5050 4000 5050
+Wire Wire Line
+	2100 5700 2100 5800
+Wire Wire Line
+	2450 5700 2800 5700
+Wire Wire Line
+	2800 5700 3100 5700
+Wire Wire Line
+	3100 5700 3400 5700
+Wire Wire Line
+	3400 5700 3700 5700
+Wire Wire Line
+	3700 5700 4000 5700
+Wire Wire Line
+	4000 5700 4850 5700
+Wire Wire Line
+	6100 5700 6400 5700
+Wire Wire Line
+	5650 3200 5650 3700
+Wire Wire Line
+	6350 3200 6350 3700
+Wire Wire Line
+	5650 3700 5650 4100
+Wire Wire Line
+	6350 3700 6350 4100
+Wire Wire Line
+	6350 4100 6650 4100
+Wire Wire Line
+	6350 4100 6350 4550
+Wire Wire Line
+	5650 4100 5650 4650
+Wire Wire Line
+	4850 5700 6100 5700
+Wire Wire Line
+	6100 4750 6450 4750
+Wire Wire Line
+	7800 4100 7800 4750
+Wire Wire Line
+	7800 3800 7800 4100
+Wire Wire Line
+	8200 3800 8200 4100
+Wire Wire Line
+	8200 4100 8200 4650
+Wire Wire Line
+	8750 4300 8750 4350
+Wire Wire Line
+	8750 5250 8750 5450
+Wire Wire Line
+	9100 4300 9350 4300
+Wire Wire Line
+	9300 4750 9300 4800
+Wire Wire Line
+	9100 5250 9350 5250
+Wire Wire Line
+	9300 5750 9300 5800
+Wire Wire Line
+	8750 4850 8750 4900
+Wire Wire Line
+	7750 4850 8750 4850
+Wire Wire Line
+	8200 4650 8200 5450
+Wire Wire Line
+	5650 2650 5700 2650
+Wire Wire Line
+	1200 2050 1200 2150
+Wire Wire Line
+	3050 1950 3800 1950
+Wire Wire Line
+	2800 1850 3550 1850
+Wire Wire Line
+	3300 2050 4050 2050
+Wire Wire Line
+	3050 1400 3300 1400
+Wire Wire Line
+	3050 1400 3050 1450
 $EndSCHEMATC

Commit message: MCU change, again
STM32L0 had quite a big problem, common reference for the comparators.
Another minus was the missing SWO for debugging.

STM32L4 has floating point, and most importantly, has embedded OPAMPS!
This means I can directly plug in the filter to the analog inputs and
everything is software. 2 opamps and 2 comparators (if needed).
External circuitry would be minimal for the PIR sensor.

It also means that I can read with the embedded 12-bit ADC the
amplified values. Precision is not crucial, we are interested in dips
and swells.
Parts:
- removed D2: 1N4148X-TP, SODFL1608X70N, symbol 1N4148X-TP:1N4148X-TP
- removed IC4, IC5: TLV3691IDCKR, SOT65P210X110-5N, symbol TLV3691IDCKR:TLV3691IDCKR
- added C?: 3.3nF, symbol device:C
- C10: value 3.3μF -> 22μF
- C12: value 3.3μF -> 47nF
- C8: value 33μF -> 22μF
- C9: value 0.01μF -> 47nF
- renumbered 6.81K1 to 13k, 68.1K1 to 13k, 1.3M1 to 56k, 1.5M1 to 680k, 68.1K2 to 680k
Connections:
- net labels added: Ambient, PIR, PIR_HIGH_TH, PIR_LOW_TH
- net labels removed: INTn, PIR_HIGH, PIR_LOW
- wire segments 140 -> 86
