File: pcb/sensor.sch (KiCad schematic (older format))
At the start: 32 parts, among them IC1 MAX44009EDT+T, IC2 IRA-S210ST01, IC3 LPV802DGKT

Commit message: Sensor logic implemented using MCU opamps
Of the ST PIR design I use the first 2 stages only, so no comparators.
1st stage using OPAMP1
2nd stage using OPAMP2

OPAMP1 amplifies the sensor output around the DC component of the PIR
sensor.

OPAMP2 amplifies the stage 1 output around half of VCC.

The output is then passed differentially to ADC which gives a
difference between stage 2 output and VCC/2.

This can be later converted into real volts by using the internal
VREFINT of the MCU because VCC can be measured against it. ST has
some (hopefully) cool factory calibration feature to compensate
for temperature deviations of the ADC which makes all this
possible  without external sigma-delta ADC.

The ADC has analog window thresholds that can be used to trigger
interrupts when input is beyond threshold. This means it is
possible to set sensitivity by modifying this threshold instead
of playing with the OPAMP2 gain (which anyway has only 4 levels).

(Just wasted a whole fucking saturday on this...)
Parts:
- removed 15M1, 15M2, 15M3, 15M4, 680k: R, symbol device:R
- removed C10: 22μF, symbol device:C
- removed C11, C13, C14: 0.1μF, symbol device:C
- removed C12: 47nF, symbol device:C
- removed IC3: LPV802DGKT, SOP65P490X110-8N, symbol LPV802DGKT:LPV802DGKT
- added 13k? (x2): R, symbol device:R
- added C?: 22uF, symbol device:C
- added C?: 47nF, symbol device:C
Connections:
- net labels added: OPAMP1+, OPAMP1-, OPAMP1OUT, OPAMP2+, OPAMP2-, OPAMP2OUT
- net labels removed: PIR, PIR_HIGH_TH, PIR_LOW_TH
- wire segments 86 -> 67

Commit message: Renamed all components
Parts:
- removed 10K3, 13k: R, symbol device:R
- added R3: 10k, symbol device:R
- added R7: 13k, symbol device:R
- R1: renamed from 10K1; value R -> 10k
- R2: renamed from 10K2; value R -> 10k
- R4: renamed from 13k; value R -> 13k
- R5: renamed from 56k; value R -> 56k
- R6: renamed from 680k; value R -> 680k
- R8, R9: renamed from 13k?; value R -> 1M
- gave numbers to parts that had none: 3
Changed lines of the file:
@@
 LIBS:ab2_usb
 LIBS:ab2_xtal
+LIBS:pir-cache
 EELAYER 25 0
 EELAYER END
@@
 $EndDescr
 $Comp
-L power:VCC #PWR03
+L power:VCC #PWR3
 U 1 1 5A74E3A0
 P 1200 4700
-F 0 "#PWR03" H 1200 4550 50  0001 C CNN
+F 0 "#PWR3" H 1200 4550 50  0001 C CNN
 F 1 "VCC" H 1200 4850 50  0000 C CNN
 F 2 "" H 1200 4700 50  0001 C CNN
@@
 $EndComp
 $Comp
-L power:Earth #PWR04
+L power:Earth #PWR4
 U 1 1 5A74FD7A
 P 2100 5800
-F 0 "#PWR04" H 2100 5550 50  0001 C CNN
+F 0 "#PWR4" H 2100 5550 50  0001 C CNN
 F 1 "Earth" H 2100 5650 50  0001 C CNN
 F 2 "" H 2100 5800 50  0001 C CNN
@@
 $EndComp
 $Comp
-L device:R 56k
+L device:R R5
 U 1 1 5A74FD88
 P 5900 5200
-F 0 "56k" V 5980 5200 50  0000 C CNN
-F 1 "R" V 5900 5200 50  0000 C CNN
+F 0 "R5" V 5980 5200 50  0000 C CNN
+F 1 "56k" V 5900 5200 50  0000 C CNN
 F 2 "" V 5830 5200 50  0001 C CNN
 F 3 "" H 5900 5200 50  0001 C CNN
@@
 $EndComp
 $Comp
-L device:R 680k
+L device:R R6
 U 1 1 5A75816E
 P 6000 4100
-F 0 "680k" V 6080 4100 50  0000 C CNN
-F 1 "R" V 6000 4100 50  0000 C CNN
+F 0 "R6" V 6080 4100 50  0000 C CNN
+F 1 "680k" V 6000 4100 50  0000 C CNN
 F 2 "" V 5930 4100 50  0001 C CNN
 F 3 "" H 6000 4100 50  0001 C CNN
@@
 $EndComp
 $Comp
-L power:Earth #PWR06
+L power:Earth #PWR6
 U 1 1 5A7586B3
 P 5100 3700
-F 0 "#PWR06" H 5100 3450 50  0001 C CNN
+F 0 "#PWR6" H 5100 3450 50  0001 C CNN
 F 1 "Earth" H 5100 3550 50  0001 C CNN
 F 2 "" H 5100 3700 50  0001 C CNN
@@
 $EndComp
 $Comp
-L device:R 13k
+L device:R R4
 U 1 1 5A758706
 P 5100 2850
-F 0 "13k" V 5180 2850 50  0000 C CNN
-F 1 "R" V 5100 2850 50  0000 C CNN
+F 0 "R4" V 5180 2850 50  0000 C CNN
+F 1 "13k" V 5100 2850 50  0000 C CNN
 F 2 "" V 5030 2850 50  0001 C CNN
 F 3 "" H 5100 2850 50  0001 C CNN
@@
 	1200 5050 1200 4700
 $Comp
-L power:Earth #PWR02
+L power:Earth #PWR2
 U 1 1 5A76FBFD
 P 1200 2150
-F 0 "#PWR02" H 1200 1900 50  0001 C CNN
+F 0 "#PWR2" H 1200 1900 50  0001 C CNN
 F 1 "Earth" H 1200 2000 50  0001 C CNN
 F 2 "" H 1200 2150 50  0001 C CNN
@@
 $EndComp
 $Comp
-L power:VCC #PWR01
+L power:VCC #PWR1
 U 1 1 5A76FC4F
 P 1200 1800
-F 0 "#PWR01" H 1200 1650 50  0001 C CNN
+F 0 "#PWR1" H 1200 1650 50  0001 C CNN
 F 1 "VCC" H 1200 1950 50  0000 C CNN
 F 2 "" H 1200 1800 50  0001 C CNN
@@
 $EndComp
 $Comp
-L device:R 10K1
+L device:R R1
 U 1 1 5A770F59
 P 2800 1600
-F 0 "10K1" V 2880 1600 50  0000 C CNN
-F 1 "R" V 2800 1600 50  0000 C CNN
+F 0 "R1" V 2880 1600 50  0000 C CNN
+F 1 "10k" V 2800 1600 50  0000 C CNN
 F 2 "" V 2730 1600 50  0001 C CNN
 F 3 "" H 2800 1600 50  0001 C CNN
@@
 $EndComp
 $Comp
-L device:R 10K2
+L device:R R2
 U 1 1 5A77107B
 P 3050 1600
-F 0 "10K2" V 3130 1600 50  0000 C CNN
-F 1 "R" V 3050 1600 50  0000 C CNN
+F 0 "R2" V 3130 1600 50  0000 C CNN
+F 1 "10k" V 3050 1600 50  0000 C CNN
 F 2 "" V 2980 1600 50  0001 C CNN
 F 3 "" H 3050 1600 50  0001 C CNN
@@
 $EndComp
 $Comp
-L device:R 10K3
-U 1 1 5A771104
-P 3300 1600
-F 0 "10K3" V 3380 1600 50  0000 C CNN
-F 1 "R" V 3300 1600 50  0000 C CNN
-F 2 "" V 3230 1600 50  0001 C CNN
-F 3 "" H 3300 1600 50  0001 C CNN
-	1    3300 1600
-	1    0    0    -1
-$EndComp
-$Comp
-L power:VCC #PWR05
+L power:VCC #PWR5
 U 1 1 5A7712E7
 P 3050 1300
-F 0 "#PWR05" H 3050 1150 50  0001 C CNN
+F 0 "#PWR5" H 3050 1150 50  0001 C CNN
 F 1 "VCC" H 3050 1450 50  0000 C CNN
 F 2 "" H 3050 1300 50  0001 C CNN
@@
 Ambient
 $Comp
-L device:C C?
+L device:C C10
 U 1 1 5A80E859
 P 6200 5200
-F 0 "C?" H 6225 5300 50  0000 L CNN
+F 0 "C10" H 6225 5300 50  0000 L CNN
 F 1 "3.3nF" H 6225 5100 50  0000 L CNN
 F 2 "" H 6238 5050 50  0001 C CNN
@@
 OPAMP2-
 $Comp
-L device:C C?
+L device:C C11
 U 1 1 5A83B4D6
 P 7000 4150
-F 0 "C?" H 7025 4250 50  0000 L CNN
+F 0 "C11" H 7025 4250 50  0000 L CNN
 F 1 "22uF" H 7025 4050 50  0000 L CNN
 F 2 "" H 7038 4000 50  0001 C CNN
@@
 	0    1    1    0
 $EndComp
-$Comp
-L device:R 13k
-U 1 1 5A83B581
-P 7450 4150
-F 0 "13k" V 7530 4150 50  0000 C CNN
-F 1 "R" V 7450 4150 50  0000 C CNN
-F 2 "" V 7380 4150 50  0001 C CNN
-F 3 "" H 7450 4150 50  0001 C CNN
-	1    7450 4150
-	0    1    1    0
-$EndComp
 Wire Wire Line
 	6650 4550 6650 4150
@@
 	7600 4150 8350 4150
 $Comp
-L power:VCC #PWR?
+L power:VCC #PWR7
 U 1 1 5A83FC10
 P 8000 4500
-F 0 "#PWR?" H 8000 4350 50  0001 C CNN
+F 0 "#PWR7" H 8000 4350 50  0001 C CNN
 F 1 "VCC" H 8000 4650 50  0000 C CNN
 F 2 "" H 8000 4500 50  0001 C CNN
@@
 $EndComp
 $Comp
-L device:R 13k?
+L device:R R8
 U 1 1 5A83FDFF
 P 8000 4750
-F 0 "13k?" V 8080 4750 50  0000 C CNN
-F 1 "R" V 8000 4750 50  0000 C CNN
+F 0 "R8" V 8080 4750 50  0000 C CNN
+F 1 "1M" V 8000 4750 50  0000 C CNN
 F 2 "" V 7930 4750 50  0001 C CNN
 F 3 "" H 8000 4750 50  0001 C CNN
@@
 $EndComp
 $Comp
-L device:R 13k?
+L device:R R9
 U 1 1 5A83FF1B
 P 8000 5150
-F 0 "13k?" V 8080 5150 50  0000 C CNN
-F 1 "R" V 8000 5150 50  0000 C CNN
+F 0 "R9" V 8080 5150 50  0000 C CNN
+F 1 "1M" V 8000 5150 50  0000 C CNN
 F 2 "" V 7930 5150 50  0001 C CNN
 F 3 "" H 8000 5150 50  0001 C CNN
@@
 $EndComp
 $Comp
-L power:Earth #PWR?
+L power:Earth #PWR8
 U 1 1 5A83FF97
 P 8000 5400
-F 0 "#PWR?" H 8000 5150 50  0001 C CNN
+F 0 "#PWR8" H 8000 5150 50  0001 C CNN
 F 1 "Earth" H 8000 5250 50  0001 C CNN
 F 2 "" H 8000 5400 50  0001 C CNN
@@
 OPAMP2OUT
 $Comp
-L device:C C?
+L device:C C12
 U 1 1 5A840800
 P 8000 3900
-F 0 "C?" H 8025 4000 50  0000 L CNN
+F 0 "C12" H 8025 4000 50  0000 L CNN
 F 1 "47nF" H 8025 3800 50  0000 L CNN
 F 2 "" H 8038 3750 50  0001 C CNN
@@
 	8000 4050 8000 4150
 Connection ~ 8000 4150
+$Comp
+L device:R R3
+U 1 1 5A80F84C
+P 3300 1600
+F 0 "R3" V 3380 1600 50  0000 C CNN
+F 1 "10k" V 3300 1600 50  0000 C CNN
+F 2 "" V 3230 1600 50  0001 C CNN
+F 3 "" H 3300 1600 50  0001 C CNN
+	1    3300 1600
+	1    0    0    -1
+$EndComp
+$Comp
+L device:R R7
+U 1 1 5A80FE16
+P 7450 4150
+F 0 "R7" V 7530 4150 50  0000 C CNN
+F 1 "13k" V 7450 4150 50  0000 C CNN
+F 2 "" V 7380 4150 50  0001 C CNN
+F 3 "" H 7450 4150 50  0001 C CNN
+	1    7450 4150
+	0    1    1    0
+$EndComp
 $EndSCHEMATC

Commit message: Replaced original PIR symbol and ran ERC tests
Parts:
- removed IC2: IRA-S210ST01, IRA-S210ST01, symbol IRA-S210ST01:IRA-S210ST01
- added IC2: IRA-S210ST01, IRA-S210ST01, symbol IRA-S210ST01
Connections:
- wire segments 67 -> 68

Commit message: Added testpoints
Parts:
- added TP1, TP2, TP3, TP4, TP5, TP6, TP7, TP8, TP9: TEST, symbol TEST
- R1: renamed from 619K1; value R -> 0
- renumbered R9 to R10, R1 to R2, R2 to R3, R3 to R4, R4 to R5, R5 to R6, R6 to R7, R7 to R8, R8 to R9
Connections:
- wire segments 68 -> 85
Changed lines of the file:
@@
 $EndDescr
 $Comp
-L power:VCC #PWR01
+L power:VCC #PWR3
 U 1 1 5A74E3A0
 P 1200 4700
-F 0 "#PWR01" H 1200 4550 50  0001 C CNN
+F 0 "#PWR3" H 1200 4550 50  0001 C CNN
 F 1 "VCC" H 1200 4850 50  0000 C CNN
 F 2 "" H 1200 4700 50  0001 C CNN
@@
 $EndComp
 $Comp
-L device:R 619K1
+L device:R R1
 U 1 1 5A74E6D1
 P 1700 5050
-F 0 "619K1" V 1780 5050 50  0000 C CNN
-F 1 "R" V 1700 5050 50  0000 C CNN
+F 0 "R1" V 1780 5050 50  0000 C CNN
+F 1 "0" V 1700 5050 50  0000 C CNN
 F 2 "" V 1630 5050 50  0001 C CNN
 F 3 "" H 1700 5050 50  0001 C CNN
@@
 $EndComp
 $Comp
-L power:Earth #PWR02
+L power:Earth #PWR4
 U 1 1 5A74FD7A
 P 2100 5800
-F 0 "#PWR02" H 2100 5550 50  0001 C CNN
+F 0 "#PWR4" H 2100 5550 50  0001 C CNN
 F 1 "Earth" H 2100 5650 50  0001 C CNN
 F 2 "" H 2100 5800 50  0001 C CNN
@@
 $EndComp
 $Comp
-L device:R R5
+L device:R R6
 U 1 1 5A74FD88
 P 5900 5200
-F 0 "R5" V 5980 5200 50  0000 C CNN
+F 0 "R6" V 5980 5200 50  0000 C CNN
 F 1 "56k" V 5900 5200 50  0000 C CNN
 F 2 "" V 5830 5200 50  0001 C CNN
@@
 $EndComp
 $Comp
-L device:R R6
+L device:R R7
 U 1 1 5A75816E
 P 6000 4100
-F 0 "R6" V 6080 4100 50  0000 C CNN
+F 0 "R7" V 6080 4100 50  0000 C CNN
 F 1 "680k" V 6000 4100 50  0000 C CNN
 F 2 "" V 5930 4100 50  0001 C CNN
@@
 $EndComp
 $Comp
-L power:Earth #PWR03
+L power:Earth #PWR6
 U 1 1 5A7586B3
 P 5100 3700
-F 0 "#PWR03" H 5100 3450 50  0001 C CNN
+F 0 "#PWR6" H 5100 3450 50  0001 C CNN
 F 1 "Earth" H 5100 3550 50  0001 C CNN
 F 2 "" H 5100 3700 50  0001 C CNN
@@
 $EndComp
 $Comp
-L device:R R4
+L device:R R5
 U 1 1 5A758706
 P 5100 2850
-F 0 "R4" V 5180 2850 50  0000 C CNN
+F 0 "R5" V 5180 2850 50  0000 C CNN
 F 1 "13k" V 5100 2850 50  0000 C CNN
 F 2 "" V 5030 2850 50  0001 C CNN
@@
 PIR Signal Amplification & Conditioning
 $Comp
-L power:Earth #PWR04
+L power:Earth #PWR2
 U 1 1 5A76FBFD
 P 1200 2150
-F 0 "#PWR04" H 1200 1900 50  0001 C CNN
+F 0 "#PWR2" H 1200 1900 50  0001 C CNN
 F 1 "Earth" H 1200 2000 50  0001 C CNN
 F 2 "" H 1200 2150 50  0001 C CNN
@@
 $EndComp
 $Comp
-L power:VCC #PWR05
+L power:VCC #PWR1
 U 1 1 5A76FC4F
 P 1200 1800
-F 0 "#PWR05" H 1200 1650 50  0001 C CNN
+F 0 "#PWR1" H 1200 1650 50  0001 C CNN
 F 1 "VCC" H 1200 1950 50  0000 C CNN
 F 2 "" H 1200 1800 50  0001 C CNN
@@
 $EndComp
 $Comp
-L device:R R1
+L device:R R2
 U 1 1 5A770F59
 P 2800 1600
-F 0 "R1" V 2880 1600 50  0000 C CNN
+F 0 "R2" V 2880 1600 50  0000 C CNN
 F 1 "10k" V 2800 1600 50  0000 C CNN
 F 2 "" V 2730 1600 50  0001 C CNN
@@
 $EndComp
 $Comp
-L device:R R2
+L device:R R3
 U 1 1 5A77107B
 P 3050 1600
-F 0 "R2" V 3130 1600 50  0000 C CNN
+F 0 "R3" V 3130 1600 50  0000 C CNN
 F 1 "10k" V 3050 1600 50  0000 C CNN
 F 2 "" V 2980 1600 50  0001 C CNN
@@
 $EndComp
 $Comp
-L power:VCC #PWR06
+L power:VCC #PWR5
 U 1 1 5A7712E7
 P 3050 1300
-F 0 "#PWR06" H 3050 1150 50  0001 C CNN
+F 0 "#PWR5" H 3050 1150 50  0001 C CNN
 F 1 "VCC" H 3050 1450 50  0000 C CNN
 F 2 "" H 3050 1300 50  0001 C CNN
@@
 Text Notes 2500 1400 2    60   ~ 0
 Ambient Light Sensor
-Text HLabel 3550 1850 2    60   Input ~ 0
+Text HLabel 4050 1850 2    60   Input ~ 0
 SDA
-Text HLabel 3800 1950 2    60   Input ~ 0
+Text HLabel 4050 1950 2    60   Input ~ 0
 SCL
 Text HLabel 4050 2050 2    60   Output ~ 0
@@
 $EndComp
 $Comp
-L power:VCC #PWR07
+L power:VCC #PWR7
 U 1 1 5A83FC10
 P 8000 4500
-F 0 "#PWR07" H 8000 4350 50  0001 C CNN
+F 0 "#PWR7" H 8000 4350 50  0001 C CNN
 F 1 "VCC" H 8000 4650 50  0000 C CNN
 F 2 "" H 8000 4500 50  0001 C CNN
@@
 $EndComp
 $Comp
-L device:R R8
+L device:R R9
 U 1 1 5A83FDFF
 P 8000 4750
-F 0 "R8" V 8080 4750 50  0000 C CNN
+F 0 "R9" V 8080 4750 50  0000 C CNN
 F 1 "1M" V 8000 4750 50  0000 C CNN
 F 2 "" V 7930 4750 50  0001 C CNN
@@
 $EndComp
 $Comp
-L device:R R9
+L device:R R10
 U 1 1 5A83FF1B
 P 8000 5150
-F 0 "R9" V 8080 5150 50  0000 C CNN
+F 0 "R10" V 8080 5150 50  0000 C CNN
 F 1 "1M" V 8000 5150 50  0000 C CNN
 F 2 "" V 7930 5150 50  0001 C CNN
@@
 $EndComp
 $Comp
-L power:Earth #PWR08
+L power:Earth #PWR8
 U 1 1 5A83FF97
 P 8000 5400
-F 0 "#PWR08" H 8000 5150 50  0001 C CNN
+F 0 "#PWR8" H 8000 5150 50  0001 C CNN
 F 1 "Earth" H 8000 5250 50  0001 C CNN
 F 2 "" H 8000 5400 50  0001 C CNN
@@
 $EndComp
 $Comp
-L device:R R3
+L device:R R4
 U 1 1 5A80F84C
 P 3300 1600
-F 0 "R3" V 3380 1600 50  0000 C CNN
+F 0 "R4" V 3380 1600 50  0000 C CNN
 F 1 "10k" V 3300 1600 50  0000 C CNN
 F 2 "" V 3230 1600 50  0001 C CNN
@@
 $EndComp
 $Comp
-L device:R R7
+L device:R R8
 U 1 1 5A80FE16
 P 7450 4150
-F 0 "R7" V 7530 4150 50  0000 C CNN
+F 0 "R8" V 7530 4150 50  0000 C CNN
 F 1 "13k" V 7450 4150 50  0000 C CNN
 F 2 "" V 7380 4150 50  0001 C CNN
@@
 Connection ~ 1200 2050
 Wire Wire Line
-	2600 1850 3550 1850
+	2600 1850 4050 1850
 Wire Wire Line
 	2800 1850 2800 1750
 Wire Wire Line
-	2600 1950 3800 1950
+	2600 1950 4050 1950
 Wire Wire Line
 	3050 1950 3050 1750
@@
 	6200 5700 6200 5350
 Wire Wire Line
-	6650 4550 6650 4150
+	6650 4150 6650 5350
 Wire Wire Line
 	6650 4150 6850 4150
@@
 	5650 5350 5650 4750
 Connection ~ 5900 4750
+$Comp
+L TEST TP4
+U 1 1 5A836267
+P 6900 5250
+F 0 "TP4" H 6900 5550 50  0000 C BNN
+F 1 "TEST" H 6900 5500 50  0000 C CNN
+F 2 "" H 6900 5250 50  0001 C CNN
+F 3 "" H 6900 5250 50  0001 C CNN
+	1    6900 5250
+	1    0    0    -1
+$EndComp
+$Comp
+L TEST TP5
+U 1 1 5A836312
+P 7100 5250
+F 0 "TP5" H 7100 5550 50  0000 C BNN
+F 1 "TEST" H 7100 5500 50  0000 C CNN
+F 2 "" H 7100 5250 50  0001 C CNN
+F 3 "" H 7100 5250 50  0001 C CNN
+	1    7100 5250
+	1    0    0    -1
+$EndComp
+$Comp
+L TEST TP6
+U 1 1 5A836377
+P 7300 5250
+F 0 "TP6" H 7300 5550 50  0000 C BNN
+F 1 "TEST" H 7300 5500 50  0000 C CNN
+F 2 "" H 7300 5250 50  0001 C CNN
+F 3 "" H 7300 5250 50  0001 C CNN
+	1    7300 5250
+	1    0    0    -1
+$EndComp
+Wire Wire Line
+	6650 5350 6900 5350
+Wire Wire Line
+	6900 5350 6900 5250
+Wire Wire Line
+	6600 4650 6600 5400
+Wire Wire Line
+	6600 5400 7100 5400
+Wire Wire Line
+	7100 5400 7100 5250
+Connection ~ 6600 4650
+Wire Wire Line
+	6550 4750 6550 5450
+Wire Wire Line
+	6550 5450 7300 5450
+Wire Wire Line
+	7300 5450 7300 5250
+Connection ~ 6550 4750
+$Comp
+L TEST TP7
+U 1 1 5A83656F
+P 7500 5250
+F 0 "TP7" H 7500 5550 50  0000 C BNN
+F 1 "TEST" H 7500 5500 50  0000 C CNN
+F 2 "" H 7500 5250 50  0001 C CNN
+F 3 "" H 7500 5250 50  0001 C CNN
+	1    7500 5250
+	1    0    0    -1
+$EndComp
+$Comp
+L TEST TP8
+U 1 1 5A8365D8
+P 7700 5250
+F 0 "TP8" H 7700 5550 50  0000 C BNN
+F 1 "TEST" H 7700 5500 50  0000 C CNN
+F 2 "" H 7700 5250 50  0001 C CNN
+F 3 "" H 7700 5250 50  0001 C CNN
+	1    7700 5250
+	1    0    0    -1
+$EndComp
+Wire Wire Line
+	7500 5250 7500 5650
+Wire Wire Line
+	7500 5650 8300 5650
+Wire Wire Line
+	8300 5650 8300 4150
+Connection ~ 8300 4150
+Wire Wire Line
+	7700 5250 7700 5600
+Wire Wire Line
+	7700 5600 8200 5600
+Wire Wire Line
+	8200 5600 8200 4950
+Connection ~ 8200 4950
+$Comp
+L TEST TP9
+U 1 1 5A83691A
+P 8150 3600
+F 0 "TP9" H 8150 3900 50  0000 C BNN
+F 1 "TEST" H 8150 3850 50  0000 C CNN
+F 2 "" H 8150 3600 50  0001 C CNN
+F 3 "" H 8150 3600 50  0001 C CNN
+	1    8150 3600
+	1    0    0    -1
+$EndComp
+$Comp
+L TEST TP1
+U 1 1 5A836F34
+P 3600 1650
+F 0 "TP1" H 3600 1950 50  0000 C BNN
+F 1 "TEST" H 3600 1900 50  0000 C CNN
+F 2 "" H 3600 1650 50  0001 C CNN
+F 3 "" H 3600 1650 50  0001 C CNN
+	1    3600 1650
+	1    0    0    -1
+$EndComp
+$Comp
+L TEST TP2
+U 1 1 5A837228
+P 3800 1650
+F 0 "TP2" H 3800 1950 50  0000 C BNN
+F 1 "TEST" H 3800 1900 50  0000 C CNN
+F 2 "" H 3800 1650 50  0001 C CNN
+F 3 "" H 3800 1650 50  0001 C CNN
+	1    3800 1650
+	1    0    0    -1
+$EndComp
+Wire Wire Line
+	3600 1650 3600 1850
+Connection ~ 3600 1850
+$Comp
+L TEST TP3
+U 1 1 5A83743E
+P 4000 1650
+F 0 "TP3" H 4000 1950 50  0000 C BNN
+F 1 "TEST" H 4000 1900 50  0000 C CNN
+F 2 "" H 4000 1650 50  0001 C CNN
+F 3 "" H 4000 1650 50  0001 C CNN
+	1    4000 1650
+	1    0    0    -1
+$EndComp
+Wire Wire Line
+	3800 1650 3800 1950
+Connection ~ 3800 1950
+Wire Wire Line
+	4000 1650 4000 2050
+Connection ~ 4000 2050
 $EndSCHEMATC

Commit message: CvPcb crashes every time on launch
This commit saves work just before trying out nightly kicad-git.
Connections:
- wire segments 85 -> 86
Other:
- moved on the sheet: TP9
Changed lines of the file:
@@
 $EndDescr
 $Comp
-L power:VCC #PWR3
+L power:VCC #PWR01
 U 1 1 5A74E3A0
 P 1200 4700
-F 0 "#PWR3" H 1200 4550 50  0001 C CNN
+F 0 "#PWR01" H 1200 4550 50  0001 C CNN
 F 1 "VCC" H 1200 4850 50  0000 C CNN
 F 2 "" H 1200 4700 50  0001 C CNN
@@
 $EndComp
 $Comp
-L power:Earth #PWR4
+L power:Earth #PWR02
 U 1 1 5A74FD7A
 P 2100 5800
-F 0 "#PWR4" H 2100 5550 50  0001 C CNN
+F 0 "#PWR02" H 2100 5550 50  0001 C CNN
 F 1 "Earth" H 2100 5650 50  0001 C CNN
 F 2 "" H 2100 5800 50  0001 C CNN
@@
 $EndComp
 $Comp
-L power:Earth #PWR6
+L power:Earth #PWR03
 U 1 1 5A7586B3
 P 5100 3700
-F 0 "#PWR6" H 5100 3450 50  0001 C CNN
+F 0 "#PWR03" H 5100 3450 50  0001 C CNN
 F 1 "Earth" H 5100 3550 50  0001 C CNN
 F 2 "" H 5100 3700 50  0001 C CNN
@@
 PIR Signal Amplification & Conditioning
 $Comp
-L power:Earth #PWR2
+L power:Earth #PWR04
 U 1 1 5A76FBFD
 P 1200 2150
-F 0 "#PWR2" H 1200 1900 50  0001 C CNN
+F 0 "#PWR04" H 1200 1900 50  0001 C CNN
 F 1 "Earth" H 1200 2000 50  0001 C CNN
 F 2 "" H 1200 2150 50  0001 C CNN
@@
 $EndComp
 $Comp
-L power:VCC #PWR1
+L power:VCC #PWR05
 U 1 1 5A76FC4F
 P 1200 1800
-F 0 "#PWR1" H 1200 1650 50  0001 C CNN
+F 0 "#PWR05" H 1200 1650 50  0001 C CNN
 F 1 "VCC" H 1200 1950 50  0000 C CNN
 F 2 "" H 1200 1800 50  0001 C CNN
@@
 $EndComp
 $Comp
-L power:VCC #PWR5
+L power:VCC #PWR06
 U 1 1 5A7712E7
 P 3050 1300
-F 0 "#PWR5" H 3050 1150 50  0001 C CNN
+F 0 "#PWR06" H 3050 1150 50  0001 C CNN
 F 1 "VCC" H 3050 1450 50  0000 C CNN
 F 2 "" H 3050 1300 50  0001 C CNN
@@
 $EndComp
 $Comp
-L power:VCC #PWR7
+L power:VCC #PWR07
 U 1 1 5A83FC10
 P 8000 4500
-F 0 "#PWR7" H 8000 4350 50  0001 C CNN
+F 0 "#PWR07" H 8000 4350 50  0001 C CNN
 F 1 "VCC" H 8000 4650 50  0000 C CNN
 F 2 "" H 8000 4500 50  0001 C CNN
@@
 $EndComp
 $Comp
-L power:Earth #PWR8
+L power:Earth #PWR08
 U 1 1 5A83FF97
 P 8000 5400
-F 0 "#PWR8" H 8000 5150 50  0001 C CNN
+F 0 "#PWR08" H 8000 5150 50  0001 C CNN
 F 1 "Earth" H 8000 5250 50  0001 C CNN
 F 2 "" H 8000 5400 50  0001 C CNN
@@
 L TEST TP9
 U 1 1 5A83691A
-P 8150 3600
-F 0 "TP9" H 8150 3900 50  0000 C BNN
-F 1 "TEST" H 8150 3850 50  0000 C CNN
-F 2 "" H 8150 3600 50  0001 C CNN
-F 3 "" H 8150 3600 50  0001 C CNN
-	1    8150 3600
+P 8150 3550
+F 0 "TP9" H 8150 3850 50  0000 C BNN
+F 1 "TEST" H 8150 3800 50  0000 C CNN
+F 2 "" H 8150 3550 50  0001 C CNN
+F 3 "" H 8150 3550 50  0001 C CNN
+	1    8150 3550
 	1    0    0    -1
 $EndComp
@@
 	4000 1650 4000 2050
 Connection ~ 4000 2050
+Wire Wire Line
+	8150 3550 8150 3600
+Connection ~ 8150 3600
 $EndSCHEMATC
