File: pcb/sensor.sch (KiCad schematic (older format))
At the start: 34 parts, among them IC1 MAX44009EDT+T, IC2 IRA-S210ST01

Commit message: Assigned footprints to all components
Parts:
- C1, C10, C11, C12, C2, C3, C4, C5, C6, C7, C8, C9: footprint (none) -> Capacitors_SMD:C_1206
- D1: footprint SODFL1608X70N -> Air_Coils_SML_NEOSID:Neosid_Air-Coil_SML_6-10turn_HDM0431A-HDM1031A
- IC1: footprint SON65P200X200X65-7N -> MAX44009EDT+T:SON65P200X200X65-7N
- IC2: footprint IRA-S210ST01 -> IRA-S210ST01:IRA-S210ST01
- R1, R10, R2, R3, R4, R5, R6, R7, R8, R9: footprint (none) -> Resistors_SMD:R_1210
- TP1, TP2, TP3, TP4, TP5, TP6, TP7, TP8, TP9: footprint (none) -> Measurement_Points:Measurement_Point_Round-TH_Small
Changed lines of the file:
@@
 F 0 "R1" V 1780 5050 50  0000 C CNN
 F 1 "0" V 1700 5050 50  0000 C CNN
-F 2 "" V 1630 5050 50  0001 C CNN
+F 2 "Resistors_SMD:R_1210" V 1630 5050 50  0001 C CNN
 F 3 "" H 1700 5050 50  0001 C CNN
 	1    1700 5050
@@
 F 0 "C1" H 2125 5500 50  0000 L CNN
 F 1 "100μF" H 2125 5300 50  0000 L CNN
-F 2 "" H 2138 5250 50  0001 C CNN
+F 2 "Capacitors_SMD:C_1206" H 2138 5250 50  0001 C CNN
 F 3 "" H 2100 5400 50  0001 C CNN
 	1    2100 5400
@@
 F 0 "C2" H 2475 5500 50  0000 L CNN
 F 1 "10μF" H 2475 5300 50  0000 L CNN
-F 2 "" H 2488 5250 50  0001 C CNN
+F 2 "Capacitors_SMD:C_1206" H 2488 5250 50  0001 C CNN
 F 3 "" H 2450 5400 50  0001 C CNN
 	1    2450 5400
@@
 F 0 "C3" H 2825 5500 50  0000 L CNN
 F 1 "1μF" H 2825 5300 50  0000 L CNN
-F 2 "" H 2838 5250 50  0001 C CNN
+F 2 "Capacitors_SMD:C_1206" H 2838 5250 50  0001 C CNN
 F 3 "" H 2800 5400 50  0001 C CNN
 	1    2800 5400
@@
 F 0 "C4" H 3125 5500 50  0000 L CNN
 F 1 "0.1μF" H 3125 5300 50  0000 L CNN
-F 2 "" H 3138 5250 50  0001 C CNN
+F 2 "Capacitors_SMD:C_1206" H 3138 5250 50  0001 C CNN
 F 3 "" H 3100 5400 50  0001 C CNN
 	1    3100 5400
@@
 F 0 "C5" H 3425 5500 50  0000 L CNN
 F 1 "0.01μF" H 3425 5300 50  0000 L CNN
-F 2 "" H 3438 5250 50  0001 C CNN
+F 2 "Capacitors_SMD:C_1206" H 3438 5250 50  0001 C CNN
 F 3 "" H 3400 5400 50  0001 C CNN
 	1    3400 5400
@@
 F 0 "C6" H 3725 5500 50  0000 L CNN
 F 1 "1000pF" H 3725 5300 50  0000 L CNN
-F 2 "" H 3738 5250 50  0001 C CNN
+F 2 "Capacitors_SMD:C_1206" H 3738 5250 50  0001 C CNN
 F 3 "" H 3700 5400 50  0001 C CNN
 	1    3700 5400
@@
 F 0 "C7" H 4025 5500 50  0000 L CNN
 F 1 "100pF" H 4025 5300 50  0000 L CNN
-F 2 "" H 4038 5250 50  0001 C CNN
+F 2 "Capacitors_SMD:C_1206" H 4038 5250 50  0001 C CNN
 F 3 "" H 4000 5400 50  0001 C CNN
 	1    4000 5400
@@
 F 0 "R6" V 5980 5200 50  0000 C CNN
 F 1 "56k" V 5900 5200 50  0000 C CNN
-F 2 "" V 5830 5200 50  0001 C CNN
+F 2 "Resistors_SMD:R_1210" V 5830 5200 50  0001 C CNN
 F 3 "" H 5900 5200 50  0001 C CNN
 	1    5900 5200
@@
 F 0 "R7" V 6080 4100 50  0000 C CNN
 F 1 "680k" V 6000 4100 50  0000 C CNN
-F 2 "" V 5930 4100 50  0001 C CNN
+F 2 "Resistors_SMD:R_1210" V 5930 4100 50  0001 C CNN
 F 3 "" H 6000 4100 50  0001 C CNN
 	1    6000 4100
@@
 F 0 "C9" H 6025 3800 50  0000 L CNN
 F 1 "47nF" H 6025 3600 50  0000 L CNN
-F 2 "" H 6038 3550 50  0001 C CNN
+F 2 "Capacitors_SMD:C_1206" H 6038 3550 50  0001 C CNN
 F 3 "" H 6000 3700 50  0001 C CNN
 	1    6000 3700
@@
 F 0 "D1" H 6000 3350 50  0000 C CNN
 F 1 "1N4148X-TP" H 6000 3050 50  0000 C CNN
-F 2 "SODFL1608X70N" H 6000 2950 50  0001 C CNN
+F 2 "Air_Coils_SML_NEOSID:Neosid_Air-Coil_SML_6-10turn_HDM0431A-HDM1031A" H 6000 2950 50  0001 C CNN
 F 3 "http://www.mouser.com/ds/2/258/1N4148X(SOD-523)-349105.pdf" H 6000 2850 50  0001 C CNN
 F 4 "Diodes - General Purpose, Power, Switching 150mA 75V" H 6000 2750 50  0001 C CNN "Description"
@@
 F 0 "R5" V 5180 2850 50  0000 C CNN
 F 1 "13k" V 5100 2850 50  0000 C CNN
-F 2 "" V 5030 2850 50  0001 C CNN
+F 2 "Resistors_SMD:R_1210" V 5030 2850 50  0001 C CNN
 F 3 "" H 5100 2850 50  0001 C CNN
 	1    5100 2850
@@
 F 0 "C8" H 5125 3500 50  0000 L CNN
 F 1 "22μF" H 5125 3300 50  0000 L CNN
-F 2 "" H 5138 3250 50  0001 C CNN
+F 2 "Capacitors_SMD:C_1206" H 5138 3250 50  0001 C CNN
 F 3 "" H 5100 3400 50  0001 C CNN
 	1    5100 3400
@@
 F 0 "IC1" H 2100 2300 50  0000 C CNN
 F 1 "MAX44009EDT+T" H 2100 1800 50  0000 C CNN
-F 2 "SON65P200X200X65-7N" H 2600 1450 50  0001 C CNN
+F 2 "MAX44009EDT+T:SON65P200X200X65-7N" H 2600 1450 50  0001 C CNN
 F 3 "https://componentsearchengine.com/Datasheets/2/MAX44009EDT T.pdf" H 2600 1350 50  0001 C CNN
 F 4 "Ambient Light Sensor with ADC OTDFN6 Maxim MAX44009EDT+T, Light Sensor IC, Light to Serial I2C 1.7  3.6 V 6-Pin UTDFN" H 2600 1250 50  0001 C CNN "Description"
@@
 F 0 "R2" V 2880 1600 50  0000 C CNN
 F 1 "10k" V 2800 1600 50  0000 C CNN
-F 2 "" V 2730 1600 50  0001 C CNN
+F 2 "Resistors_SMD:R_1210" V 2730 1600 50  0001 C CNN
 F 3 "" H 2800 1600 50  0001 C CNN
 	1    2800 1600
@@
 F 0 "R3" V 3130 1600 50  0000 C CNN
 F 1 "10k" V 3050 1600 50  0000 C CNN
-F 2 "" V 2980 1600 50  0001 C CNN
+F 2 "Resistors_SMD:R_1210" V 2980 1600 50  0001 C CNN
 F 3 "" H 3050 1600 50  0001 C CNN
 	1    3050 1600
@@
 F 0 "C10" H 6225 5300 50  0000 L CNN
 F 1 "3.3nF" H 6225 5100 50  0000 L CNN
-F 2 "" H 6238 5050 50  0001 C CNN
+F 2 "Capacitors_SMD:C_1206" H 6238 5050 50  0001 C CNN
 F 3 "" H 6200 5200 50  0001 C CNN
 	1    6200 5200
@@
 F 0 "C11" H 7025 4250 50  0000 L CNN
 F 1 "22uF" H 7025 4050 50  0000 L CNN
-F 2 "" H 7038 4000 50  0001 C CNN
+F 2 "Capacitors_SMD:C_1206" H 7038 4000 50  0001 C CNN
 F 3 "" H 7000 4150 50  0001 C CNN
 	1    7000 4150
@@
 F 0 "R9" V 8080 4750 50  0000 C CNN
 F 1 "1M" V 8000 4750 50  0000 C CNN
-F 2 "" V 7930 4750 50  0001 C CNN
+F 2 "Resistors_SMD:R_1210" V 7930 4750 50  0001 C CNN
 F 3 "" H 8000 4750 50  0001 C CNN
 	1    8000 4750
@@
 F 0 "R10" V 8080 5150 50  0000 C CNN
 F 1 "1M" V 8000 5150 50  0000 C CNN
-F 2 "" V 7930 5150 50  0001 C CNN
+F 2 "Resistors_SMD:R_1210" V 7930 5150 50  0001 C CNN
 F 3 "" H 8000 5150 50  0001 C CNN
 	1    8000 5150
@@
 F 0 "C12" H 8025 4000 50  0000 L CNN
 F 1 "47nF" H 8025 3800 50  0000 L CNN
-F 2 "" H 8038 3750 50  0001 C CNN
+F 2 "Capacitors_SMD:C_1206" H 8038 3750 50  0001 C CNN
 F 3 "" H 8000 3900 50  0001 C CNN
 	1    8000 3900
@@
 F 0 "R4" V 3380 1600 50  0000 C CNN
 F 1 "10k" V 3300 1600 50  0000 C CNN
-F 2 "" V 3230 1600 50  0001 C CNN
+F 2 "Resistors_SMD:R_1210" V 3230 1600 50  0001 C CNN
 F 3 "" H 3300 1600 50  0001 C CNN
 	1    3300 1600
@@
 F 0 "R8" V 7530 4150 50  0000 C CNN
 F 1 "13k" V 7450 4150 50  0000 C CNN
-F 2 "" V 7380 4150 50  0001 C CNN
+F 2 "Resistors_SMD:R_1210" V 7380 4150 50  0001 C CNN
 F 3 "" H 7450 4150 50  0001 C CNN
 	1    7450 4150
@@
 F 0 "IC2" H 4850 5300 50  0000 L CNN
 F 1 "IRA-S210ST01" H 4600 5200 50  0000 L CNN
-F 2 "IRA-S210ST01" H 5300 5150 50  0001 L CNN
+F 2 "IRA-S210ST01:IRA-S210ST01" H 5300 5150 50  0001 L CNN
 F 3 "https://www.murata.com/~/media/webrenewal/products/sensor/infrared/datasheet_pir.ashx?la=en" H 5300 5050 50  0001 L CNN
 F 4 "Air Purge Collar" H 5300 4950 50  0001 L CNN "Description"
@@
 F 0 "TP4" H 6900 5550 50  0000 C BNN
 F 1 "TEST" H 6900 5500 50  0000 C CNN
-F 2 "" H 6900 5250 50  0001 C CNN
+F 2 "Measurement_Points:Measurement_Point_Round-TH_Small" H 6900 5250 50  0001 C CNN
 F 3 "" H 6900 5250 50  0001 C CNN
 	1    6900 5250
@@
 F 0 "TP5" H 7100 5550 50  0000 C BNN
 F 1 "TEST" H 7100 5500 50  0000 C CNN
-F 2 "" H 7100 5250 50  0001 C CNN
+F 2 "Measurement_Points:Measurement_Point_Round-TH_Small" H 7100 5250 50  0001 C CNN
 F 3 "" H 7100 5250 50  0001 C CNN
 	1    7100 5250
@@
 F 0 "TP6" H 7300 5550 50  0000 C BNN
 F 1 "TEST" H 7300 5500 50  0000 C CNN
-F 2 "" H 7300 5250 50  0001 C CNN
+F 2 "Measurement_Points:Measurement_Point_Round-TH_Small" H 7300 5250 50  0001 C CNN
 F 3 "" H 7300 5250 50  0001 C CNN
 	1    7300 5250
@@
 F 0 "TP7" H 7500 5550 50  0000 C BNN
 F 1 "TEST" H 7500 5500 50  0000 C CNN
-F 2 "" H 7500 5250 50  0001 C CNN
+F 2 "Measurement_Points:Measurement_Point_Round-TH_Small" H 7500 5250 50  0001 C CNN
 F 3 "" H 7500 5250 50  0001 C CNN
 	1    7500 5250
@@
 F 0 "TP8" H 7700 5550 50  0000 C BNN
 F 1 "TEST" H 7700 5500 50  0000 C CNN
-F 2 "" H 7700 5250 50  0001 C CNN
+F 2 "Measurement_Points:Measurement_Point_Round-TH_Small" H 7700 5250 50  0001 C CNN
 F 3 "" H 7700 5250 50  0001 C CNN
 	1    7700 5250
@@
 F 0 "TP9" H 8150 3850 50  0000 C BNN
 F 1 "TEST" H 8150 3800 50  0000 C CNN
-F 2 "" H 8150 3550 50  0001 C CNN
+F 2 "Measurement_Points:Measurement_Point_Round-TH_Small" H 8150 3550 50  0001 C CNN
 F 3 "" H 8150 3550 50  0001 C CNN
 	1    8150 3550
@@
 F 0 "TP1" H 3600 1950 50  0000 C BNN
 F 1 "TEST" H 3600 1900 50  0000 C CNN
-F 2 "" H 3600 1650 50  0001 C CNN
+F 2 "Measurement_Points:Measurement_Point_Round-TH_Small" H 3600 1650 50  0001 C CNN
 F 3 "" H 3600 1650 50  0001 C CNN
 	1    3600 1650
@@
 F 0 "TP2" H 3800 1950 50  0000 C BNN
 F 1 "TEST" H 3800 1900 50  0000 C CNN
-F 2 "" H 3800 1650 50  0001 C CNN
+F 2 "Measurement_Points:Measurement_Point_Round-TH_Small" H 3800 1650 50  0001 C CNN
 F 3 "" H 3800 1650 50  0001 C CNN
 	1    3800 1650
@@
 F 0 "TP3" H 4000 1950 50  0000 C BNN
 F 1 "TEST" H 4000 1900 50  0000 C CNN
-F 2 "" H 4000 1650 50  0001 C CNN
+F 2 "Measurement_Points:Measurement_Point_Round-TH_Small" H 4000 1650 50  0001 C CNN
 F 3 "" H 4000 1650 50  0001 C CNN
 	1    4000 1650
