File: pcb/sensor.sch (KiCad schematic (older format))
At the start: 34 parts, among them IC1 MAX44009EDT+T, IC2 IRA-S210ST01

Commit message: Reassigned some footprints, added some libraries
Normally I can start working on PCB.
Parts:
- added C41: 0.1uF, Capacitors_SMD:C_1206, symbol device:C
- added JP4: Jumper, Pin_Headers:Pin_Header_Straight_1x02_Pitch2.54mm, symbol Jumper
- R1, R10, R2, R3, R4, R5, R6, R7, R8, R9: footprint Resistors_SMD:R_1210 -> Resistors_SMD:R_1206
Connections:
- wire segments 86 -> 89
Other:
- moved on the sheet: R2, R3, R4, TP1, TP2, TP3

Commit message: Started placing some components, finally
Parts:
- added MK1: IML-0688, Murata-Fresnel:IML-0688, symbol Mounting_Hole
- D1: footprint Air_Coils_SML_NEOSID:Neosid_Air-Coil_SML_6-10turn_HDM0431A-HDM1031A -> Diodes_SMD:D_SOD-123
Changed lines of the file:
@@
 F 0 "D1" H 6000 3350 50  0000 C CNN
 F 1 "1N4148X-TP" H 6000 3050 50  0000 C CNN
-F 2 "Air_Coils_SML_NEOSID:Neosid_Air-Coil_SML_6-10turn_HDM0431A-HDM1031A" H 6000 2950 50  0001 C CNN
+F 2 "Diodes_SMD:D_SOD-123" H 6000 2950 50  0001 C CNN
 F 3 "http://www.mouser.com/ds/2/258/1N4148X(SOD-523)-349105.pdf" H 6000 2850 50  0001 C CNN
 F 4 "Diodes - General Purpose, Power, Switching 150mA 75V" H 6000 2750 50  0001 C CNN "Description"
@@
 	2950 1750 2950 1700
 Connection ~ 2950 1700
+$Comp
+L Mounting_Hole MK1
+U 1 1 5A8B525D
+P 4700 6400
+F 0 "MK1" H 4700 6600 50  0000 C CNN
+F 1 "IML-0688" H 4700 6525 50  0000 C CNN
+F 2 "Murata-Fresnel:IML-0688" H 4700 6400 50  0001 C CNN
+F 3 "" H 4700 6400 50  0001 C CNN
+	1    4700 6400
+	1    0    0    -1
+$EndComp
 $EndSCHEMATC
