File: pcb/user.sch (KiCad schematic (older format))
At the start: 29 parts

Commit message: Reverted to KiCad 4.0.7
+ Reworked debouncing for pushbuttons
Parts:
- removed C? (x2): 2200pF, symbol device:C_Small
- removed R? (x2): 47K, symbol device:R
- removed SW? (x2): SW_Push, symbol switches:SW_Push
- added C? (x2): 100nF, symbol device:C_Small
- added IC?: SI2302CDS-T1-GE3, SOT95P237X112-3N, symbol SI2302CDS-T1-GE3:SI2302CDS-T1-GE3
- added R?: 1K, symbol device:R
- added R? (x3): 10k, symbol device:R
- added R? (x2): 100k, symbol device:R
- added SW? (x2): SW_Push, symbol switches:SW_Push
- C?: value 2200pF -> 100nF
- R?: value 47K -> 100k
Connections:
- net labels added: EINK_PWR, EINK_VCC
- wire segments 93 -> 85
Other:
- note added: "E-Ink power on/off switch controlled by MCU"
- moved on the sheet: R?

Commit message: MCU change, again
STM32L0 had quite a big problem, common reference for the comparators.
Another minus was the missing SWO for debugging.

STM32L4 has floating point, and most importantly, has embedded OPAMPS!
This means I can directly plug in the filter to the analog inputs and
everything is software. 2 opamps and 2 comparators (if needed).
External circuitry would be minimal for the PIR sensor.

It also means that I can read with the embedded 12-bit ADC the
amplified values. Precision is not crucial, we are interested in dips
and swells.
Parts:
- added C? (x2): 100nF, symbol device:C_Small
- added R? (x2): 100k, symbol device:R
- added R? (x2): 10k, symbol device:R
- added SW? (x2): SW_Push, symbol switches:SW_Push
Connections:
- net labels added: Down, Left, OK, Right, Up
- net labels removed: CenterButton, LeftButton, RightButton
- wire segments 85 -> 99
Other:
- moved on the sheet: R?

Commit message: Renamed all components
Parts:
- gave numbers to parts that had none: 42

Commit message: Replaced original PIR symbol and ran ERC tests
Connections:
- wire segments 99 -> 100
Changed lines of the file:
@@
 LIBS:ab2_xtal
 LIBS:EL817S
+LIBS:IRA-S210ST01
 LIBS:pir-cache
 EELAYER 25 0
@@
 $EndDescr
 $Comp
-L power:VCC #PWR15
+L power:VCC #PWR015
 U 1 1 5A7F0431
 P 1200 1400
-F 0 "#PWR15" H 1200 1250 50  0001 C CNN
+F 0 "#PWR015" H 1200 1250 50  0001 C CNN
 F 1 "VCC" H 1200 1550 50  0000 C CNN
 F 2 "" H 1200 1400 50  0001 C CNN
@@
 $EndComp
 $Comp
-L power:Earth #PWR16
+L power:Earth #PWR016
 U 1 1 5A7F044C
 P 1200 2550
-F 0 "#PWR16" H 1200 2300 50  0001 C CNN
+F 0 "#PWR016" H 1200 2300 50  0001 C CNN
 F 1 "Earth" H 1200 2400 50  0001 C CNN
 F 2 "" H 1200 2550 50  0001 C CNN
@@
 	1750 1950 1750 2100
 $Comp
-L power:Earth #PWR17
+L power:Earth #PWR017
 U 1 1 5A7F0458
 P 1750 2400
-F 0 "#PWR17" H 1750 2150 50  0001 C CNN
+F 0 "#PWR017" H 1750 2150 50  0001 C CNN
 F 1 "Earth" H 1750 2250 50  0001 C CNN
 F 2 "" H 1750 2400 50  0001 C CNN
@@
 $EndComp
 $Comp
-L power:Earth #PWR25
+L power:Earth #PWR018
 U 1 1 5A7F6EBE
 P 5150 4950
-F 0 "#PWR25" H 5150 4700 50  0001 C CNN
+F 0 "#PWR018" H 5150 4700 50  0001 C CNN
 F 1 "Earth" H 5150 4800 50  0001 C CNN
 F 2 "" H 5150 4950 50  0001 C CNN
@@
 	7850 4900 9400 4900
 $Comp
-L power:Earth #PWR33
+L power:Earth #PWR019
 U 1 1 5A7F8DE2
 P 7850 4800
-F 0 "#PWR33" H 7850 4550 50  0001 C CNN
+F 0 "#PWR019" H 7850 4550 50  0001 C CNN
 F 1 "Earth" H 7850 4650 50  0001 C CNN
 F 2 "" H 7850 4800 50  0001 C CNN
@@
 Connection ~ 5150 4800
 $Comp
-L power:Earth #PWR38
+L power:Earth #PWR020
 U 1 1 5A7FC712
 P 9750 4950
-F 0 "#PWR38" H 9750 4700 50  0001 C CNN
+F 0 "#PWR020" H 9750 4700 50  0001 C CNN
 F 1 "Earth" H 9750 4800 50  0001 C CNN
 F 2 "" H 9750 4950 50  0001 C CNN
@@
 Connection ~ 9750 4900
 Wire Wire Line
-	9750 4700 9150 4700
+	9100 4700 9750 4700
 Connection ~ 9750 4700
 Wire Wire Line
@@
 	8100 5500 7850 5500
 $Comp
-L power:Earth #PWR30
+L power:Earth #PWR021
 U 1 1 5A80C7A8
-P 6450 5500
-F 0 "#PWR30" H 6450 5250 50  0001 C CNN
-F 1 "Earth" H 6450 5350 50  0001 C CNN
-F 2 "" H 6450 5500 50  0001 C CNN
-F 3 "~" H 6450 5500 50  0001 C CNN
-	1    6450 5500
+P 6400 5500
+F 0 "#PWR021" H 6400 5250 50  0001 C CNN
+F 1 "Earth" H 6400 5350 50  0001 C CNN
+F 2 "" H 6400 5500 50  0001 C CNN
+F 3 "~" H 6400 5500 50  0001 C CNN
+	1    6400 5500
 	0    1    1    0
 $EndComp
 $Comp
-L power:Earth #PWR35
+L power:Earth #PWR022
 U 1 1 5A80C7EF
 P 8300 5400
-F 0 "#PWR35" H 8300 5150 50  0001 C CNN
+F 0 "#PWR022" H 8300 5150 50  0001 C CNN
 F 1 "Earth" H 8300 5250 50  0001 C CNN
 F 2 "" H 8300 5400 50  0001 C CNN
@@
 $EndComp
 $Comp
-L power:Earth #PWR23
+L power:Earth #PWR023
 U 1 1 5A81732B
 P 4600 3350
-F 0 "#PWR23" H 4600 3100 50  0001 C CNN
+F 0 "#PWR023" H 4600 3100 50  0001 C CNN
 F 1 "Earth" H 4600 3200 50  0001 C CNN
 F 2 "" H 4600 3350 50  0001 C CNN
@@
 $EndComp
 $Comp
-L power:Earth #PWR18
+L power:Earth #PWR024
 U 1 1 5A82A5F3
 P 2600 4700
-F 0 "#PWR18" H 2600 4450 50  0001 C CNN
+F 0 "#PWR024" H 2600 4450 50  0001 C CNN
 F 1 "Earth" H 2600 4550 50  0001 C CNN
 F 2 "" H 2600 4700 50  0001 C CNN
@@
 	2600 4550 2600 4700
 $Comp
-L power:Earth #PWR19
+L power:Earth #PWR025
 U 1 1 5A831908
 P 2700 6000
-F 0 "#PWR19" H 2700 5750 50  0001 C CNN
+F 0 "#PWR025" H 2700 5750 50  0001 C CNN
 F 1 "Earth" H 2700 5850 50  0001 C CNN
 F 2 "" H 2700 6000 50  0001 C CNN
@@
 	4350 6650 5000 6650
 $Comp
-L power:Earth #PWR24
+L power:Earth #PWR026
 U 1 1 5A7EF878
 P 4800 7300
-F 0 "#PWR24" H 4800 7050 50  0001 C CNN
+F 0 "#PWR026" H 4800 7050 50  0001 C CNN
 F 1 "Earth" H 4800 7150 50  0001 C CNN
 F 2 "" H 4800 7300 50  0001 C CNN
@@
 EINK_PWR
 $Comp
-L power:VCC #PWR29
+L power:VCC #PWR027
 U 1 1 5A7EFC51
 P 6050 6450
-F 0 "#PWR29" H 6050 6300 50  0001 C CNN
+F 0 "#PWR027" H 6050 6300 50  0001 C CNN
 F 1 "VCC" H 6050 6600 50  0000 C CNN
 F 2 "" H 6050 6450 50  0001 C CNN
@@
 Connection ~ 1200 1950
 $Comp
-L power:VCC #PWR26
+L power:VCC #PWR028
 U 1 1 5A7F43D1
 P 5450 1350
-F 0 "#PWR26" H 5450 1200 50  0001 C CNN
+F 0 "#PWR028" H 5450 1200 50  0001 C CNN
 F 1 "VCC" H 5450 1500 50  0000 C CNN
 F 2 "" H 5450 1350 50  0001 C CNN
@@
 $EndComp
 $Comp
-L power:Earth #PWR27
+L power:Earth #PWR029
 U 1 1 5A7F43E9
 P 5450 2500
-F 0 "#PWR27" H 5450 2250 50  0001 C CNN
+F 0 "#PWR029" H 5450 2250 50  0001 C CNN
 F 1 "Earth" H 5450 2350 50  0001 C CNN
 F 2 "" H 5450 2500 50  0001 C CNN
@@
 	6000 1900 6000 2050
 $Comp
-L power:Earth #PWR28
+L power:Earth #PWR030
 U 1 1 5A7F43F3
 P 6000 2350
-F 0 "#PWR28" H 6000 2100 50  0001 C CNN
+F 0 "#PWR030" H 6000 2100 50  0001 C CNN
 F 1 "Earth" H 6000 2200 50  0001 C CNN
 F 2 "" H 6000 2350 50  0001 C CNN
@@
 Connection ~ 5450 1900
 $Comp
-L power:VCC #PWR31
+L power:VCC #PWR031
 U 1 1 5A7F4771
 P 7400 1300
-F 0 "#PWR31" H 7400 1150 50  0001 C CNN
+F 0 "#PWR031" H 7400 1150 50  0001 C CNN
 F 1 "VCC" H 7400 1450 50  0000 C CNN
 F 2 "" H 7400 1300 50  0001 C CNN
@@
 $EndComp
 $Comp
-L power:Earth #PWR32
+L power:Earth #PWR032
 U 1 1 5A7F4789
 P 7400 2450
-F 0 "#PWR32" H 7400 2200 50  0001 C CNN
+F 0 "#PWR032" H 7400 2200 50  0001 C CNN
 F 1 "Earth" H 7400 2300 50  0001 C CNN
 F 2 "" H 7400 2450 50  0001 C CNN
@@
 	7950 1850 7950 2000
 $Comp
-L power:Earth #PWR34
+L power:Earth #PWR033
 U 1 1 5A7F4793
 P 7950 2300
-F 0 "#PWR34" H 7950 2050 50  0001 C CNN
+F 0 "#PWR033" H 7950 2050 50  0001 C CNN
 F 1 "Earth" H 7950 2150 50  0001 C CNN
 F 2 "" H 7950 2300 50  0001 C CNN
@@
 Connection ~ 7400 1850
 $Comp
-L power:VCC #PWR20
+L power:VCC #PWR034
 U 1 1 5A81CDD6
 P 3350 1350
-F 0 "#PWR20" H 3350 1200 50  0001 C CNN
+F 0 "#PWR034" H 3350 1200 50  0001 C CNN
 F 1 "VCC" H 3350 1500 50  0000 C CNN
 F 2 "" H 3350 1350 50  0001 C CNN
@@
 $EndComp
 $Comp
-L power:Earth #PWR21
+L power:Earth #PWR035
 U 1 1 5A81CDEE
 P 3350 2500
-F 0 "#PWR21" H 3350 2250 50  0001 C CNN
+F 0 "#PWR035" H 3350 2250 50  0001 C CNN
 F 1 "Earth" H 3350 2350 50  0001 C CNN
 F 2 "" H 3350 2500 50  0001 C CNN
@@
 	3900 1900 3900 2050
 $Comp
-L power:Earth #PWR22
+L power:Earth #PWR036
 U 1 1 5A81CDF8
 P 3900 2350
-F 0 "#PWR22" H 3900 2100 50  0001 C CNN
+F 0 "#PWR036" H 3900 2100 50  0001 C CNN
 F 1 "Earth" H 3900 2200 50  0001 C CNN
 F 2 "" H 3900 2350 50  0001 C CNN
@@
 Connection ~ 3350 1900
 $Comp
-L power:VCC #PWR36
+L power:VCC #PWR037
 U 1 1 5A81D403
 P 9250 1300
-F 0 "#PWR36" H 9250 1150 50  0001 C CNN
+F 0 "#PWR037" H 9250 1150 50  0001 C CNN
 F 1 "VCC" H 9250 1450 50  0000 C CNN
 F 2 "" H 9250 1300 50  0001 C CNN
@@
 $EndComp
 $Comp
-L power:Earth #PWR37
+L power:Earth #PWR038
 U 1 1 5A81D41B
 P 9250 2450
-F 0 "#PWR37" H 9250 2200 50  0001 C CNN
+F 0 "#PWR038" H 9250 2200 50  0001 C CNN
 F 1 "Earth" H 9250 2300 50  0001 C CNN
 F 2 "" H 9250 2450 50  0001 C CNN
@@
 	9800 1850 9800 2000
 $Comp
-L power:Earth #PWR39
+L power:Earth #PWR039
 U 1 1 5A81D425
 P 9800 2300
-F 0 "#PWR39" H 9800 2050 50  0001 C CNN
+F 0 "#PWR039" H 9800 2050 50  0001 C CNN
 F 1 "Earth" H 9800 2150 50  0001 C CNN
 F 2 "" H 9800 2300 50  0001 C CNN
@@
 Text HLabel 1950 1950 2    60   Input ~ 0
 Left
+Wire Wire Line
+	6400 5500 6450 5500
 $EndSCHEMATC

Commit message: Added testpoints
Parts:
- added TP11, TP12, TP13, TP14, TP15, TP16, TP17, TP18, TP19, TP20, TP21, TP22: TEST, symbol TEST
- renumbered R11 to R14, R12 to R15, R13 to R16, R14 to R17, R15 to R18, R16 to R19, R17 to R20, R18 to R21, R19 to R22, R20 to R23, R21 to R24, R22 to R25, R23 to R26
Connections:
- wire segments 100 -> 114
