File: pcb/user.sch (KiCad schematic (older format))
At the start: 54 parts, among them IC5 SI2302CDS-T1-GE3, IC6 SI2302CDS-T1-GE3, J2 FH12-24S-0.5SH(55), SW1 SW_Push, SW2 SW_Push, SW3 SW_Push, SW4 SW_Push, SW5 SW_Push

Commit message: Assigned footprints to all components
Parts:
- C18, C19, C20, C21, C22, C23, C24, C25, C26, C27, C28, C29, C30, C31, C32, C33, C34: footprint (none) -> Capacitors_SMD:C_1210
- IC5, IC6: footprint SOT95P237X112-3N -> SI2323DS-T1-E3:SOT95P237X112-3N
- J2: footprint FH12-24S-0.5SH(55) -> FH12-24S-0.5SH(55):FH12-24S-0.5SH(55)
- L1: footprint (none) -> Inductors_SMD:L_0402
- R14, R15, R16, R17, R18, R19, R20, R21, R22, R23, R24, R25, R26: footprint (none) -> Resistors_SMD:R_1210
- SW1, SW2, SW3, SW4, SW5: footprint (none) -> Buttons_Switches_SMD:SW_SPST_Panasonic_EVQPL_3PL_5PL_PT_A08
- TP11, TP12, TP13, TP14, TP15, TP16, TP17, TP18, TP19, TP20, TP21, TP22: footprint (none) -> Measurement_Points:Measurement_Point_Round-TH_Small

Commit message: Reassigned some footprints, added some libraries
Normally I can start working on PCB.
Parts:
- removed IC5, IC6: SI2302CDS-T1-GE3, SI2323DS-T1-E3:SOT95P237X112-3N, symbol SI2302CDS-T1-GE3:SI2302CDS-T1-GE3
- added Q2, Q3: RE1C002UN, RE1C002UNTCL:SOT50P160X85-3N, symbol Q_NMOS_GSD
- C18, C19, C20, C21, C22, C23, C24, C25, C26, C27, C28, C29, C30, C31, C32, C33, C34: footprint Capacitors_SMD:C_1210 -> Capacitors_SMD:C_1206
- D3, D4, D5: footprint Diodes_SMD:SOD-123 -> MBR0530:SOD3716X135N
- R14, R15, R16, R17, R18, R19, R21, R22, R23, R24, R25, R26: footprint Resistors_SMD:R_1210 -> Resistors_SMD:R_1206
- R20: value 1K -> 10k; footprint Resistors_SMD:R_1210 -> Resistors_SMD:R_1206
Connections:
- wire segments 114 -> 115

Commit message: More work on the PCB
The opamp circuit is done.
Currently working on camera interface.
TODO: screen, buttons.
Parts:
- C19: value 100n -> 4.7uF
- C31: value 1uF -> 4.7uF
- L1: value 68nH -> 68uH
- R17: value 3R -> 0.47
Changed lines of the file:
@@
 LIBS:xilinx
 LIBS:zetex
-LIBS:SparkFun
-LIBS:ab2_7segment
-LIBS:ab2_audio
-LIBS:ab2_buffer
-LIBS:ab2_capacitor
-LIBS:ab2_connectivity
-LIBS:ab2_dac
-LIBS:ab2_diode
-LIBS:ab2_fuse
-LIBS:ab2_gpio_expansion
-LIBS:ab2_header
-LIBS:ab2_idc
-LIBS:ab2_inductor
-LIBS:ab2_input_devices
-LIBS:ab2_jumper
-LIBS:ab2_lcd
-LIBS:ab2_led
-LIBS:ab2_memory
-LIBS:ab2_opamp
-LIBS:ab2_pinouts
-LIBS:ab2_pot
-LIBS:ab2_power
-LIBS:ab2_regulator
-LIBS:ab2_relay
-LIBS:ab2_resistor
-LIBS:ab2_sensor
-LIBS:ab2_stepper
-LIBS:ab2_supply
-LIBS:ab2_terminal_block
-LIBS:ab2_test
-LIBS:ab2_transistor
-LIBS:ab2_uC
-LIBS:ab2_usb
-LIBS:ab2_xtal
 LIBS:EL817S
 LIBS:IRA-S210ST01
@@
 P 8750 4600
 F 0 "C31" H 8760 4670 50  0000 L CNN
-F 1 "1uF" H 8760 4520 50  0000 L CNN
+F 1 "4.7uF" H 8760 4520 50  0000 L CNN
 F 2 "Capacitors_SMD:C_1206" H 8750 4600 50  0001 C CNN
 F 3 "" H 8750 4600 50  0001 C CNN
@@
 P 3050 4200
 F 0 "L1" V 3240 4200 50  0000 C CNN
-F 1 "68nH" V 3149 4200 50  0000 C CNN
+F 1 "68uH" V 3149 4200 50  0000 C CNN
 F 2 "Inductors_SMD:L_0402" H 3050 4200 50  0001 C CNN
 F 3 "" H 3050 4200 50  0001 C CNN
@@
 P 2600 4450
 F 0 "C19" H 2610 4520 50  0000 L CNN
-F 1 "100n" H 2610 4370 50  0000 L CNN
+F 1 "4.7uF" H 2610 4370 50  0000 L CNN
 F 2 "Capacitors_SMD:C_1206" H 2600 4450 50  0001 C CNN
 F 3 "" H 2600 4450 50  0001 C CNN
@@
 P 2900 5700
 F 0 "R17" V 2980 5700 50  0000 C CNN
-F 1 "3R" V 2900 5700 50  0000 C CNN
+F 1 "0.47" V 2900 5700 50  0000 C CNN
 F 2 "Resistors_SMD:R_1206" V 2830 5700 50  0001 C CNN
 F 3 "" H 2900 5700 50  0001 C CNN

Commit message: Finished the display components placement.
Parts:
- L1: footprint Inductors_SMD:L_0402 -> Inductors_SMD:L_1206
Changed lines of the file:
@@
 LIBS:xilinx
 LIBS:zetex
+LIBS:SparkFun
+LIBS:ab2_7segment
+LIBS:ab2_audio
+LIBS:ab2_buffer
+LIBS:ab2_capacitor
+LIBS:ab2_connectivity
+LIBS:ab2_dac
+LIBS:ab2_diode
+LIBS:ab2_fuse
+LIBS:ab2_gpio_expansion
+LIBS:ab2_header
+LIBS:ab2_idc
+LIBS:ab2_inductor
+LIBS:ab2_input_devices
+LIBS:ab2_jumper
+LIBS:ab2_lcd
+LIBS:ab2_led
+LIBS:ab2_memory
+LIBS:ab2_opamp
+LIBS:ab2_pinouts
+LIBS:ab2_pot
+LIBS:ab2_power
+LIBS:ab2_regulator
+LIBS:ab2_relay
+LIBS:ab2_resistor
+LIBS:ab2_sensor
+LIBS:ab2_stepper
+LIBS:ab2_supply
+LIBS:ab2_terminal_block
+LIBS:ab2_test
+LIBS:ab2_transistor
+LIBS:ab2_uC
+LIBS:ab2_usb
+LIBS:ab2_xtal
 LIBS:EL817S
 LIBS:IRA-S210ST01
@@
 F 0 "L1" V 3240 4200 50  0000 C CNN
 F 1 "68uH" V 3149 4200 50  0000 C CNN
-F 2 "Inductors_SMD:L_0402" H 3050 4200 50  0001 C CNN
+F 2 "Inductors_SMD:L_1206" H 3050 4200 50  0001 C CNN
 F 3 "" H 3050 4200 50  0001 C CNN
 	1    3050 4200

Commit message: Placed all components
Still some routing to do though, and many TP's are not placed.
Parts:
- removed TP14, TP19, TP20, TP21, TP22: TEST, Measurement_Points:Measurement_Point_Round-TH_Small, symbol TEST
Changed lines of the file:
@@
 Text HLabel 1950 1950 2    60   Input ~ 0
 Left
-$Comp
-L TEST TP14
-U 1 1 5A83C384
-P 1750 1950
-F 0 "TP14" H 1750 2250 50  0000 C BNN
-F 1 "TEST" H 1750 2200 50  0000 C CNN
-F 2 "Measurement_Points:Measurement_Point_Round-TH_Small" H 1750 1950 50  0001 C CNN
-F 3 "" H 1750 1950 50  0001 C CNN
-	1    1750 1950
-	1    0    0    -1
-$EndComp
-$Comp
-L TEST TP19
-U 1 1 5A83C448
-P 3900 1900
-F 0 "TP19" H 3900 2200 50  0000 C BNN
-F 1 "TEST" H 3900 2150 50  0000 C CNN
-F 2 "Measurement_Points:Measurement_Point_Round-TH_Small" H 3900 1900 50  0001 C CNN
-F 3 "" H 3900 1900 50  0001 C CNN
-	1    3900 1900
-	1    0    0    -1
-$EndComp
-$Comp
-L TEST TP20
-U 1 1 5A83C6BC
-P 6000 1900
-F 0 "TP20" H 6000 2200 50  0000 C BNN
-F 1 "TEST" H 6000 2150 50  0000 C CNN
-F 2 "Measurement_Points:Measurement_Point_Round-TH_Small" H 6000 1900 50  0001 C CNN
-F 3 "" H 6000 1900 50  0001 C CNN
-	1    6000 1900
-	1    0    0    -1
-$EndComp
-$Comp
-L TEST TP21
-U 1 1 5A83C79B
-P 7950 1850
-F 0 "TP21" H 7950 2150 50  0000 C BNN
-F 1 "TEST" H 7950 2100 50  0000 C CNN
-F 2 "Measurement_Points:Measurement_Point_Round-TH_Small" H 7950 1850 50  0001 C CNN
-F 3 "" H 7950 1850 50  0001 C CNN
-	1    7950 1850
-	1    0    0    -1
-$EndComp
-$Comp
-L TEST TP22
-U 1 1 5A83C945
-P 9800 1850
-F 0 "TP22" H 9800 2150 50  0000 C BNN
-F 1 "TEST" H 9800 2100 50  0000 C CNN
-F 2 "Measurement_Points:Measurement_Point_Round-TH_Small" H 9800 1850 50  0001 C CNN
-F 3 "" H 9800 1850 50  0001 C CNN
-	1    9800 1850
-	1    0    0    -1
-$EndComp
 Text HLabel 1050 6750 0    50   Input ~ 0
 EINK_MOSI

Commit message: OK button MOVED TO A WKUP pin. PCB routing done.
DRC passed.
Unconnected tracks : 0.
Parts:
- TP11, TP12, TP13, TP15, TP16, TP17, TP18: footprint Measurement_Points:Measurement_Point_Round-TH_Small -> Measurement_Points:Measurement_Point_Round-SMD-Pad_Small
Changed lines of the file:
@@
 F 0 "TP11" H 1150 6950 50  0000 C BNN
 F 1 "TEST" H 1150 6900 50  0000 C CNN
-F 2 "Measurement_Points:Measurement_Point_Round-TH_Small" H 1150 6650 50  0001 C CNN
+F 2 "Measurement_Points:Measurement_Point_Round-SMD-Pad_Small" H 1150 6650 50  0001 C CNN
 F 3 "" H 1150 6650 50  0001 C CNN
 	1    1150 6650
@@
 F 0 "TP12" H 1350 6950 50  0000 C BNN
 F 1 "TEST" H 1350 6900 50  0000 C CNN
-F 2 "Measurement_Points:Measurement_Point_Round-TH_Small" H 1350 6650 50  0001 C CNN
+F 2 "Measurement_Points:Measurement_Point_Round-SMD-Pad_Small" H 1350 6650 50  0001 C CNN
 F 3 "" H 1350 6650 50  0001 C CNN
 	1    1350 6650
@@
 F 0 "TP13" H 1550 6950 50  0000 C BNN
 F 1 "TEST" H 1550 6900 50  0000 C CNN
-F 2 "Measurement_Points:Measurement_Point_Round-TH_Small" H 1550 6650 50  0001 C CNN
+F 2 "Measurement_Points:Measurement_Point_Round-SMD-Pad_Small" H 1550 6650 50  0001 C CNN
 F 3 "" H 1550 6650 50  0001 C CNN
 	1    1550 6650
@@
 F 0 "TP15" H 1750 6950 50  0000 C BNN
 F 1 "TEST" H 1750 6900 50  0000 C CNN
-F 2 "Measurement_Points:Measurement_Point_Round-TH_Small" H 1750 6650 50  0001 C CNN
+F 2 "Measurement_Points:Measurement_Point_Round-SMD-Pad_Small" H 1750 6650 50  0001 C CNN
 F 3 "" H 1750 6650 50  0001 C CNN
 	1    1750 6650
@@
 F 0 "TP16" H 1950 6950 50  0000 C BNN
 F 1 "TEST" H 1950 6900 50  0000 C CNN
-F 2 "Measurement_Points:Measurement_Point_Round-TH_Small" H 1950 6650 50  0001 C CNN
+F 2 "Measurement_Points:Measurement_Point_Round-SMD-Pad_Small" H 1950 6650 50  0001 C CNN
 F 3 "" H 1950 6650 50  0001 C CNN
 	1    1950 6650
@@
 F 0 "TP17" H 2150 6950 50  0000 C BNN
 F 1 "TEST" H 2150 6900 50  0000 C CNN
-F 2 "Measurement_Points:Measurement_Point_Round-TH_Small" H 2150 6650 50  0001 C CNN
+F 2 "Measurement_Points:Measurement_Point_Round-SMD-Pad_Small" H 2150 6650 50  0001 C CNN
 F 3 "" H 2150 6650 50  0001 C CNN
 	1    2150 6650
@@
 F 0 "TP18" H 2350 6950 50  0000 C BNN
 F 1 "TEST" H 2350 6900 50  0000 C CNN
-F 2 "Measurement_Points:Measurement_Point_Round-TH_Small" H 2350 6650 50  0001 C CNN
+F 2 "Measurement_Points:Measurement_Point_Round-SMD-Pad_Small" H 2350 6650 50  0001 C CNN
 F 3 "" H 2350 6650 50  0001 C CNN
 	1    2350 6650

Commit message: Changed buttons from Panasonic to C&K
Parts:
- removed SW1, SW2, SW3, SW4, SW5: SW_Push, Buttons_Switches_SMD:SW_SPST_Panasonic_EVQPL_3PL_5PL_PT_A08, symbol switches:SW_Push
- added SW1, SW2, SW3, SW4, SW5: SW_DPST-KSC931, KSC931J_LFS:KSC8(J), symbol SW_DPST-KSC931
Connections:
- wire segments 115 -> 132
Changed lines of the file:
@@
 EESchema Schematic File Version 2
+LIBS:pir-rescue
 LIBS:74xgxx
 LIBS:74xx
@@
 LIBS:RE1C002UNTCL
 LIBS:SJ-2523-SMT-TR
+LIBS:KSC931J_LFS
 LIBS:pir-cache
 EELAYER 25 0
@@
 L power:VCC #PWR018
 U 1 1 5A7F0431
-P 1200 1400
-F 0 "#PWR018" H 1200 1250 50  0001 C CNN
-F 1 "VCC" H 1200 1550 50  0000 C CNN
-F 2 "" H 1200 1400 50  0001 C CNN
-F 3 "" H 1200 1400 50  0001 C CNN
-	1    1200 1400
+P 1200 1050
+F 0 "#PWR018" H 1200 900 50  0001 C CNN
+F 1 "VCC" H 1200 1200 50  0000 C CNN
+F 2 "" H 1200 1050 50  0001 C CNN
+F 3 "" H 1200 1050 50  0001 C CNN
+	1    1200 1050
 	1    0    0    -1
 $EndComp
@@
 	1    1200 2250
 	-1   0    0    1
-$EndComp
-$Comp
-L switches:SW_Push SW1
-U 1 1 5A7F043E
-P 1200 1700
-F 0 "SW1" H 1250 1800 50  0000 L CNN
-F 1 "SW_Push" H 1200 1640 50  0000 C CNN
-F 2 "Buttons_Switches_SMD:SW_SPST_Panasonic_EVQPL_3PL_5PL_PT_A08" H 1200 1900 50  0001 C CNN
-F 3 "" H 1200 1900 50  0001 C CNN
-	1    1200 1700
-	0    -1   -1   0
 $EndComp
 $Comp
@@
 L power:VCC #PWR031
 U 1 1 5A7F43D1
-P 5450 1350
-F 0 "#PWR031" H 5450 1200 50  0001 C CNN
-F 1 "VCC" H 5450 1500 50  0000 C CNN
-F 2 "" H 5450 1350 50  0001 C CNN
-F 3 "" H 5450 1350 50  0001 C CNN
-	1    5450 1350
+P 5450 1100
+F 0 "#PWR031" H 5450 950 50  0001 C CNN
+F 1 "VCC" H 5450 1250 50  0000 C CNN
+F 2 "" H 5450 1100 50  0001 C CNN
+F 3 "" H 5450 1100 50  0001 C CNN
+	1    5450 1100
 	1    0    0    -1
 $EndComp
@@
 $EndComp
 $Comp
-L switches:SW_Push SW3
-U 1 1 5A7F43DD
-P 5450 1650
-F 0 "SW3" H 5500 1750 50  0000 L CNN
-F 1 "SW_Push" H 5450 1590 50  0000 C CNN
-F 2 "Buttons_Switches_SMD:SW_SPST_Panasonic_EVQPL_3PL_5PL_PT_A08" H 5450 1850 50  0001 C CNN
-F 3 "" H 5450 1850 50  0001 C CNN
-	1    5450 1650
-	0    -1   -1   0
-$EndComp
-$Comp
 L device:C_Small C24
 U 1 1 5A7F43E3
@@
 L power:VCC #PWR034
 U 1 1 5A7F4771
-P 7400 1300
-F 0 "#PWR034" H 7400 1150 50  0001 C CNN
-F 1 "VCC" H 7400 1450 50  0000 C CNN
-F 2 "" H 7400 1300 50  0001 C CNN
-F 3 "" H 7400 1300 50  0001 C CNN
-	1    7400 1300
+P 7400 1050
+F 0 "#PWR034" H 7400 900 50  0001 C CNN
+F 1 "VCC" H 7400 1200 50  0000 C CNN
+F 2 "" H 7400 1050 50  0001 C CNN
+F 3 "" H 7400 1050 50  0001 C CNN
+	1    7400 1050
 	1    0    0    -1
 $EndComp
@@
 $EndComp
 $Comp
-L switches:SW_Push SW4
-U 1 1 5A7F477D
-P 7400 1600
-F 0 "SW4" H 7450 1700 50  0000 L CNN
-F 1 "SW_Push" H 7400 1540 50  0000 C CNN
-F 2 "Buttons_Switches_SMD:SW_SPST_Panasonic_EVQPL_3PL_5PL_PT_A08" H 7400 1800 50  0001 C CNN
-F 3 "" H 7400 1800 50  0001 C CNN
-	1    7400 1600
-	0    -1   -1   0
-$EndComp
-$Comp
 L device:C_Small C28
 U 1 1 5A7F4783
@@
 L power:VCC #PWR037
 U 1 1 5A81CDD6
-P 3350 1350
-F 0 "#PWR037" H 3350 1200 50  0001 C CNN
-F 1 "VCC" H 3350 1500 50  0000 C CNN
-F 2 "" H 3350 1350 50  0001 C CNN
-F 3 "" H 3350 1350 50  0001 C CNN
-	1    3350 1350
+P 3350 1050
+F 0 "#PWR037" H 3350 900 50  0001 C CNN
+F 1 "VCC" H 3350 1200 50  0000 C CNN
+F 2 "" H 3350 1050 50  0001 C CNN
+F 3 "" H 3350 1050 50  0001 C CNN
+	1    3350 1050
 	1    0    0    -1
 $EndComp
@@
 $EndComp
 $Comp
-L switches:SW_Push SW2
-U 1 1 5A81CDE2
-P 3350 1650
-F 0 "SW2" H 3400 1750 50  0000 L CNN
-F 1 "SW_Push" H 3350 1590 50  0000 C CNN
-F 2 "Buttons_Switches_SMD:SW_SPST_Panasonic_EVQPL_3PL_5PL_PT_A08" H 3350 1850 50  0001 C CNN
-F 3 "" H 3350 1850 50  0001 C CNN
-	1    3350 1650
-	0    -1   -1   0
-$EndComp
-$Comp
 L device:C_Small C21
 U 1 1 5A81CDE8
@@
 L power:VCC #PWR040
 U 1 1 5A81D403
-P 9250 1300
-F 0 "#PWR040" H 9250 1150 50  0001 C CNN
-F 1 "VCC" H 9250 1450 50  0000 C CNN
-F 2 "" H 9250 1300 50  0001 C CNN
-F 3 "" H 9250 1300 50  0001 C CNN
-	1    9250 1300
+P 9250 1050
+F 0 "#PWR040" H 9250 900 50  0001 C CNN
+F 1 "VCC" H 9250 1200 50  0000 C CNN
+F 2 "" H 9250 1050 50  0001 C CNN
+F 3 "" H 9250 1050 50  0001 C CNN
+	1    9250 1050
 	1    0    0    -1
 $EndComp
@@
 	1    9250 2150
 	-1   0    0    1
-$EndComp
-$Comp
-L switches:SW_Push SW5
-U 1 1 5A81D40F
-P 9250 1600
-F 0 "SW5" H 9300 1700 50  0000 L CNN
-F 1 "SW_Push" H 9250 1540 50  0000 C CNN
-F 2 "Buttons_Switches_SMD:SW_SPST_Panasonic_EVQPL_3PL_5PL_PT_A08" H 9250 1800 50  0001 C CNN
-F 3 "" H 9250 1800 50  0001 C CNN
-	1    9250 1600
-	0    -1   -1   0
 $EndComp
 $Comp
@@
 Connection ~ 9250 1850
 Wire Wire Line
-	9350 1850 9250 1850
+	9050 1850 9350 1850
 Connection ~ 9800 1850
 Wire Wire Line
-	9250 1300 9250 1400
+	9250 1050 9250 1250
 Wire Wire Line
 	9800 2200 9800 2300
@@
 	9650 1850 10000 1850
 Wire Wire Line
-	9250 1800 9250 2000
+	9250 1650 9250 2000
 Wire Wire Line
 	9250 2450 9250 2300
 Connection ~ 3350 1900
 Wire Wire Line
-	3450 1900 3350 1900
+	3150 1900 3450 1900
 Connection ~ 3900 1900
 Wire Wire Line
-	3350 1350 3350 1450
+	3350 1050 3350 1300
 Wire Wire Line
 	3900 2250 3900 2350
@@
 	3750 1900 4100 1900
 Wire Wire Line
-	3350 1850 3350 2050
+	3350 1700 3350 2050
 Wire Wire Line
 	3350 2500 3350 2350
 Connection ~ 7400 1850
 Wire Wire Line
-	7500 1850 7400 1850
+	7200 1850 7500 1850
 Connection ~ 7950 1850
 Wire Wire Line
-	7400 1300 7400 1400
+	7400 1050 7400 1250
 Wire Wire Line
 	7950 2200 7950 2300
@@
 Connection ~ 5450 1900
 Wire Wire Line
-	5550 1900 5450 1900
+	5250 1900 5550 1900
 Connection ~ 6000 1900
 Wire Wire Line
-	5450 1350 5450 1450
+	5450 1100 5450 1300
 Wire Wire Line
 	6000 2250 6000 2350
@@
 Connection ~ 1200 1950
 Wire Wire Line
-	1300 1950 1200 1950
+	1000 1950 1300 1950
 Connection ~ 1750 1950
 Wire Wire Line
-	1200 1400 1200 1500
+	1200 1050 1200 1350
 Wire Wire Line
 	6100 4900 6950 4900
@@
 Connection ~ 9750 4700
 Wire Wire Line
-	9100 4700 9750 4700
+	9750 4700 9100 4700
 Connection ~ 9750 4900
 Wire Wire Line
@@
 	1600 1950 1950 1950
 Wire Wire Line
-	1200 1900 1200 2100
+	1200 1750 1200 2100
 Wire Wire Line
 	1200 2550 1200 2400
@@
 Wire Wire Line
 	3750 5450 3750 5300
+$Comp
+L SW_DPST-KSC931 SW1
+U 1 1 5A8F4B6A
+P 1100 1550
+F 0 "SW1" H 1100 1750 50  0000 C CNN
+F 1 "SW_DPST-KSC931" H 1100 1350 50  0000 C CNN
+F 2 "KSC931J_LFS:KSC8(J)" H 1100 1550 50  0001 C CNN
+F 3 "" H 1100 1550 50  0001 C CNN
+	1    1100 1550
+	0    1    1    0
+$EndComp
+Wire Wire Line
+	1000 1350 1000 1250
+Wire Wire Line
+	1000 1250 1200 1250
+Connection ~ 1200 1250
+Wire Wire Line
+	1000 1750 1000 1950
+$Comp
+L SW_DPST-KSC931 SW2
+U 1 1 5A8F5ECA
+P 3250 1500
+F 0 "SW2" H 3250 1700 50  0000 C CNN
+F 1 "SW_DPST-KSC931" H 3250 1300 50  0000 C CNN
+F 2 "KSC931J_LFS:KSC8(J)" H 3250 1500 50  0001 C CNN
+F 3 "" H 3250 1500 50  0001 C CNN
+	1    3250 1500
+	0    1    1    0
+$EndComp
+Wire Wire Line
+	3150 1300 3150 1250
+Wire Wire Line
+	3150 1250 3350 1250
+Connection ~ 3350 1250
+Wire Wire Line
+	3150 1700 3150 1900
+$Comp
+L SW_DPST-KSC931 SW3
+U 1 1 5A8F6920
+P 5350 1500
+F 0 "SW3" H 5350 1700 50  0000 C CNN
+F 1 "SW_DPST-KSC931" H 5350 1300 50  0000 C CNN
+F 2 "KSC931J_LFS:KSC8(J)" H 5350 1500 50  0001 C CNN
+F 3 "" H 5350 1500 50  0001 C CNN
+	1    5350 1500
+	0    1    1    0
+$EndComp
+Wire Wire Line
+	5250 1300 5250 1200
+Wire Wire Line
+	5250 1200 5450 1200
+Connection ~ 5450 1200
+Wire Wire Line
+	5250 1700 5250 1900
+Wire Wire Line
+	5450 1700 5450 1900
+$Comp
+L SW_DPST-KSC931 SW4
+U 1 1 5A8F72C9
+P 7300 1450
+F 0 "SW4" H 7300 1650 50  0000 C CNN
+F 1 "SW_DPST-KSC931" H 7300 1250 50  0000 C CNN
+F 2 "KSC931J_LFS:KSC8(J)" H 7300 1450 50  0001 C CNN
+F 3 "" H 7300 1450 50  0001 C CNN
+	1    7300 1450
+	0    1    1    0
+$EndComp
+Wire Wire Line
+	7200 1650 7200 1850
+Wire Wire Line
+	7400 1650 7400 1850
+Wire Wire Line
+	7200 1250 7200 1200
+Wire Wire Line
+	7200 1200 7400 1200
+Connection ~ 7400 1200
+$Comp
+L SW_DPST-KSC931 SW5
+U 1 1 5A8F7CB8
+P 9150 1450
+F 0 "SW5" H 9150 1650 50  0000 C CNN
+F 1 "SW_DPST-KSC931" H 9150 1250 50  0000 C CNN
+F 2 "KSC931J_LFS:KSC8(J)" H 9150 1450 50  0001 C CNN
+F 3 "" H 9150 1450 50  0001 C CNN
+	1    9150 1450
+	0    1    1    0
+$EndComp
+Wire Wire Line
+	9050 1250 9050 1200
+Wire Wire Line
+	9050 1200 9250 1200
+Connection ~ 9250 1200
+Wire Wire Line
+	9050 1650 9050 1850
 $EndSCHEMATC
