File: pcb/user.sch (KiCad schematic (older format))
At the start: 49 parts, among them J2 FH12-24S-0.5SH(55), Q2 RE1C002UN, Q3 RE1C002UN, SW1 SW_DPST-KSC931, SW2 SW_DPST-KSC931, SW3 SW_DPST-KSC931, SW4 SW_DPST-KSC931, SW5 SW_DPST-KSC931

Commit message: Changed FPC display connector
Same model from Hirose but Top-connect not Bottom-connect as it
previously was. Huge mistake, got it in time.

Created GDEW027W3 schematic symbol for the display.
Parts:
- removed J2: FH12-24S-0.5SH(55), FH12-24S-0.5SH(55):FH12-24S-0.5SH(55), symbol FH12-24S-0.5SH(55):FH12-24S-0.5SH(55)
- added J2: GDEW027W3, FH12A-24S-0.5SH(55):FH12A-24S-0.5SH, symbol GDEW027W3
Connections:
- wire segments 132 -> 130
- no-connect marks 3 -> 2
