File: pcb/pir.kicad_pcb (KiCad board)
At the start: 2 copper layers, 0 parts

Commit message: Put the first components on layout
Parts:
- added BT1: CR2477 3V Battery, Battery_Holders:Keystone_105_1x2430-CoinCell, F.Cu at (147.2, 100.3)
- added C1: 100μF, Capacitors_SMD:C_1206, F.Cu at (269.2, 106.3)
- added C10: 3.3nF, Capacitors_SMD:C_1206, F.Cu at (269.2, 106.3)
- added C11: 22uF, Capacitors_SMD:C_1206, F.Cu at (269.2, 106.3)
- added C12, C9: 47nF, Capacitors_SMD:C_1206, F.Cu at (269.2, 106.3)
- added C13: 100u, Capacitors_SMD:CP_Elec_5x5.3, F.Cu at (269.2, 106.3)
- added C14: 10μF, Capacitors_SMD:C_1210, F.Cu at (269.2, 106.3)
- added C15: 1μF, Capacitors_SMD:C_1210, F.Cu at (269.2, 106.3)
- added C16: 0.1μF, Capacitors_SMD:C_1210, F.Cu at (269.2, 106.3)
- added C17: 0.01μF, Capacitors_SMD:C_1210, F.Cu at (269.2, 106.3)
- added C18, C21, C24, C28, C34, C38, C40: 100nF, Capacitors_SMD:C_1210, F.Cu at (269.2, 106.3)
- added C19, C20, C33: 100n, Capacitors_SMD:C_1210, F.Cu at (269.2, 106.3)
- added C2: 10μF, Capacitors_SMD:C_1206, F.Cu at (269.2, 106.3)
- added C22, C23, C25, C26, C27, C29, C30, C31, C32: 1uF, Capacitors_SMD:C_1210, F.Cu at (269.2, 106.3)
- added C3: 1μF, Capacitors_SMD:C_1206, F.Cu at (269.2, 106.3)
- added C35, C36, C37, C39: 12pF, Capacitors_SMD:C_1210, F.Cu at (269.2, 106.3)
- added C4: 0.1μF, Capacitors_SMD:C_1206, F.Cu at (269.2, 106.3)
- added C5: 0.01μF, Capacitors_SMD:C_1206, F.Cu at (269.2, 106.3)
- added C6: 1000pF, Capacitors_SMD:C_1206, F.Cu at (269.2, 106.3)
- added C7: 100pF, Capacitors_SMD:C_1206, F.Cu at (269.2, 106.3)
- added C8: 22μF, Capacitors_SMD:C_1206, F.Cu at (269.2, 106.3)
- added D1: 1N4148X-TP, Air_Coils_SML_NEOSID:Neosid_Air-Coil_SML_6-10turn_HDM0431A-HDM1031A, F.Cu at (269.2, 106.3)
- added IC1: MAX44009EDT+T, MAX44009EDT+T:SON65P200X200X65-7N, F.Cu at (280.9, 94.6)
- added IC2: IRA-S210ST01, IRA-S210ST01:IRA-S210ST01, F.Cu at (243.8, 109.2)
- added IC3, IC4: EL817S, EL817S:EL817S, F.Cu at (269.2, 106.3)
- added IC5, IC6: SI2302CDS-T1-GE3, SI2323DS-T1-E3:SOT95P237X112-3N, F.Cu at (269.2, 106.3)
- added J2: FH12-24S-0.5SH(55), FH12-24S-0.5SH(55):FH12-24S-0.5SH(55), F.Cu at (232.4, 95.2)
- added J3: SWD, Pin_Headers:Pin_Header_Angled_1x06_Pitch2.54mm, F.Cu at (158.8, 52.1)
- added J4: UART, Pin_Headers:Pin_Header_Angled_1x03_Pitch2.54mm, F.Cu at (257.8, 88.9)
- added JP1: Jumper, Pin_Headers:Pin_Header_Angled_1x02_Pitch2.54mm, F.Cu at (278.1, 82.5)
- added JP2: Jumper, Pin_Headers:Pin_Header_Angled_1x02_Pitch2.54mm, F.Cu at (269.2, 106.3)
- added JP3: Jumper_NC_Dual, Pin_Headers:Pin_Header_Angled_1x03_Pitch2.54mm, F.Cu at (269.2, 106.3)
- added L1: 68nH, Inductors_SMD:L_0402, F.Cu at (269.2, 106.3)
- added Q1: SI2323DS, SI2323DS-T1-E3:SOT95P237X112-3N, F.Cu at (269.2, 106.3)
- added R1: 0, Resistors_SMD:R_1210, F.Cu at (269.2, 106.3)
- added R10, R9: 1M, Resistors_SMD:R_1210, F.Cu at (269.2, 106.3)
- added R11: 3.3K, Resistors_SMD:R_1210, F.Cu at (269.2, 106.3)
- added R12, R13: 150, Resistors_SMD:R_1210, F.Cu at (269.2, 106.3)
- added R14, R18, R21, R23, R25: 100k, Resistors_SMD:R_1210, F.Cu at (269.2, 106.3)
- added R15, R16, R19, R2, R22, R24, R26, R3, R4: 10k, Resistors_SMD:R_1210, F.Cu at (269.2, 106.3)
- added R17: 3R, Resistors_SMD:R_1210, F.Cu at (269.2, 106.3)
- added R20, R27: 1K, Resistors_SMD:R_1210, F.Cu at (269.2, 106.3)
- added R5, R8: 13k, Resistors_SMD:R_1210, F.Cu at (269.2, 106.3)
- added R6: 56k, Resistors_SMD:R_1210, F.Cu at (269.2, 106.3)
- added R7: 680k, Resistors_SMD:R_1210, F.Cu at (269.2, 106.3)
- added SW1, SW2, SW3, SW4, SW5: SW_Push, Buttons_Switches_SMD:SW_SPST_Panasonic_EVQPL_3PL_5PL_PT_A08, F.Cu at (269.2, 106.3)
- added TP1, TP10, TP11, TP12, TP13, TP14, TP15, TP16, TP17, TP18, TP19, TP2, TP20, TP21, TP22, TP23, TP24, TP25, TP26, TP27, TP28, TP29, TP3, TP30, TP31, TP32, TP33, TP34, TP35, TP36, TP37, TP38, TP39, TP4, TP40, TP41, TP5, TP6, TP7, TP8, TP9: TEST, Measurement_Points:Measurement_Point_Round-TH_Small, F.Cu at (269.2, 106.3)
- added U1: STM32L476RETx, Housings_QFP:LQFP-64_10x10mm_Pitch0.5mm, F.Cu at (224.8, 113.0)
- added Y1, Y2: 32 Mhz, Crystals:Crystal_SMD_2012-2pin_2.0x1.2mm_HandSoldering, F.Cu at (269.2, 106.3)
